File: eagle/LCmeter0-perfboard-new.brd (EAGLE design)
At the start: 63.5 x 50.5 mm, 25 parts, among them IC1 PIC16F876A-X/SP, K2 DS2Y, Q1 20MHz, Q2 BC548, SW1 SPST, SW2 DPDT

Commit message: ...
Parts:
- IC1: device lc-meter:DIL28-3 -> mcu:DIL28-3
- SW1: device lc-meter:PB-5 -> mcu:PB-5
- SW2: device lc-meter:DPDT -> mcu:DPDT
Changed lines of the file:
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@@
 <element name="C9" library="rcl" package="C025-024X044" value="100nF" x="53.34" y="16.51" rot="R270"/>
 <element name="D1" library="diode" package="DO35-7" value="1N4148" x="13.97" y="5.08" rot="R180"/>
-<element name="IC1" library="lc-meter" package="DIL28-3" value="PIC16F876A-X/SP" x="46.99" y="21.59" rot="R270"/>
+<element name="IC1" library="mcu" package="DIL28-3" value="PIC16F876A-X/SP" x="46.99" y="21.59" rot="R270"/>
 <element name="K2" library="relay" package="DS2Y" value="DS2Y" x="13.97" y="16.51" rot="R90">
 <attribute name="OC_FARNELL" value="unknown" x="13.97" y="16.51" size="1.778" layer="27" rot="R90" display="off"/>
@@
 <element name="R5" library="resistor" package="0207/10" value="4.7kΩ" x="35.56" y="25.4" rot="R180"/>
 <element name="R6" library="resistor" package="0204V" value="10kΩ" x="29.21" y="7.62" rot="R180"/>
-<element name="SW1" library="lc-meter" package="PB-5" value="SPST" x="50.8" y="45.72" rot="R180"/>
-<element name="SW2" library="lc-meter" package="DPDT" value="DPDT" x="6.35" y="30.48" rot="R270"/>
+<element name="SW1" library="mcu" package="PB-5" value="SPST" x="50.8" y="45.72" rot="R180"/>
+<element name="SW2" library="mcu" package="DPDT" value="DPDT" x="6.35" y="30.48" rot="R270"/>
 </elements>
 <signals>

Commit message: ...
Parts:
- D1: device diode:DO35-7 -> d:DO35-7
- Q1: device crystal:HC49/S -> q:HC49/S
- Q2: device transistor-npn:TO92-EBC -> t:TO92-EBC
- R10, R5: device resistor:0207/10 -> r:0207/10
- R2, R3, R4, R6: device resistor:0204V -> r:0204V
Changed lines of the file:
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@@
 <element name="C8" library="rcl" package="E2,5-5" value="10μF" x="31.75" y="38.1"/>
 <element name="C9" library="rcl" package="C025-024X044" value="100nF" x="53.34" y="16.51" rot="R270"/>
-<element name="D1" library="diode" package="DO35-7" value="1N4148" x="13.97" y="5.08" rot="R180"/>
+<element name="D1" library="d" package="DO35-7" value="1N4148" x="13.97" y="5.08" rot="R180"/>
 <element name="IC1" library="mcu" package="DIL28-3" value="PIC16F876A-X/SP" x="46.99" y="21.59" rot="R270"/>
 <element name="K2" library="relay" package="DS2Y" value="DS2Y" x="13.97" y="16.51" rot="R90">
@@
 <attribute name="MF" value="" x="60.96" y="29.21" size="1.778" layer="27" rot="R90" display="off"/>
 </element>
-<element name="Q1" library="crystal" package="HC49/S" value="20MHz" x="38.1" y="15.24" rot="R270">
+<element name="Q1" library="q" package="HC49/S" value="20MHz" x="38.1" y="15.24" rot="R270">
 <attribute name="OC_FARNELL" value="1667008" x="38.1" y="15.24" size="1.778" layer="27" rot="R270" display="off"/>
 <attribute name="OC_NEWARK" value="unknown" x="38.1" y="15.24" size="1.778" layer="27" rot="R270" display="off"/>
@@
 <attribute name="MF" value="" x="38.1" y="15.24" size="1.778" layer="27" rot="R270" display="off"/>
 </element>
-<element name="Q2" library="transistor-npn" package="TO92-EBC" value="BC548" x="21.59" y="7.62" rot="R90"/>
+<element name="Q2" library="t" package="TO92-EBC" value="BC548" x="21.59" y="7.62" rot="R90"/>
 <element name="R1" library="rcl" package="0204/7" value="100kΩ" x="26.67" y="35.56"/>
-<element name="R10" library="resistor" package="0207/10" value="4.7kΩ" x="38.1" y="43.18" rot="R180"/>
-<element name="R2" library="resistor" package="0204V" value="100kΩ" x="22.86" y="29.21" rot="R270"/>
-<element name="R3" library="resistor" package="0204V" value="100kΩ" x="24.13" y="38.1"/>
-<element name="R4" library="resistor" package="0204V" value="47kΩ" x="38.1" y="34.29" rot="R90"/>
-<element name="R5" library="resistor" package="0207/10" value="4.7kΩ" x="35.56" y="25.4" rot="R180"/>
-<element name="R6" library="resistor" package="0204V" value="10kΩ" x="29.21" y="7.62" rot="R180"/>
+<element name="R10" library="r" package="0207/10" value="4.7kΩ" x="38.1" y="43.18" rot="R180"/>
+<element name="R2" library="r" package="0204V" value="100kΩ" x="22.86" y="29.21" rot="R270"/>
+<element name="R3" library="r" package="0204V" value="100kΩ" x="24.13" y="38.1"/>
+<element name="R4" library="r" package="0204V" value="47kΩ" x="38.1" y="34.29" rot="R90"/>
+<element name="R5" library="r" package="0207/10" value="4.7kΩ" x="35.56" y="25.4" rot="R180"/>
+<element name="R6" library="r" package="0204V" value="10kΩ" x="29.21" y="7.62" rot="R180"/>
 <element name="SW1" library="mcu" package="PB-5" value="SPST" x="50.8" y="45.72" rot="R180"/>
 <element name="SW2" library="mcu" package="DPDT" value="DPDT" x="6.35" y="30.48" rot="R270"/>
