File: eagle/LCmeter0-LCD-8pinlcd.sch (EAGLE design)
At the start: 25 parts, among them IC1 PIC16F876A-X/SP, K2 DS2Y, Q1 20MHz, Q2 BC548, SW1 SPST, SW2 DPDT

Commit message: ...
Parts:
- C3: device rcl:CPOL-EUE2.5-6 -> rcl:CPOL-EUE5-4
- C4: device rcl:CPOL-EUE5-6 -> rcl:CPOL-EUE5-4
- C5, C6: device rcl:C-EU050-025X075 -> rcl:C-EU050-024X044
- LCD1: value (none) -> HD44780
- Q1: device crystal:CRYSTALHC49U70 -> crystal:CRYSTALHC49U-V
- R1, R2, R4: device resistor:R-EU_0207/10 -> resistor:R-EU_0204/2V
- R6: value (none) -> 10kΩ
Connections:
- removed net N$1: C2.2, K23.P
- removed net VSS: C1.2, C4.-, C5.1, C6.1, C7.-, C8.-, C9.2, D1.A, IC1.VSS, IC1.VSS_2, K21.-, K23.S, LCD1.1, Q2.E, R2.1, SW1.P
- new net C2_CON: C2.2, K22.P
- new net GND: C1.2, C4.-, C5.1, C6.1, C7.-, C8.-, C9.2, IC1.VSS, IC1.VSS_2, K22.S, LCD1.1, Q2.E, R2.1, SW1.P
- net VCC: now also D1.A, K21.-
Other:
- moved on the sheet: D1, K2
Changed lines of the file:
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@@
 <setting verticaltext="up"/>
 </settings>
-<grid distance="0.05" unitdist="inch" unit="inch" style="lines" multiple="2" display="no" altdistance="0.025" altunitdist="inch" altunit="inch"/>
+<grid distance="0.05" unitdist="inch" unit="inch" style="lines" multiple="2" display="no" altdistance="0.01" altunitdist="inch" altunit="inch"/>
 <layers>
 <layer number="1" name="Top" color="4" fill="1" visible="yes" active="no"/>
@@
 <parts>
 <part name="IC1" library="lc-meter" deviceset="PIC16F876A-X/SP" device=""/>
-<part name="R1" library="resistor" deviceset="R-EU_" device="0207/10" value="100kΩ"/>
-<part name="R2" library="resistor" deviceset="R-EU_" device="0207/10" value="100kΩ"/>
+<part name="R1" library="resistor" deviceset="R-EU_" device="0204/2V" value="100kΩ"/>
+<part name="R2" library="resistor" deviceset="R-EU_" device="0204/2V" value="100kΩ"/>
 <part name="R3" library="resistor" deviceset="R-EU_" device="0204/2V" value="100kΩ"/>
-<part name="R4" library="resistor" deviceset="R-EU_" device="0207/10" value="47kΩ"/>
+<part name="R4" library="resistor" deviceset="R-EU_" device="0204/2V" value="47kΩ"/>
 <part name="R10" library="resistor" deviceset="R-EU_" device="0204/2V" value="4.7kΩ"/>
 <part name="C1" library="rcl" deviceset="C-EU" device="050-025X075" value="1nF"/>
 <part name="C2" library="rcl" deviceset="C-EU" device="050-025X075" value="1nF"/>
-<part name="C3" library="rcl" deviceset="CPOL-EU" device="E2.5-6" value="10μF"/>
-<part name="C4" library="rcl" deviceset="CPOL-EU" device="E5-6" value="10μF"/>
-<part name="C5" library="rcl" deviceset="C-EU" device="050-025X075" value="33pF"/>
-<part name="C6" library="rcl" deviceset="C-EU" device="050-025X075" value="33pF"/>
+<part name="C3" library="rcl" deviceset="CPOL-EU" device="E5-4" value="10μF"/>
+<part name="C4" library="rcl" deviceset="CPOL-EU" device="E5-4" value="10μF"/>
+<part name="C5" library="rcl" deviceset="C-EU" device="050-024X044" value="33pF"/>
+<part name="C6" library="rcl" deviceset="C-EU" device="050-024X044" value="33pF"/>
 <part name="C7" library="rcl" deviceset="CPOL-EU" device="E2.5-6" value="100μF"/>
 <part name="C8" library="rcl" deviceset="CPOL-EU" device="E2.5-5" value="10μF"/>
 <part name="C9" library="rcl" deviceset="C-EU" device="025-024X044" value="100nF"/>
-<part name="GND1" library="supply1" deviceset="GND" device=""/>
 <part name="GND2" library="supply1" deviceset="GND" device=""/>
 <part name="GND3" library="supply1" deviceset="GND" device=""/>
@@
 <part name="D1" library="diode" deviceset="1N4148" device="DO35-7" value="1N4148"/>
 <part name="L1" library="rcl" deviceset="L-US" device="0207/10" value="100μH"/>
-<part name="Q1" library="crystal" deviceset="CRYSTAL" device="HC49U70" value="20MHz"/>
+<part name="Q1" library="crystal" deviceset="CRYSTAL" device="HC49U-V" value="20MHz"/>
 <part name="P+1" library="supply1" deviceset="VCC" device=""/>
 <part name="GND11" library="supply1" deviceset="GND" device=""/>
@@
 <part name="Q2" library="transistor-npn" deviceset="BC548*" device=""/>
 <part name="GND8" library="supply1" deviceset="GND" device=""/>
-<part name="R6" library="rcl" deviceset="R-EU_" device="0207/10"/>
-<part name="LCD1" library="con-lstb" deviceset="MA08-1" device=""/>
+<part name="R6" library="rcl" deviceset="R-EU_" device="0207/10" value="10kΩ"/>
+<part name="LCD1" library="con-lstb" deviceset="MA08-1" device="" value="HD44780"/>
+<part name="P+7" library="supply1" deviceset="VCC" device=""/>
 </parts>
 <sheets>
@@
 <instance part="C2" gate="G$1" x="-11.43" y="20.32"/>
 <instance part="C3" gate="G$1" x="-3.81" y="30.48" smashed="yes" rot="R270">
-<attribute name="VALUE" x="-3.429" y="34.544" size="1.778" layer="96" rot="R180"/>
+<attribute name="NAME" x="-4.953" y="27.4574" size="1.778" layer="95" rot="R180"/>
+<attribute name="VALUE" x="-7.747" y="33.5026" size="1.778" layer="96"/>
 </instance>
 <instance part="C4" gate="G$1" x="21.59" y="5.08"/>
@@
 <attribute name="VALUE" x="-27.051" y="4.064" size="1.778" layer="96" rot="R90" align="center"/>
 </instance>
-<instance part="GND1" gate="1" x="1.27" y="-7.62"/>
 <instance part="GND2" gate="1" x="21.59" y="-7.62"/>
 <instance part="GND3" gate="1" x="36.83" y="-7.62"/>
 <instance part="GND4" gate="1" x="-45.72" y="-7.62"/>
 <instance part="GND5" gate="1" x="-19.05" y="-7.62"/>
-<instance part="GND6" gate="1" x="-8.89" y="-7.62"/>
+<instance part="GND6" gate="1" x="-5.08" y="-7.62"/>
 <instance part="GND7" gate="1" x="1.27" y="15.24" rot="MR0"/>
-<instance part="D1" gate="G$1" x="10.16" y="3.81" smashed="yes" rot="R90">
-<attribute name="NAME" x="11.43" y="5.08" size="1.778" layer="95" align="top-left"/>
-<attribute name="VALUE" x="11.43" y="2.54" size="1.778" layer="96" rot="R180" align="bottom-right"/>
+<instance part="D1" gate="G$1" x="10.16" y="0" smashed="yes" rot="MR270">
+<attribute name="NAME" x="11.43" y="-1.27" size="1.778" layer="95" rot="MR180" align="top-left"/>
+<attribute name="VALUE" x="11.43" y="1.27" size="1.778" layer="96" rot="MR0" align="bottom-right"/>
 </instance>
 <instance part="L1" gate="G$1" x="-29.21" y="25.4" rot="R90"/>
@@
 <attribute name="VALUE" x="146.05" y="1.27" size="1.778" layer="96" rot="R90" align="top-center"/>
 </instance>
-<instance part="K2" gate="1" x="1.27" y="3.81" smashed="yes">
-<attribute name="VALUE" x="2.54" y="-0.889" size="1.778" layer="96"/>
-<attribute name="PART" x="2.54" y="6.35" size="1.778" layer="95"/>
-</instance>
-<instance part="K2" gate="3" x="-11.43" y="6.35" rot="R180"/>
+<instance part="K2" gate="1" x="1.27" y="0" smashed="yes" rot="MR180">
+<attribute name="VALUE" x="2.54" y="4.699" size="1.778" layer="96" rot="MR180"/>
+<attribute name="PART" x="2.54" y="-2.54" size="1.778" layer="95" rot="MR180"/>
+</instance>
+<instance part="K2" gate="3" x="-34.29" y="-16.51" rot="R180"/>
 <instance part="P+6" gate="VCC" x="153.67" y="63.5" smashed="yes">
 <attribute name="VALUE" x="153.67" y="64.77" size="1.778" layer="96" align="bottom-center"/>
@@
 <instance part="R6" gate="G$1" x="114.3" y="2.54"/>
 <instance part="LCD1" gate="1" x="187.96" y="31.75" rot="MR0"/>
+<instance part="K2" gate="2" x="-11.43" y="5.08" rot="R180"/>
+<instance part="P+7" gate="VCC" x="10.16" y="11.43" smashed="yes">
+<attribute name="VALUE" x="10.16" y="12.7" size="1.778" layer="96" align="bottom-center"/>
+</instance>
 </instances>
 <busses>
@@
 </segment>
 </net>
-<net name="VSS" class="0">
+<net name="GND" class="0">
 <segment>
 <pinref part="R2" gate="G$1" pin="1"/>
 <pinref part="GND7" gate="1" pin="GND"/>
-</segment>
-<segment>
-<pinref part="GND1" gate="1" pin="GND"/>
-<wire x1="1.27" y1="-5.08" x2="1.27" y2="-2.54" width="0.1524" layer="91"/>
-<pinref part="D1" gate="G$1" pin="A"/>
-<wire x1="1.27" y1="-2.54" x2="10.16" y2="-2.54" width="0.1524" layer="91"/>
-<wire x1="10.16" y1="-2.54" x2="10.16" y2="1.27" width="0.1524" layer="91"/>
-<wire x1="1.27" y1="-1.27" x2="1.27" y2="-2.54" width="0.1524" layer="91"/>
-<junction x="1.27" y="-2.54"/>
-<pinref part="K2" gate="1" pin="-"/>
 </segment>
 <segment>
@@
 </segment>
 <segment>
-<pinref part="GND6" gate="1" pin="GND"/>
-<wire x1="-6.35" y1="1.27" x2="-8.89" y2="1.27" width="0.1524" layer="91"/>
-<wire x1="-8.89" y1="1.27" x2="-8.89" y2="-5.08" width="0.1524" layer="91"/>
-<pinref part="K2" gate="3" pin="S"/>
-</segment>
-<segment>
 <pinref part="SW1" gate="G$1" pin="P"/>
 <pinref part="GND12" gate="1" pin="GND"/>
@@
 <pinref part="GND8" gate="1" pin="GND"/>
 <wire x1="127" y1="-2.54" x2="127" y2="-5.08" width="0.1524" layer="91"/>
+</segment>
+<segment>
+<pinref part="K2" gate="2" pin="S"/>
+<wire x1="-6.35" y1="0" x2="-5.08" y2="0" width="0.1524" layer="91"/>
+<wire x1="-5.08" y1="0" x2="-5.08" y2="-5.08" width="0.1524" layer="91"/>
+<pinref part="GND6" gate="1" pin="GND"/>
 </segment>
 </net>
@@
 <wire x1="180.34" y1="26.67" x2="153.67" y2="26.67" width="0.1524" layer="91"/>
 </segment>
+<segment>
+<wire x1="10.16" y1="8.89" x2="10.16" y2="6.35" width="0.1524" layer="91"/>
+<pinref part="D1" gate="G$1" pin="A"/>
+<wire x1="10.16" y1="6.35" x2="10.16" y2="2.54" width="0.1524" layer="91"/>
+<wire x1="1.27" y1="5.08" x2="1.27" y2="6.35" width="0.1524" layer="91"/>
+<wire x1="1.27" y1="6.35" x2="10.16" y2="6.35" width="0.1524" layer="91"/>
+<junction x="10.16" y="6.35"/>
+<pinref part="K2" gate="1" pin="-"/>
+<pinref part="P+7" gate="VCC" pin="VCC"/>
+</segment>
 </net>
 <net name="D4" class="0">
@@
 <segment>
 <pinref part="D1" gate="G$1" pin="C"/>
-<wire x1="10.16" y1="6.35" x2="10.16" y2="10.16" width="0.1524" layer="91"/>
-<junction x="10.16" y="10.16"/>
-<wire x1="10.16" y1="10.16" x2="16.51" y2="10.16" width="0.1524" layer="91"/>
-<wire x1="10.16" y1="10.16" x2="1.27" y2="10.16" width="0.1524" layer="91"/>
-<label x="11.43" y="10.16" size="1.778" layer="95"/>
-<wire x1="1.27" y1="8.89" x2="1.27" y2="10.16" width="0.1524" layer="91"/>
+<wire x1="10.16" y1="-2.54" x2="10.16" y2="-17.78" width="0.1524" layer="91"/>
+<junction x="10.16" y="-17.78"/>
+<wire x1="10.16" y1="-17.78" x2="29.21" y2="-17.78" width="0.1524" layer="91"/>
+<wire x1="10.16" y1="-17.78" x2="1.27" y2="-17.78" width="0.1524" layer="91"/>
+<label x="21.59" y="-17.78" size="1.778" layer="95" rot="MR180"/>
+<wire x1="1.27" y1="-5.08" x2="1.27" y2="-17.78" width="0.1524" layer="91"/>
 <pinref part="K2" gate="1" pin="+"/>
 </segment>
@@
 </segment>
 </net>
-<net name="N$1" class="0">
-<segment>
-<pinref part="K2" gate="3" pin="P"/>
-<pinref part="C2" gate="G$1" pin="2"/>
-<wire x1="-11.43" y1="8.89" x2="-11.43" y2="15.24" width="0.1524" layer="91"/>
-</segment>
-</net>
 <net name="RC5" class="0">
 <segment>
@@
 </segment>
 </net>
+<net name="C2_CON" class="0">
+<segment>
+<pinref part="C2" gate="G$1" pin="2"/>
+<pinref part="K2" gate="2" pin="P"/>
+<wire x1="-11.43" y1="15.24" x2="-11.43" y2="7.62" width="0.1524" layer="91"/>
+</segment>
+</net>

Commit message: ...
Parts:
- removed SW2: DPDT, lc-meter:S-DPDT
- added S1: TL46PO, switch:TL46PO
- added X2: C-GRID-02-70543, con-molex:C-GRID-02-70543
Connections:
- new net M+: S1.P, X2-2.S
- new net M-: S1.P1, X2-1.S
- net /LC: now also S1.S1; no longer SW2.2-3
- net N$2: now also S1.O; no longer SW2.1-2
- net N$7: now also S1.O1, S1.S; no longer SW2.1-3, SW2.2-2

Commit message: ...
Parts:
- added X1: FREQ, con-molex:C-GRID-02-70543
- R5: device resistor:R-EU_0204/2V -> resistor:R-EU_0207/10
- X2: value C-GRID-02-70543 -> L/C
Connections:
- new net FREQ: IC1.RC2/CCP1, X1-2.S
- net GND: now also X1-1.S
Other:
- moved on the sheet: C1, C2, C3, C4, C5, C6, C7, C8, C9, D1, IC1, K2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

Commit message: ...
Parts:
- R1, R10, R3, R4: device resistor:R-EU_0204/2V -> r:R0202/2V
- R5: device resistor:R-EU_0207/10 -> r:R0202/10
Changed lines of the file:
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@@
 <parts>
 <part name="IC1" library="lc-meter" deviceset="PIC16F876A-X/SP" device=""/>
-<part name="R1" library="resistor" deviceset="R-EU_" device="0204/2V" value="100kΩ"/>
+<part name="R1" library="r" deviceset="R" device="0202/2V" value="100kΩ"/>
 <part name="R2" library="resistor" deviceset="R-EU_" device="0204/2V" value="100kΩ"/>
-<part name="R3" library="resistor" deviceset="R-EU_" device="0204/2V" value="100kΩ"/>
-<part name="R4" library="resistor" deviceset="R-EU_" device="0204/2V" value="47kΩ"/>
-<part name="R10" library="resistor" deviceset="R-EU_" device="0204/2V" value="4.7kΩ"/>
+<part name="R3" library="r" deviceset="R" device="0202/2V" value="100kΩ"/>
+<part name="R4" library="r" deviceset="R" device="0202/2V" value="47kΩ"/>
+<part name="R10" library="r" deviceset="R" device="0202/2V" value="4.7kΩ"/>
 <part name="C1" library="rcl" deviceset="C-EU" device="050-025X075" value="1nF"/>
 <part name="C2" library="rcl" deviceset="C-EU" device="050-025X075" value="1nF"/>
@@
 <part name="P+4" library="supply1" deviceset="VCC" device=""/>
 <part name="GND12" library="supply1" deviceset="GND" device=""/>
-<part name="R5" library="resistor" deviceset="R-EU_" device="0207/10" value="4.7kΩ"/>
+<part name="R5" library="r" deviceset="R" device="0202/10" value="4.7kΩ"/>
 <part name="P+5" library="supply1" deviceset="VCC" device=""/>
 <part name="GND14" library="supply1" deviceset="GND" device=""/>
@@
 <pinref part="R1" gate="G$1" pin="1"/>
 <pinref part="R3" gate="G$1" pin="1"/>
-<wire x1="5.08" y1="43.18" x2="5.08" y2="38.1" width="0.1524" layer="91"/>
+<wire x1="10.16" y1="48.26" x2="5.08" y2="38.1" width="0.1524" layer="91"/>
 <junction x="5.08" y="38.1"/>
-<wire x1="5.08" y1="38.1" x2="10.16" y2="38.1" width="0.1524" layer="91"/>
+<wire x1="5.08" y1="38.1" x2="15.24" y2="33.02" width="0.1524" layer="91"/>
 <pinref part="R2" gate="G$1" pin="2"/>
 <wire x1="5.08" y1="27.94" x2="5.08" y2="30.48" width="0.1524" layer="91"/>
@@
 <pinref part="R4" gate="G$1" pin="2"/>
 <pinref part="R1" gate="G$1" pin="2"/>
-<wire x1="25.4" y1="27.94" x2="25.4" y2="38.1" width="0.1524" layer="91"/>
-<wire x1="25.4" y1="38.1" x2="20.32" y2="38.1" width="0.1524" layer="91"/>
+<wire x1="20.32" y1="22.86" x2="25.4" y2="38.1" width="0.1524" layer="91"/>
+<wire x1="25.4" y1="38.1" x2="15.24" y2="43.18" width="0.1524" layer="91"/>
 <pinref part="IC1" gate="A" pin="RA0/AN0"/>
 <wire x1="25.4" y1="38.1" x2="41.91" y2="38.1" width="0.1524" layer="91"/>
@@
 <pinref part="R4" gate="G$1" pin="1"/>
 <pinref part="C4" gate="G$1" pin="+"/>
-<wire x1="25.4" y1="17.78" x2="25.4" y2="15.24" width="0.1524" layer="91"/>
+<wire x1="30.48" y1="22.86" x2="25.4" y2="15.24" width="0.1524" layer="91"/>
 <wire x1="25.4" y1="12.7" x2="25.4" y2="15.24" width="0.1524" layer="91"/>
 <wire x1="25.4" y1="15.24" x2="30.48" y2="15.24" width="0.1524" layer="91"/>
@@
 <pinref part="P+2" gate="VCC" pin="VCC"/>
 <pinref part="R10" gate="G$1" pin="2"/>
-<wire x1="175.26" y1="55.88" x2="175.26" y2="30.48" width="0.1524" layer="91"/>
+<wire x1="175.26" y1="55.88" x2="180.34" y2="25.4" width="0.1524" layer="91"/>
 <label x="149.86" y="20.32" size="1.778" layer="95"/>
 </segment>
@@
 <pinref part="R3" gate="G$1" pin="2"/>
 <pinref part="P+4" gate="VCC" pin="VCC"/>
-<wire x1="5.08" y1="53.34" x2="5.08" y2="55.88" width="0.1524" layer="91"/>
+<wire x1="0" y1="48.26" x2="5.08" y2="55.88" width="0.1524" layer="91"/>
 </segment>
 <segment>
 <pinref part="R5" gate="G$1" pin="2"/>
 <pinref part="P+5" gate="VCC" pin="VCC"/>
-<wire x1="50.8" y1="53.34" x2="50.8" y2="55.88" width="0.1524" layer="91"/>
+<wire x1="55.88" y1="48.26" x2="50.8" y2="55.88" width="0.1524" layer="91"/>
 </segment>
 <segment>
@@
 <pinref part="R5" gate="G$1" pin="1"/>
 <wire x1="60.96" y1="27.94" x2="50.8" y2="27.94" width="0.1524" layer="91"/>
-<wire x1="50.8" y1="27.94" x2="50.8" y2="43.18" width="0.1524" layer="91"/>
+<wire x1="50.8" y1="27.94" x2="45.72" y2="48.26" width="0.1524" layer="91"/>
 </segment>
 </net>
@@
 <segment>
 <pinref part="R10" gate="G$1" pin="1"/>
-<wire x1="175.26" y1="20.32" x2="175.26" y2="7.62" width="0.1524" layer="91"/>
+<wire x1="170.18" y1="25.4" x2="175.26" y2="7.62" width="0.1524" layer="91"/>
 <wire x1="175.26" y1="7.62" x2="163.83" y2="7.62" width="0.1524" layer="91"/>
 <label x="165.1" y="7.62" size="1.778" layer="95"/>
