File: eagle/LCmeter0-LCD-8pinlcd.sch (EAGLE design)
At the start: 27 parts, among them IC1 PIC16F876A-X/SP, K2 DS2Y, Q1 20MHz, Q2 BC548, SW1 SPST, X1 FREQ, X2 L/C

Commit message: ...
Parts:
- C1, C2: device rcl:C-EU050-025X075 -> c:C050-020X036
- C3, C4: device rcl:CPOL-EUE5-4 -> c:CPOLE5-4
- C5, C6: device rcl:C-EU050-024X044 -> c:C025-020X036
- L1: device rcl:L-US0207/10 -> r:R0202/7
- Q2: value BC548 -> BC547CBE; device transistor-npn:BC548 -> t:BC547CBE
- R2: device resistor:R-EU_0204/2V -> r:R0202/2V
- R6: device rcl:R-EU_0207/10 -> r:R0202/5
Other:
- moved on the sheet: C3, C4

Commit message: ...
Parts:
- C5, C6: device c:C025-020X036 -> c:C025-015X024
- Q1: device crystal:CRYSTALHC49U-V -> q:CRYSTALHC49
- S1: value TL46PO -> SL-SW-2P-2T; device switch:TL46PO -> sw:SL-SW-2P-2T
Other:
- moved on the sheet: R2, R6
Changed lines of the file:
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@@
 <part name="C3" library="c" deviceset="CPOL" device="E5-4" value="10μF"/>
 <part name="C4" library="c" deviceset="CPOL" device="E5-4" value="10μF"/>
-<part name="C5" library="c" deviceset="C" device="025-020X036" value="33pF"/>
-<part name="C6" library="c" deviceset="C" device="025-020X036" value="33pF"/>
+<part name="C5" library="c" deviceset="C" device="025-015X024" value="33pF"/>
+<part name="C6" library="c" deviceset="C" device="025-015X024" value="33pF"/>
 <part name="C7" library="rcl" deviceset="CPOL-EU" device="E2.5-6" value="100μF"/>
 <part name="C8" library="rcl" deviceset="CPOL-EU" device="E2.5-5" value="10μF"/>
@@
 <part name="D1" library="diode" deviceset="1N4148" device="DO35-7" value="1N4148"/>
 <part name="L1" library="r" deviceset="R" device="0202/7" value="100μH"/>
-<part name="Q1" library="crystal" deviceset="CRYSTAL" device="HC49U-V" value="20MHz"/>
+<part name="Q1" library="q" deviceset="CRYSTAL" device="HC49" value="20MHz"/>
 <part name="GND11" library="supply1" deviceset="GND" device=""/>
 <part name="P+2" library="supply1" deviceset="VCC" device=""/>
@@
 <part name="LCD1" library="con-lstb" deviceset="MA08-1" device="" value="HD44780"/>
 <part name="P+7" library="supply1" deviceset="VCC" device=""/>
-<part name="S1" library="switch" deviceset="TL46PO" device=""/>
+<part name="S1" library="sw" deviceset="SL-SW-2P-2T" device=""/>
 <part name="X2" library="con-molex" deviceset="C-GRID-02" device="-70543" value="L/C"/>
 <part name="X1" library="con-molex" deviceset="C-GRID-02" device="-70543" value="FREQ"/>
@@
 <instance part="IC1" gate="A" x="88.9" y="22.86"/>
 <instance part="R1" gate="G$1" x="15.24" y="38.1" rot="R270"/>
-<instance part="R2" gate="G$1" x="5.08" y="22.86" rot="R90"/>
+<instance part="R2" gate="G$1" x="5.08" y="22.86"/>
 <instance part="R3" gate="G$1" x="5.08" y="48.26"/>
 <instance part="R4" gate="G$1" x="25.4" y="22.86"/>
@@
 </instance>
 <instance part="GND8" gate="1" x="96.52" y="-25.4" rot="MR0"/>
-<instance part="R6" gate="G$1" x="109.22" y="-15.24" rot="MR0"/>
+<instance part="R6" gate="G$1" x="109.22" y="-15.24" rot="MR270"/>
 <instance part="LCD1" gate="1" x="162.56" y="25.4" rot="MR0"/>
 <instance part="K2" gate="2" x="-10.16" y="10.16" rot="R180"/>
@@
 <attribute name="VALUE" x="15.24" y="13.97" size="1.778" layer="96" align="bottom-center"/>
 </instance>
-<instance part="S1" gate="BEF1" x="-45.72" y="27.94" smashed="yes" rot="R270">
-<attribute name="NAME" x="-46.99" y="34.29" size="1.778" layer="95"/>
+<instance part="S1" gate="G$1" x="-44.45" y="22.86" smashed="yes" rot="R270">
+<attribute name="NAME" x="-45.72" y="29.21" size="1.778" layer="95"/>
 </instance>
 <instance part="X2" gate="-2" x="-63.5" y="27.94" rot="R180"/>
@@
 <wire x1="5.08" y1="38.1" x2="10.16" y2="38.1" width="0.1524" layer="91"/>
 <pinref part="R2" gate="G$1" pin="2"/>
-<wire x1="0" y1="22.86" x2="5.08" y2="30.48" width="0.1524" layer="91"/>
+<wire x1="5.08" y1="27.94" x2="5.08" y2="30.48" width="0.1524" layer="91"/>
 <junction x="5.08" y="30.48"/>
 <pinref part="C3" gate="G$1" pin="+"/>
@@
 <wire x1="-10.16" y1="30.48" x2="-5.08" y2="30.48" width="0.1524" layer="91"/>
 <junction x="-10.16" y="30.48"/>
-<wire x1="-40.64" y1="30.48" x2="-17.78" y2="30.48" width="0.1524" layer="91"/>
+<wire x1="-39.37" y1="30.48" x2="-17.78" y2="30.48" width="0.1524" layer="91"/>
 <junction x="-17.78" y="30.48"/>
 <junction x="-17.78" y="25.4"/>
-<pinref part="S1" gate="BEF1" pin="O"/>
+<pinref part="S1" gate="G$1" pin="O"/>
 </segment>
 </net>
@@
 <pinref part="R2" gate="G$1" pin="1"/>
 <pinref part="GND7" gate="1" pin="GND"/>
-<wire x1="5.08" y1="17.78" x2="10.16" y2="22.86" width="0.1524" layer="91"/>
 </segment>
 <segment>
@@
 <pinref part="L1" gate="G$1" pin="1"/>
 <wire x1="-22.86" y1="25.4" x2="-38.1" y2="25.4" width="0.1524" layer="91"/>
-<wire x1="-40.64" y1="25.4" x2="-38.1" y2="25.4" width="0.1524" layer="91"/>
+<wire x1="-39.37" y1="25.4" x2="-38.1" y2="25.4" width="0.1524" layer="91"/>
 <junction x="-38.1" y="25.4"/>
-<wire x1="-40.64" y1="20.32" x2="-38.1" y2="20.32" width="0.1524" layer="91"/>
-<pinref part="S1" gate="BEF1" pin="S"/>
-<pinref part="S1" gate="BEF1" pin="O1"/>
+<wire x1="-39.37" y1="20.32" x2="-38.1" y2="20.32" width="0.1524" layer="91"/>
+<pinref part="S1" gate="G$1" pin="S"/>
+<pinref part="S1" gate="G$1" pin="O1"/>
 </segment>
 </net>
@@
 <net name="/LC" class="0">
 <segment>
-<wire x1="-40.64" y1="15.24" x2="-35.56" y2="15.24" width="0.1524" layer="91"/>
+<wire x1="-39.37" y1="15.24" x2="-35.56" y2="15.24" width="0.1524" layer="91"/>
 <label x="-40.64" y="15.24" size="1.778" layer="95"/>
-<pinref part="S1" gate="BEF1" pin="S1"/>
+<pinref part="S1" gate="G$1" pin="S1"/>
 <wire x1="-35.56" y1="15.24" x2="-35.56" y2="-33.02" width="0.1524" layer="91"/>
 <wire x1="-35.56" y1="-33.02" x2="119.38" y2="-33.02" width="0.1524" layer="91"/>
@@
 <wire x1="114.3" y1="10.16" x2="127" y2="10.16" width="0.1524" layer="91"/>
 <wire x1="127" y1="10.16" x2="127" y2="-15.24" width="0.1524" layer="91"/>
-<wire x1="127" y1="-15.24" x2="109.22" y2="-20.32" width="0.1524" layer="91"/>
+<wire x1="127" y1="-15.24" x2="114.3" y2="-15.24" width="0.1524" layer="91"/>
 <pinref part="R6" gate="G$1" pin="1"/>
 </segment>
@@
 <segment>
 <pinref part="Q2" gate="G$1" pin="B"/>
-<wire x1="109.22" y1="-10.16" x2="101.6" y2="-15.24" width="0.1524" layer="91"/>
+<wire x1="104.14" y1="-15.24" x2="101.6" y2="-15.24" width="0.1524" layer="91"/>
 <pinref part="R6" gate="G$1" pin="2"/>
 </segment>
@@
 <net name="M+" class="0">
 <segment>
-<wire x1="-60.96" y1="27.94" x2="-50.8" y2="27.94" width="0.1524" layer="91"/>
+<wire x1="-60.96" y1="27.94" x2="-49.53" y2="27.94" width="0.1524" layer="91"/>
 <pinref part="X2" gate="-2" pin="S"/>
-<pinref part="S1" gate="BEF1" pin="P"/>
+<pinref part="S1" gate="G$1" pin="P"/>
 </segment>
 </net>
 <net name="M-" class="0">
 <segment>
-<pinref part="S1" gate="BEF1" pin="P1"/>
+<pinref part="S1" gate="G$1" pin="P1"/>
 <wire x1="-60.96" y1="22.86" x2="-53.34" y2="22.86" width="0.1524" layer="91"/>
 <wire x1="-53.34" y1="22.86" x2="-53.34" y2="17.78" width="0.1524" layer="91"/>
-<wire x1="-53.34" y1="17.78" x2="-50.8" y2="17.78" width="0.1524" layer="91"/>
+<wire x1="-53.34" y1="17.78" x2="-49.53" y2="17.78" width="0.1524" layer="91"/>
 <pinref part="X2" gate="-1" pin="S"/>
 </segment>

Commit message: ...
Parts:
- C7: device rcl:CPOL-EUE2.5-6 -> c:CPOLE5-6
- C8: device rcl:CPOL-EUE2.5-5 -> c:CPOLE5-4
- D1: device diode:1N4148DO35-7 -> d:1N414834-7
- L1: device r:R0202/7 -> r:L02/7
- R2: device r:R0202/2V -> r:R0202/5
Other:
- moved on the sheet: C7, C8
Changed lines of the file:
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@@
 <layer number="98" name="Guide" color="6" fill="1" visible="yes" active="yes"/>
 <layer number="99" name="SpiceOrder" color="5" fill="1" visible="no" active="yes"/>
+<layer number="250" name="trash" color="7" fill="1" visible="yes" active="yes"/>
 </layers>
 <schematic xreflabel="%F%N/%S.%C%R" xrefpart="/%S.%C%R">
@@
 <part name="IC1" library="lc-meter" deviceset="PIC16F876A-X/SP" device=""/>
 <part name="R1" library="r" deviceset="R" device="0202/2V" value="100kΩ"/>
-<part name="R2" library="r" deviceset="R" device="0202/2V" value="100kΩ"/>
+<part name="R2" library="r" deviceset="R" device="0202/5" value="100kΩ"/>
 <part name="R3" library="r" deviceset="R" device="0202/2V" value="100kΩ"/>
 <part name="R4" library="r" deviceset="R" device="0202/2V" value="47kΩ"/>
@@
 <part name="C5" library="c" deviceset="C" device="025-015X024" value="33pF"/>
 <part name="C6" library="c" deviceset="C" device="025-015X024" value="33pF"/>
-<part name="C7" library="rcl" deviceset="CPOL-EU" device="E2.5-6" value="100μF"/>
-<part name="C8" library="rcl" deviceset="CPOL-EU" device="E2.5-5" value="10μF"/>
+<part name="C7" library="c" deviceset="CPOL" device="E5-6" value="100μF"/>
+<part name="C8" library="c" deviceset="CPOL" device="E5-4" value="10μF"/>
 <part name="C9" library="rcl" deviceset="C-EU" device="025-024X044" value="100nF"/>
 <part name="GND2" library="supply1" deviceset="GND" device=""/>
@@
 <part name="GND6" library="supply1" deviceset="GND" device=""/>
 <part name="GND7" library="supply1" deviceset="GND" device=""/>
-<part name="D1" library="diode" deviceset="1N4148" device="DO35-7" value="1N4148"/>
-<part name="L1" library="r" deviceset="R" device="0202/7" value="100μH"/>
+<part name="D1" library="d" deviceset="1N4148" device="34-7" value="1N4148"/>
+<part name="L1" library="r" deviceset="L" device="02/7" value="100μH"/>
 <part name="Q1" library="q" deviceset="CRYSTAL" device="HC49" value="20MHz"/>
 <part name="GND11" library="supply1" deviceset="GND" device=""/>
@@
 <pinref part="C1" gate="G$1" pin="1"/>
 <wire x1="-17.78" y1="22.86" x2="-17.78" y2="25.4" width="0.1524" layer="91"/>
-<wire x1="-33.02" y1="25.4" x2="-17.78" y2="25.4" width="0.1524" layer="91"/>
+<wire x1="-20.32" y1="25.4" x2="-17.78" y2="25.4" width="0.1524" layer="91"/>
 <wire x1="-17.78" y1="25.4" x2="-17.78" y2="30.48" width="0.1524" layer="91"/>
 <pinref part="L1" gate="G$1" pin="2"/>
@@
 <wire x1="144.78" y1="-22.86" x2="144.78" y2="-20.32" width="0.1524" layer="91"/>
 <pinref part="C7" gate="G$1" pin="-"/>
-<wire x1="144.78" y1="-20.32" x2="144.78" y2="-17.78" width="0.1524" layer="91"/>
+<wire x1="144.78" y1="-20.32" x2="144.78" y2="-16.51" width="0.1524" layer="91"/>
 <pinref part="C8" gate="G$1" pin="-"/>
 <wire x1="144.78" y1="-20.32" x2="152.4" y2="-20.32" width="0.1524" layer="91"/>
-<wire x1="152.4" y1="-20.32" x2="152.4" y2="-17.78" width="0.1524" layer="91"/>
+<wire x1="152.4" y1="-20.32" x2="152.4" y2="-16.51" width="0.1524" layer="91"/>
 <pinref part="C9" gate="G$1" pin="2"/>
 <wire x1="152.4" y1="-20.32" x2="160.02" y2="-20.32" width="0.1524" layer="91"/>
@@
 <wire x1="-38.1" y1="25.4" x2="-38.1" y2="20.32" width="0.1524" layer="91"/>
 <pinref part="L1" gate="G$1" pin="1"/>
-<wire x1="-22.86" y1="25.4" x2="-38.1" y2="25.4" width="0.1524" layer="91"/>
+<wire x1="-35.56" y1="25.4" x2="-38.1" y2="25.4" width="0.1524" layer="91"/>
 <wire x1="-39.37" y1="25.4" x2="-38.1" y2="25.4" width="0.1524" layer="91"/>
 <junction x="-38.1" y="25.4"/>
@@
 <segment>
 <pinref part="C7" gate="G$1" pin="+"/>
-<wire x1="144.78" y1="-7.62" x2="144.78" y2="-10.16" width="0.1524" layer="91"/>
+<wire x1="144.78" y1="-7.62" x2="144.78" y2="-8.89" width="0.1524" layer="91"/>
 <pinref part="C8" gate="G$1" pin="+"/>
 <wire x1="144.78" y1="-7.62" x2="152.4" y2="-7.62" width="0.1524" layer="91"/>
-<wire x1="152.4" y1="-7.62" x2="152.4" y2="-10.16" width="0.1524" layer="91"/>
+<wire x1="152.4" y1="-7.62" x2="152.4" y2="-8.89" width="0.1524" layer="91"/>
 <pinref part="C9" gate="G$1" pin="1"/>
 <wire x1="152.4" y1="-7.62" x2="160.02" y2="-7.62" width="0.1524" layer="91"/>
@@
 <wire x1="15.24" y1="10.16" x2="15.24" y2="7.62" width="0.1524" layer="91"/>
 <pinref part="D1" gate="G$1" pin="A"/>
-<wire x1="15.24" y1="7.62" x2="15.24" y2="2.54" width="0.1524" layer="91"/>
+<wire x1="15.24" y1="7.62" x2="17.78" y2="0" width="0.1524" layer="91"/>
 <wire x1="7.62" y1="5.08" x2="7.62" y2="7.62" width="0.1524" layer="91"/>
 <wire x1="7.62" y1="7.62" x2="15.24" y2="7.62" width="0.1524" layer="91"/>
@@
 <label x="95.25" y="-7.62" size="1.778" layer="95" rot="MR0"/>
 <pinref part="D1" gate="G$1" pin="C"/>
-<wire x1="15.24" y1="-2.54" x2="15.24" y2="-7.62" width="0.1524" layer="91"/>
+<wire x1="12.7" y1="0" x2="15.24" y2="-7.62" width="0.1524" layer="91"/>
 <junction x="15.24" y="-7.62"/>
 <wire x1="15.24" y1="-7.62" x2="96.52" y2="-7.62" width="0.1524" layer="91"/>

Commit message: ...
Parts:
- added R7: 10kΩ, r:R0202/5
Connections:
- net /LC: now also R7.2
- net VCC: now also R7.1
Other:
- moved on the sheet: D1

Commit message: ...
Parts:
- removed LCD1: HD44780, con-lstb:MA08-1
- removed Q2: BC547CBE, t:BC547CBE
- added J1: HD44780-4BIT-8PIN, pinconn:HD44780-4BIT-8PIN
- added R8, R9: 100, r:R0202/5
- added T1: BC547CBE-A, t:BC547CBE-A
- added U$1: PIC-ICSP, pinconn:PIC-ICSP
- C5, C6: device c:C025-015X024 -> c:C025-020X036
- C7: device c:CPOLE5-6 -> c:CPOLE2.5-6
- C8: device c:CPOLE5-4 -> c:CPOLE2,5-4
- R2, R6: device r:R0202/5 -> r:R0202/7
- R5: device r:R0202/10 -> r:R0202/7
- R7: device r:R0202/5 -> r:R0202/10
Connections:
- new net N$1: R8.1, U$1.PGC
- new net N$3: R9.1, U$1.PGD
- net /MCLR: now also SW1.P, U$1.MCLR; no longer SW1.S
- net /RELAY: now also T1.C; no longer Q2.C
- net D4: now also J1.D4; no longer LCD1.5
- net D5: now also J1.D5; no longer LCD1.6
- net D6: now also J1.D6, R9.2; no longer LCD1.7
- net D7: now also J1.D7, R8.2; no longer LCD1.8
- net E: now also J1.E; no longer LCD1.4
- net GND: now also J1.GND, SW1.S, T1.E, U$1.VSS; no longer LCD1.1, Q2.E, SW1.P
- net N$5: now also T1.B; no longer Q2.B
- net RS: now also J1.RS; no longer LCD1.3
- net VCC: now also J1.VCC, U$1.VDD; no longer LCD1.2
Other:
- moved on the sheet: C7, C8, SW1

Commit message: ...
Parts:
- added LED1: TLLG4400, led:TLLG4400
- added R11: 1k, r:R0202/5
Connections:
- new net N$4: IC1.RC3/SCK/SCL, R11.1
- new net N$6: LED1.A, R11.2
- net GND: now also LED1.C
Changed lines of the file:
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@@
 <part name="R9" library="r" deviceset="R" device="0202/5" value="100"/>
 <part name="J1" library="pinconn" deviceset="HD44780-4BIT" device="-8PIN"/>
+<part name="R11" library="r" deviceset="R" device="0202/5" value="1k"/>
+<part name="LED1" library="led" deviceset="TLLG4400" device=""/>
+<part name="GND10" library="supply1" deviceset="GND" device=""/>
 </parts>
 <sheets>
@@
 <attribute name="VALUE" x="50.8" y="-5.08" size="1.778" layer="96" align="bottom-center"/>
 </instance>
-<instance part="P+2" gate="VCC" x="175.26" y="58.42" smashed="yes">
-<attribute name="VALUE" x="175.26" y="59.69" size="1.778" layer="96" align="bottom-center"/>
+<instance part="P+2" gate="VCC" x="175.26" y="48.26" smashed="yes">
+<attribute name="VALUE" x="175.26" y="49.53" size="1.778" layer="96" align="bottom-center"/>
 </instance>
 <instance part="P+3" gate="VCC" x="160.02" y="0" smashed="yes">
@@
 <instance part="R9" gate="G$1" x="154.94" y="63.5" rot="R90"/>
 <instance part="J1" gate="G$1" x="154.94" y="25.4"/>
+<instance part="R11" gate="G$1" x="58.42" y="0" rot="MR180"/>
+<instance part="LED1" gate="G$1" x="58.42" y="-13.97"/>
+<instance part="GND10" gate="1" x="58.42" y="-27.94"/>
 </instances>
 <busses>
@@
 <wire x1="175.26" y1="-22.86" x2="175.26" y2="-15.24" width="0.1524" layer="91"/>
 </segment>
+<segment>
+<pinref part="LED1" gate="G$1" pin="C"/>
+<pinref part="GND10" gate="1" pin="GND"/>
+<wire x1="58.42" y1="-17.78" x2="58.42" y2="-25.4" width="0.1524" layer="91"/>
+</segment>
 </net>
 <net name="N$7" class="0">
@@
 <pinref part="P+2" gate="VCC" pin="VCC"/>
 <pinref part="R10" gate="G$1" pin="2"/>
-<wire x1="175.26" y1="55.88" x2="175.26" y2="35.56" width="0.1524" layer="91"/>
+<wire x1="175.26" y1="45.72" x2="175.26" y2="35.56" width="0.1524" layer="91"/>
 <label x="149.86" y="20.32" size="1.778" layer="95"/>
 </segment>
@@
 <pinref part="S1" gate="G$1" pin="S1"/>
 <wire x1="-35.56" y1="15.24" x2="-35.56" y2="-33.02" width="0.1524" layer="91"/>
-<wire x1="-35.56" y1="-33.02" x2="124.46" y2="-33.02" width="0.1524" layer="91"/>
-<wire x1="124.46" y1="-33.02" x2="124.46" y2="2.54" width="0.1524" layer="91"/>
+<wire x1="-35.56" y1="-33.02" x2="121.92" y2="-33.02" width="0.1524" layer="91"/>
+<wire x1="121.92" y1="-33.02" x2="121.92" y2="2.54" width="0.1524" layer="91"/>
 <pinref part="IC1" gate="A" pin="RC4/SDI/SDA"/>
-<wire x1="114.3" y1="7.62" x2="124.46" y2="7.62" width="0.1524" layer="91"/>
-<wire x1="124.46" y1="7.62" x2="124.46" y2="2.54" width="0.1524" layer="91"/>
+<wire x1="114.3" y1="7.62" x2="121.92" y2="7.62" width="0.1524" layer="91"/>
+<wire x1="121.92" y1="7.62" x2="121.92" y2="2.54" width="0.1524" layer="91"/>
 <label x="119.38" y="7.62" size="1.778" layer="95" rot="R180"/>
 <label x="30.48" y="-33.02" size="1.778" layer="95" rot="MR180"/>
 <pinref part="R7" gate="G$1" pin="2"/>
-<wire x1="124.46" y1="2.54" x2="139.7" y2="2.54" width="0.1524" layer="91"/>
-<junction x="124.46" y="2.54"/>
+<wire x1="121.92" y1="2.54" x2="139.7" y2="2.54" width="0.1524" layer="91"/>
+<junction x="121.92" y="2.54"/>
 </segment>
 </net>
@@
 </segment>
 </net>
+<net name="N$4" class="0">
+<segment>
+<pinref part="R11" gate="G$1" pin="1"/>
+<wire x1="58.42" y1="5.08" x2="58.42" y2="7.62" width="0.1524" layer="91"/>
+<pinref part="IC1" gate="A" pin="RC3/SCK/SCL"/>
+<wire x1="58.42" y1="7.62" x2="60.96" y2="7.62" width="0.1524" layer="91"/>
+</segment>
+</net>
+<net name="N$6" class="0">
+<segment>
+<pinref part="R11" gate="G$1" pin="2"/>
+<pinref part="LED1" gate="G$1" pin="A"/>
+<wire x1="58.42" y1="-5.08" x2="58.42" y2="-10.16" width="0.1524" layer="91"/>
+</segment>
+</net>
