File: eagle/LCmeter0-LCD-8pinlcd.brd (EAGLE design)
At the start: 55.9 x 50.5 mm, 25 parts, among them IC1 PIC16F876A-X/SP, K2 DS2Y, Q1 20MHz, Q2 BC548, SW1 SPST, SW2 DPDT

Commit message: ...
Parts:
- C3: device rcl:E2,5-6 -> rcl:E5-4
- C4: device rcl:E5-6 -> rcl:E5-4
- C5, C6: device rcl:C050-025X075 -> rcl:C050-024X044
- LCD1: value (none) -> HD44780
- Q1: device crystal:HC49U70 -> crystal:HC49U-V
- R1, R2, R4: device resistor:0207/10 -> resistor:0204V
- R6: value (none) -> 10kΩ
- moved C7 43.3 mm to (41.9, 12.7), turned to 0 degrees
- moved Q2 30.6 mm to (16.5, 5.08), turned to 90 degrees
- moved R6 24.1 mm to (25.4, 5.08), turned to 180 degrees
- moved D1 13.1 mm to (8.89, 2.54), turned to 180 degrees
- moved C6 7.73 mm to (17.8, 14.0)
- moved LCD1 7.62 mm to (43.2, 34.3)
- moved R4 6.84 mm to (25.4, 39.4)
- moved C8 6.35 mm to (40.6, 19.1)
- moved C9 6.35 mm to (45.7, 19.1)
- moved C5 5.24 mm to (22.9, 14.0)
- moved C3 5.24 mm to (17.8, 38.1), turned to 180 degrees
- moved C4 5.08 mm to (22.9, 33.0)
- moved R10 5.08 mm to (25.4, 44.5)
- moved R5 5.08 mm to (22.9, 44.5)
- moved K2 5.08 mm to (8.89, 14.0)
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Connections:
- removed net N$1: C2.2, K2.13
- removed net VSS: C1.2, C4.-, C5.1, C6.1, C7.-, C8.-, C9.2, D1.A, IC1.19, IC1.8, K2.16, K2.9, LCD1.1, Q2.E, R2.1, SW1.1
- new net C2_CON: C2.2, K2.4
- new net GND: C1.2, C4.-, C5.1, C6.1, C7.-, C8.-, C9.2, IC1.19, IC1.8, K2.8, LCD1.1, Q2.E, R2.1, SW1.1
- net VCC: now also D1.A, K2.16
Routing:
- net VSS: track 161.9 -> 0.00 mm, vias 1 -> 0
- net GND: track 0.00 -> 114.3 mm
- net VCC: track 70.1 -> 115.3 mm
- net A4: track 56.3 -> 16.3 mm
- net /RELAY: track 34.8 -> 7.62 mm
- net N$1: track 19.0 -> 0.00 mm
- net A1: track 24.2 -> 6.58 mm
- net C2_CON: track 0.00 -> 16.9 mm
- net A3: track 29.4 -> 17.8 mm
- net RC5: track 2.54 -> 10.7 mm
- net N$5: track 9.42 -> 2.54 mm
- net /MCLR: track 34.0 -> 27.7 mm
- net A0: track 24.6 -> 22.0 mm
- net RS: track 10.2 -> 7.62 mm
- net E: track 10.2 -> 7.62 mm
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Other:
- board size 55.9 x 50.5 mm -> 48.6 x 49.5 mm
- board text added: "D4"
- board text added: "D5"
- board text added: "D6"
- board text added: "D7"
- board text added: "E"
- board text added: "RS"

Commit message: ...
Parts:
- removed SW2: DPDT, lc-meter:DPDT
- added S1: TL46PO, switch:TL4XPO
- added X2: C-GRID-02-70543, con-molex:70543-02
- moved C4 10.2 mm to (33.0, 33.0)
- moved C5 10.2 mm to (33.0, 14.0)
- moved C7 10.2 mm to (52.1, 12.7)
- moved C9 10.2 mm to (55.9, 19.1)
- moved LCD1 10.2 mm to (53.3, 34.3)
- moved R10 10.2 mm to (35.6, 44.5)
- moved R4 10.2 mm to (35.6, 39.4)
- moved R5 10.2 mm to (33.0, 44.5)
- moved R6 10.2 mm to (35.6, 5.08)
- moved C1 10.2 mm to (22.9, 30.5)
- moved C3 10.2 mm to (27.9, 38.1)
- moved C6 10.2 mm to (27.9, 14.0)
- moved D1 10.2 mm to (19.1, 2.54)
- moved K2 10.2 mm to (19.1, 14.0)
- moved L1 10.2 mm to (19.1, 31.8)
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Connections:
- new net M+: S1.2, X2.2
- new net M-: S1.5, X2.1
- net /LC: now also S1.6; no longer SW2.2-3
- net N$2: now also S1.1; no longer SW2.1-2
- net N$7: now also S1.3, S1.4; no longer SW2.1-3, SW2.2-2
Routing:
- net M+: track 0.00 -> 12.3 mm
- net M-: track 0.00 -> 6.13 mm
- net /MCLR: track 27.7 -> 30.3 mm
- net /LC: track 67.6 -> 69.8 mm
- net GND: track 114.3 -> 112.6 mm
- net N$7: track 14.1 -> 12.6 mm
- net N$2: track 18.5 -> 17.5 mm
Other:
- board size 48.6 x 49.5 mm -> 58.4 x 48.2 mm

Commit message: ...
Parts:
- added X1: FREQ, con-molex:70543-02
- R5: device resistor:0204V -> resistor:0207/10
- X2: value C-GRID-02-70543 -> L/C
- moved R5 3.81 mm to (33.0, 40.6)
- moved C3 2.54 mm to (25.4, 38.1)
- moved C4 2.54 mm to (30.5, 33.0)
- moved R1 2.54 mm to (29.2, 40.6)
- moved R2 2.54 mm to (27.9, 31.8)
- moved R3 2.54 mm to (27.9, 44.5)
Connections:
- new net FREQ: IC1.13, X1.2
- net GND: now also X1.1
Routing:
- net GND: track 112.6 -> 144.3 mm
- net A4: track 16.3 -> 10.2 mm, vias 0 -> 2
- net A1: track 6.58 -> 10.6 mm
- net A0: track 22.0 -> 24.5 mm
- net A3: track 17.8 -> 20.3 mm
- net VCC: track 115.3 -> 116.6 mm
- net N$2: track 17.5 -> 18.1 mm

Commit message: ...
Parts:
- R1, R10, R3, R4: device resistor:0204V -> r:0202/2V
- R5: device resistor:0207/10 -> r:0202/10
- moved X1 5.08 mm to (5.08, 14.0)
- moved L1 4.02 mm to (20.3, 27.9)
- moved S1 2.54 mm to (12.7, 30.5)
- turned R1 to 270 degrees
- turned R10 to 0 degrees
- flipped R3 to the top, turned to 0 degrees
- turned R4 to 0 degrees
- turned R5 to 0 degrees
Routing:
- net M+: track 12.3 -> 21.4 mm, vias 0 -> 2
- net GND: track 144.3 -> 151.1 mm, vias 0 -> 2
- net N$2: track 18.1 -> 15.2 mm
- net /LC: track 69.8 -> 67.2 mm
- net N$7: track 12.6 -> 14.4 mm
- net M-: track 6.13 -> 5.08 mm

Commit message: ...
Parts:
- C1, C2: device rcl:C050-025X075 -> c:C050-020X036
- C3, C4: device rcl:E5-4 -> c:E5-4
- C5, C6: device rcl:C050-024X044 -> c:C025-020X036
- L1: device rcl:0207/10 -> r:0202/7
- Q2: value BC548 -> BC547CBE; device transistor-npn:TO92-EBC -> t:TO92-CBE
- R2: device resistor:0204V -> r:0202/2V
- R6: device rcl:0207/10 -> r:0202/5
- moved C6 8.98 mm to (29.2, 22.9)
- moved R6 7.62 mm to (43.2, 5.08), turned to 90 degrees
- moved C5 5.39 mm to (29.2, 17.8)
- moved Q1 2.54 mm to (33.0, 20.3), turned to 270 degrees
- moved L1 1.27 mm to (20.3, 29.2), turned to 0 degrees
- moved Q2 1.27 mm to (27.9, 5.08)
- turned C1 to 0 degrees
- turned C2 to 0 degrees
- turned R2 to 0 degrees
Routing:
- net GND: track 151.1 -> 127.3 mm
- net OSC1: track 15.9 -> 0.00 mm
- net N$5: track 2.54 -> 12.7 mm
- net OSC2: track 8.89 -> 0.00 mm
- net /LC: track 67.2 -> 70.4 mm
- net RC5: track 10.7 -> 12.7 mm, vias 0 -> 2
- net N$7: track 14.4 -> 13.3 mm

Commit message: ...
Parts:
- C5, C6: device c:C025-020X036 -> c:C025-015X024
- Q1: device crystal:HC49U-V -> q:HC49
- S1: value TL46PO -> SL-SW-2P-2T; device switch:TL4XPO -> sw:SLSW-2P2T
- moved S1 13.5 mm to (3.81, 40.6), turned to 180 degrees
- moved L1 7.41 mm to (14.0, 33.0), turned to 270 degrees
Routing:
- net GND: track 127.3 -> 97.0 mm
- net /LC: track 70.4 -> 45.0 mm
- net M+: track 21.4 -> 0.00 mm, vias 2 -> 0
- net N$7: track 13.3 -> 0.00 mm
- net OSC2: track 0.00 -> 8.67 mm
- net OSC1: track 0.00 -> 7.62 mm
- net N$2: track 15.2 -> 7.62 mm
- net M-: track 5.08 -> 0.00 mm
Changed lines of the file:
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@@
 <element name="C3" library="c" package="E5-4" value="10μF" x="25.4" y="38.1" rot="R180"/>
 <element name="C4" library="c" package="E5-4" value="10μF" x="30.48" y="33.02" rot="R270"/>
-<element name="C5" library="c" package="C025-020X036" value="33pF" x="29.21" y="17.78" rot="R90"/>
-<element name="C6" library="c" package="C025-020X036" value="33pF" x="29.21" y="22.86" rot="R90"/>
+<element name="C5" library="c" package="C025-015X024" value="33pF" x="29.21" y="17.78" rot="R90"/>
+<element name="C6" library="c" package="C025-015X024" value="33pF" x="29.21" y="22.86" rot="R90"/>
 <element name="C7" library="rcl" package="E2,5-6" value="100μF" x="52.07" y="12.7"/>
 <element name="C8" library="rcl" package="E2,5-5" value="10μF" x="50.8" y="19.05" smashed="yes" rot="R270">
@@
 <element name="D1" library="diode" package="DO35-7" value="1N4148" x="19.05" y="2.54" rot="R180"/>
 <element name="IC1" library="lc-meter" package="DIL28-3" value="PIC16F876A-X/SP" x="41.91" y="26.67" rot="R270"/>
-<element name="L1" library="r" package="0202/7" value="100μH" x="20.32" y="29.21"/>
-<element name="Q1" library="crystal" package="HC49U-V" value="20MHz" x="33.02" y="20.32" rot="R270">
-<attribute name="OC_NEWARK" value="unknown" x="33.02" y="20.32" size="1.778" layer="27" rot="R270" display="off"/>
-<attribute name="MPN" value="" x="33.02" y="20.32" size="1.778" layer="27" rot="R270" display="off"/>
-<attribute name="MF" value="" x="33.02" y="20.32" size="1.778" layer="27" rot="R270" display="off"/>
-<attribute name="OC_FARNELL" value="1666969" x="33.02" y="20.32" size="1.778" layer="27" rot="R270" display="off"/>
-</element>
+<element name="L1" library="r" package="0202/7" value="100μH" x="13.97" y="33.02" rot="R270"/>
+<element name="Q1" library="q" package="HC49" value="20MHz" x="33.02" y="20.32" rot="R270"/>
 <element name="R1" library="r" package="0202/2V" value="100kΩ" x="29.21" y="40.64" rot="R270"/>
 <element name="R10" library="r" package="0202/2V" value="4.7kΩ" x="35.56" y="44.45"/>
@@
 <attribute name="OC_FARNELL" value="unknown" x="53.34" y="34.29" size="1.778" layer="27" rot="R90" display="off"/>
 </element>
-<element name="S1" library="switch" package="TL4XPO" value="TL46PO" x="12.7" y="30.48" rot="R270"/>
+<element name="S1" library="sw" package="SLSW-2P2T" value="SL-SW-2P-2T" x="3.81" y="40.64" rot="R180"/>
 <element name="X2" library="con-molex" package="70543-02" value="L/C" x="5.08" y="29.21" rot="R270">
 <attribute name="OC_NEWARK" value="unknown" x="5.08" y="29.21" size="1.778" layer="27" rot="R270" display="off"/>
@@
 <contactref element="C3" pad="-"/>
 <wire x1="22.86" y1="38.1" x2="22.86" y2="33.02" width="0.4064" layer="16"/>
-<wire x1="20.32" y1="33.02" x2="15.24" y2="33.02" width="0.4064" layer="16"/>
 <wire x1="25.4" y1="33.02" x2="22.86" y2="33.02" width="0.4064" layer="16"/>
-<wire x1="22.86" y1="33.02" x2="20.32" y2="33.02" width="0.4064" layer="16"/>
 <contactref element="S1" pad="1"/>
+<wire x1="20.32" y1="25.4" x2="20.32" y2="33.02" width="0" layer="19" extent="1-16"/>
+<wire x1="20.32" y1="25.4" x2="20.32" y2="25.4" width="0" layer="19" extent="1-16"/>
+<wire x1="20.32" y1="33.02" x2="22.86" y2="33.02" width="0" layer="19" extent="16-16"/>
+<wire x1="17.78" y1="33.02" x2="20.32" y2="33.02" width="0" layer="19" extent="16-16"/>
+<wire x1="5.08" y1="38.1" x2="17.78" y2="33.02" width="0" layer="19" extent="1-1"/>
 </signal>
 <signal name="A0">
@@
 <wire x1="55.88" y1="17.78" x2="53.34" y2="15.24" width="0.4064" layer="16"/>
 <wire x1="53.34" y1="15.24" x2="53.34" y2="12.7" width="0.4064" layer="16"/>
-<wire x1="38.1" y1="25.4" x2="33.02" y2="25.4" width="0.4064" layer="16"/>
-<wire x1="33.02" y1="25.4" x2="33.02" y2="30.48" width="0.4064" layer="1"/>
-<wire x1="33.02" y1="30.48" x2="30.48" y2="30.48" width="0.4064" layer="16"/>
 <contactref element="K2" pad="8"/>
 <wire x1="27.94" y1="30.48" x2="22.86" y2="30.48" width="0.4064" layer="16"/>
 <wire x1="22.86" y1="27.94" x2="22.86" y2="30.48" width="0.4064" layer="16"/>
-<wire x1="22.86" y1="30.48" x2="18.0975" y2="30.48" width="0.4064" layer="16"/>
-<wire x1="18.0975" y1="30.48" x2="16.8275" y2="31.75" width="0.4064" layer="16"/>
-<wire x1="16.8275" y1="31.75" x2="13.97" y2="31.75" width="0.4064" layer="16"/>
-<wire x1="12.7" y1="35.56" x2="15.24" y2="40.64" width="0.4064" layer="16"/>
-<wire x1="22.86" y1="27.94" x2="22.86" y2="22.86" width="0.4064" layer="16"/>
+<wire x1="22.86" y1="27.94" x2="22.86" y2="25.4" width="0.4064" layer="16"/>
 <contactref element="X1" pad="1"/>
-<wire x1="13.97" y1="31.75" x2="12.7" y2="33.02" width="0.4064" layer="16"/>
-<wire x1="12.7" y1="33.02" x2="12.7" y2="35.56" width="0.4064" layer="16"/>
-<wire x1="12.7" y1="35.56" x2="2.54" y2="35.56" width="0.4064" layer="16"/>
-<wire x1="2.54" y1="35.56" x2="1.27" y2="34.29" width="0.4064" layer="16"/>
-<wire x1="1.27" y1="34.29" x2="1.27" y2="19.05" width="0.4064" layer="16"/>
+<wire x1="22.86" y1="25.4" x2="22.86" y2="22.86" width="0.4064" layer="16"/>
 <wire x1="1.27" y1="19.05" x2="5.08" y2="15.24" width="0.4064" layer="16"/>
-<via x="33.02" y="25.4" extent="1-16" drill="0.6" shape="square"/>
-<via x="33.02" y="30.48" extent="1-16" drill="0.6" shape="square"/>
-<wire x1="38.1" y1="25.4" x2="45.72" y2="20.32" width="0" layer="19" extent="1-1"/>
-<wire x1="27.94" y1="22.86" x2="22.86" y2="22.86" width="0" layer="19" extent="1-1"/>
+<wire x1="38.1" y1="25.4" x2="40.64" y2="25.4" width="0.4064" layer="16"/>
+<wire x1="40.64" y1="25.4" x2="41.91" y2="24.13" width="0.4064" layer="16"/>
+<wire x1="41.91" y1="24.13" x2="41.91" y2="21.59" width="0.4064" layer="16"/>
+<wire x1="41.91" y1="21.59" x2="43.18" y2="20.32" width="0.4064" layer="16"/>
+<wire x1="43.18" y1="20.32" x2="45.72" y2="20.32" width="0.4064" layer="16"/>
+<wire x1="27.94" y1="22.86" x2="27.94" y2="25.4" width="0.4064" layer="16"/>
+<wire x1="27.94" y1="25.4" x2="22.86" y2="25.4" width="0.4064" layer="1"/>
+<via x="27.94" y="25.4" extent="1-16" drill="0.6" shape="square"/>
+<via x="22.86" y="25.4" extent="1-16" drill="0.6" shape="square"/>
+<wire x1="38.1" y1="25.4" x2="27.94" y2="25.4" width="0.4064" layer="16"/>
+<wire x1="22.86" y1="30.48" x2="15.24" y2="40.64" width="0" layer="19" extent="16-16"/>
+<wire x1="5.08" y1="15.24" x2="22.86" y2="22.86" width="0" layer="19" extent="1-1"/>
 </signal>
 <signal name="N$7">
@@
 <contactref element="S1" pad="3"/>
 <contactref element="S1" pad="4"/>
-<wire x1="20.32" y1="25.4" x2="17.78" y2="25.4" width="0.4064" layer="16"/>
-<wire x1="17.78" y1="25.4" x2="15.24" y2="27.94" width="0.4064" layer="16"/>
-<wire x1="15.24" y1="27.94" x2="10.16" y2="33.02" width="0.4064" layer="1"/>
+<wire x1="2.54" y1="38.1" x2="10.16" y2="33.02" width="0" layer="19" extent="1-1"/>
+<wire x1="5.08" y1="43.18" x2="2.54" y2="38.1" width="0" layer="19" extent="1-1"/>
 </signal>
 <signal name="OSC1">
@@
 <contactref element="Q1" pad="1"/>
 <contactref element="IC1" pad="9"/>
-<wire x1="33.02" y1="22.733" x2="38.1" y2="22.86" width="0" layer="19" extent="1-1"/>
-<wire x1="30.48" y1="22.86" x2="33.02" y2="22.733" width="0" layer="19" extent="1-1"/>
+<wire x1="30.48" y1="22.86" x2="33.02" y2="22.86" width="0.4064" layer="16"/>
+<wire x1="33.02" y1="22.86" x2="38.1" y2="22.86" width="0.4064" layer="16"/>
 </signal>
 <signal name="OSC2">
@@
 <contactref element="Q1" pad="2"/>
 <contactref element="IC1" pad="10"/>
-<wire x1="33.02" y1="17.907" x2="38.1" y2="20.32" width="0" layer="19" extent="1-1"/>
-<wire x1="30.48" y1="17.78" x2="33.02" y2="17.907" width="0" layer="19" extent="1-1"/>
+<wire x1="38.1" y1="20.32" x2="35.56" y2="20.32" width="0.4064" layer="16"/>
+<wire x1="35.56" y1="20.32" x2="33.02" y2="17.78" width="0.4064" layer="16"/>
+<wire x1="33.02" y1="17.78" x2="30.48" y2="17.78" width="0.4064" layer="16"/>
 </signal>
 <signal name="VCC">
@@
 <contactref element="R5" pad="1"/>
 <wire x1="33.02" y1="35.56" x2="35.56" y2="35.56" width="0.4064" layer="16"/>
-<wire x1="35.56" y1="35.56" x2="35.56" y2="30.48" width="0.4064" layer="1"/>
 <wire x1="35.56" y1="30.48" x2="38.1" y2="30.48" width="0.4064" layer="16"/>
 <via x="35.56" y="35.56" extent="1-16" drill="0.6" shape="square"/>
 <via x="35.56" y="30.48" extent="1-16" drill="0.6" shape="square"/>
+<wire x1="35.56" y1="35.56" x2="35.56" y2="30.48" width="0.4064" layer="1"/>
 </signal>
 <signal name="/LC">
@@
 <wire x1="43.18" y1="10.16" x2="45.72" y2="10.16" width="0.4064" layer="16"/>
 <contactref element="S1" pad="6"/>
-<wire x1="10.16" y1="2.54" x2="10.16" y2="27.94" width="0.4064" layer="16"/>
+<wire x1="10.16" y1="2.54" x2="2.54" y2="43.18" width="0" layer="19" extent="16-16"/>
 </signal>
 <signal name="/RELAY">
@@
 <contactref element="S1" pad="5"/>
 <contactref element="X2" pad="1"/>
-<wire x1="5.08" y1="30.48" x2="10.16" y2="30.48" width="0.4064" layer="16"/>
+<wire x1="5.08" y1="30.48" x2="2.54" y2="40.64" width="0" layer="19" extent="1-1"/>
 </signal>
 <signal name="M+">
 <contactref element="X2" pad="2"/>
 <contactref element="S1" pad="2"/>
-<wire x1="5.08" y1="27.94" x2="5.08" y2="22.86" width="0.4064" layer="16"/>
-<wire x1="5.08" y1="22.86" x2="12.7" y2="22.86" width="0.4064" layer="1"/>
-<wire x1="12.7" y1="22.86" x2="12.7" y2="27.94" width="0.4064" layer="16"/>
-<wire x1="12.7" y1="27.94" x2="15.24" y2="30.48" width="0.4064" layer="16"/>
-<via x="5.08" y="22.86" extent="1-16" drill="0.6" shape="square"/>
-<via x="12.7" y="22.86" extent="1-16" drill="0.6" shape="square"/>
+<wire x1="5.08" y1="27.94" x2="5.08" y2="40.64" width="0" layer="19" extent="1-1"/>
 </signal>
 <signal name="FREQ">

Commit message: ...
Parts:
- C7: device rcl:E2,5-6 -> c:E5-6
- C8: device rcl:E2,5-5 -> c:E5-4
- D1: device diode:DO35-7 -> d:DO34-7
- L1: device r:0202/7 -> r:L-02/7
- R2: device r:0202/2V -> r:0202/5
- moved R6 13.0 mm to (30.5, 2.54)
- moved C8 11.7 mm to (53.3, 7.62), turned to 0 degrees
- moved C7 10.2 mm to (53.3, 2.54)
- moved S1 10.2 mm to (3.81, 30.5), turned to 0 degrees
- moved C2 8.03 mm to (17.8, 27.9)
- moved C3 7.62 mm to (25.4, 30.5)
- moved X2 7.62 mm to (5.08, 21.6)
- moved R2 6.35 mm to (33.0, 27.9)
- moved C9 5.08 mm to (50.8, 19.1)
- moved X1 5.08 mm to (5.08, 8.89)
- moved Q2 3.59 mm to (25.4, 2.54), turned to 270 degrees
- moved L1 3.59 mm to (16.5, 35.6), turned to 90 degrees
- moved C1 3.59 mm to (20.3, 27.9)
- moved C4 3.59 mm to (27.9, 35.6), turned to 180 degrees
- moved LCD1 3.59 mm to (55.9, 31.8)
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Routing:
- net GND: track 97.0 -> 194.1 mm
- net FREQ: track 0.00 -> 35.3 mm
- net N$2: track 7.62 -> 40.6 mm
- net M-: track 0.00 -> 22.9 mm
- net /LC: track 45.0 -> 65.0 mm, vias 0 -> 4
- net N$7: track 0.00 -> 18.8 mm
- net M+: track 0.00 -> 17.8 mm
- net RC5: track 12.7 -> 25.4 mm, vias 2 -> 3
- net N$5: track 12.7 -> 2.54 mm
- net /RELAY: track 7.62 -> 5.08 mm
- net RS: track 7.62 -> 10.2 mm
- net OSC1: track 7.62 -> 10.2 mm
- net E: track 7.62 -> 10.2 mm
- net D7: track 7.62 -> 10.2 mm
- net D6: track 8.89 -> 11.4 mm
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Other:
- board size 58.4 x 48.2 mm -> 59.7 x 49.5 mm

Commit message: ...
Parts:
- added R7: 10kΩ, r:0202/5
- moved X1 2.54 mm to (5.08, 11.4)
Connections:
- net /LC: now also R7.2
- net VCC: now also R7.1
Routing:
- net VCC: track 118.6 -> 121.7 mm
- net GND: track 194.1 -> 196.6 mm
- net FREQ: track 35.3 -> 33.7 mm
Changed lines of the file:
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@@
 <attribute name="OC_FARNELL" value="unknown" x="5.08" y="21.59" size="1.778" layer="27" rot="R270" display="off"/>
 </element>
-<element name="X1" library="con-molex" package="70543-02" value="FREQ" x="5.08" y="8.89" rot="R270">
-<attribute name="MPN" value="" x="5.08" y="8.89" size="1.778" layer="27" rot="R270" display="off"/>
-<attribute name="OC_NEWARK" value="unknown" x="5.08" y="8.89" size="1.778" layer="27" rot="R270" display="off"/>
-<attribute name="MF" value="" x="5.08" y="8.89" size="1.778" layer="27" rot="R270" display="off"/>
-<attribute name="OC_FARNELL" value="unknown" x="5.08" y="8.89" size="1.778" layer="27" rot="R270" display="off"/>
+<element name="X1" library="con-molex" package="70543-02" value="FREQ" x="5.08" y="11.43" rot="R270">
+<attribute name="MPN" value="" x="5.08" y="11.43" size="1.778" layer="27" rot="R270" display="off"/>
+<attribute name="OC_NEWARK" value="unknown" x="5.08" y="11.43" size="1.778" layer="27" rot="R270" display="off"/>
+<attribute name="MF" value="" x="5.08" y="11.43" size="1.778" layer="27" rot="R270" display="off"/>
+<attribute name="OC_FARNELL" value="unknown" x="5.08" y="11.43" size="1.778" layer="27" rot="R270" display="off"/>
 </element>
+<element name="R7" library="r" package="0202/5" value="10kΩ" x="12.7" y="10.16"/>
 </elements>
 <signals>
@@
 <wire x1="25.4" y1="22.86" x2="25.4" y2="25.4" width="0.4064" layer="16"/>
 <wire x1="25.4" y1="25.4" x2="33.02" y2="25.4" width="0.4064" layer="16"/>
-<wire x1="5.08" y1="10.16" x2="2.54" y2="10.16" width="0.4064" layer="16"/>
-<wire x1="2.54" y1="10.16" x2="2.54" y2="0" width="0.4064" layer="16"/>
+<wire x1="5.08" y1="12.7" x2="2.54" y2="12.7" width="0.4064" layer="16"/>
+<wire x1="2.54" y1="12.7" x2="2.54" y2="0" width="0.4064" layer="16"/>
 <wire x1="20.32" y1="0" x2="25.4" y2="0" width="0.4064" layer="16"/>
 <wire x1="25.4" y1="0" x2="55.88" y2="0" width="0.4064" layer="16"/>
@@
 <wire x1="43.18" y1="20.32" x2="43.18" y2="43.18" width="0.4064" layer="16"/>
 <wire x1="43.18" y1="43.18" x2="35.56" y2="43.18" width="0.4064" layer="16"/>
+<contactref element="R7" pad="1"/>
+<wire x1="12.7" y1="7.62" x2="12.7" y2="8.128" width="0.4064" layer="16"/>
+<wire x1="12.7" y1="8.128" x2="15.24" y2="8.128" width="0.4064" layer="16"/>
 <wire x1="45.72" y1="20.32" x2="46.355" y2="20.32" width="0" layer="19" extent="1-1"/>
 </signal>
@@
 <via x="30.48" y="11.176" extent="1-16" drill="0.6" shape="square"/>
 <via x="30.48" y="6.604" extent="1-16" drill="0.6" shape="square"/>
-<wire x1="30.48" y1="11.176" x2="10.16" y2="11.176" width="0.4064" layer="16"/>
-<wire x1="10.16" y1="11.176" x2="10.16" y2="13.97" width="0.4064" layer="16"/>
-<wire x1="10.16" y1="13.97" x2="10.16" y2="27.94" width="0.4064" layer="1"/>
+<wire x1="30.48" y1="11.176" x2="12.7" y2="11.176" width="0.4064" layer="16"/>
+<wire x1="12.7" y1="12.7" x2="10.16" y2="12.7" width="0.4064" layer="16"/>
+<wire x1="10.16" y1="12.7" x2="10.16" y2="27.94" width="0.4064" layer="1"/>
 <wire x1="10.16" y1="27.94" x2="5.08" y2="27.94" width="0.4064" layer="16"/>
-<via x="10.16" y="13.97" extent="1-16" drill="0.6" shape="square"/>
+<via x="10.16" y="12.7" extent="1-16" drill="0.6" shape="square"/>
 <via x="10.16" y="27.94" extent="1-16" drill="0.6" shape="square"/>
+<contactref element="R7" pad="2"/>
+<wire x1="12.7" y1="11.176" x2="12.7" y2="12.7" width="0.4064" layer="16"/>
 </signal>
 <signal name="/RELAY">
@@
 <wire x1="38.1" y1="10.16" x2="32.258" y2="10.16" width="0.4064" layer="16"/>
 <wire x1="32.258" y1="10.16" x2="31.75" y2="9.652" width="0.4064" layer="16"/>
-<wire x1="5.08" y1="7.62" x2="10.16" y2="7.62" width="0.4064" layer="16"/>
-<wire x1="10.16" y1="7.62" x2="10.16" y2="9.652" width="0.4064" layer="16"/>
-<wire x1="10.16" y1="9.652" x2="31.75" y2="9.652" width="0.4064" layer="16"/>
+<wire x1="5.08" y1="10.16" x2="5.08" y2="9.652" width="0.4064" layer="16"/>
+<wire x1="5.08" y1="9.652" x2="31.75" y2="9.652" width="0.4064" layer="16"/>
 </signal>
 </signals>
