File: eagle/LCmeter0-LCD-8pinlcd-alt2.brd (EAGLE design)
At the start: 58.4 x 50.8 mm, 34 parts, among them IC1 PIC16F876A-X/SP, J1 HD44780-4BIT-8PIN, J2 PIC-UART, J3 PIC-ICSP, K2 DS2Y, Q1 20MHz, SW1 SPST, T1 BC547CBE-A, X1 FREQ, X2 L/C

Commit message: ...
Routing:
- net A3: vias 4 -> 2
Changed lines of the file:
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@@
 <wire x1="27.94" y1="43.18" x2="25.4" y2="43.18" width="0.4064" layer="16"/>
 <wire x1="25.4" y1="38.1" x2="27.94" y2="38.1" width="0.4064" layer="16"/>
-<via x="33.02" y="30.48" extent="1-16" drill="0.6" shape="square"/>
-<wire x1="33.02" y1="30.48" x2="27.94" y2="30.48" width="0.4064" layer="1"/>
-<via x="27.94" y="30.48" extent="1-16" drill="0.6" shape="square"/>
-<wire x1="27.94" y1="30.48" x2="25.4" y2="30.48" width="0.4064" layer="16"/>
+<wire x1="27.94" y1="25.4" x2="25.4" y2="25.4" width="0.4064" layer="16"/>
 <via x="25.4" y="38.1" extent="1-16" drill="0.6" shape="square"/>
-<wire x1="25.4" y1="38.1" x2="25.4" y2="30.48" width="0.4064" layer="1"/>
-<via x="25.4" y="30.48" extent="1-16" drill="0.6" shape="square"/>
+<wire x1="25.4" y1="38.1" x2="25.4" y2="25.4" width="0.4064" layer="1"/>
+<via x="25.4" y="25.4" extent="1-16" drill="0.6" shape="square"/>
 <wire x1="25.4" y1="43.18" x2="25.4" y2="38.1" width="0.4064" layer="16"/>
 <wire x1="25.4" y1="38.1" x2="25.4" y2="40.64" width="0.4064" layer="16"/>
@@
 <wire x1="12.7" y1="15.24" x2="12.7" y2="27.94" width="0.4064" layer="16"/>
 <via x="12.7" y="27.94" extent="1-16" drill="0.6" shape="square"/>
-<wire x1="12.7" y1="27.94" x2="25.4" y2="27.94" width="0.4064" layer="1"/>
-<via x="25.4" y="27.94" extent="1-16" drill="0.6" shape="square"/>
-<wire x1="25.4" y1="27.94" x2="27.94" y2="27.94" width="0.4064" layer="16"/>
+<wire x1="12.7" y1="27.94" x2="22.86" y2="27.94" width="0.4064" layer="1"/>
+<via x="22.86" y="27.94" extent="1-16" drill="0.6" shape="square"/>
+<wire x1="22.86" y1="27.94" x2="27.94" y2="27.94" width="0.4064" layer="16"/>
 <wire x1="45.72" y1="20.32" x2="43.18" y2="20.32" width="0.4064" layer="16"/>
 <wire x1="43.18" y1="20.32" x2="43.18" y2="43.18" width="0.4064" layer="16"/>

Commit message: ...
Parts:
- removed SW1: SPST, lc-meter:PB-5
- added U$1: PB-1P-1T, sw:PB-1P1T
- L1: device r:L-02/7 -> r:L-09R
- moved L1 6.35 mm to (10.2, 43.2), turned to 0 degrees
- moved C1 2.54 mm to (15.2, 35.6)
- moved C2 2.54 mm to (12.7, 35.6)
- moved C3 2.54 mm to (21.6, 38.1), flipped to the top, turned to 0 degrees
- moved C4 2.54 mm to (21.6, 33.0)
- moved X2 2.54 mm to (5.08, 19.1)
- turned R10 to 270 degrees
Connections:
- net /MCLR: now also R10.2, U$1.2; no longer R10.1, SW1.1
- net GND: now also U$1.1; no longer SW1.3
- net N$2: now also L1.P$2; no longer L1.2
- net N$7: now also L1.P$1; no longer L1.1
- net VCC: now also R10.1; no longer R10.2
Routing:
- net N$2: track 22.9 -> 35.6 mm
- net /MCLR: track 40.6 -> 27.9 mm
- net GND: track 195.6 -> 190.5 mm
- net M-: track 17.8 -> 20.3 mm
- net C2_CON: track 33.0 -> 30.5 mm
- net A3: track 47.0 -> 44.5 mm
- net N$7: track 13.8 -> 16.3 mm
- net M+: track 17.8 -> 20.3 mm
