File: eagle/LCmeter0-LCD-8pinlcd-alt2.brd (EAGLE design)
At the start: 34 parts, among them IC1 PIC16F876A-X/SP, J1 HD44780-4BIT-8PIN, J2 PIC-UART, J3 PIC-ICSP, K2 DS2Y, Q1 20MHz, T1 BC547CBE-A, X1 FREQ, X2 L/C

Commit message: ...
Parts:
- L1: device r:L-09R -> r:L-8R
Changed lines of the file:
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@@
         <element name="D1" library="d" package="DO34-7" value="1N4148" x="19.05" y="2.54" rot="R180" />
         <element name="IC1" library="mcu" package="DIL28-3" value="PIC16F876A-X/SP" x="41.91" y="24.13" rot="R270" />
-        <element name="L1" library="r" package="L-09R" value="100μH" x="10.16" y="43.18" />
+        <element name="L1" library="r" package="L-8R" value="100μH" x="10.16" y="43.18" />
         <element name="Q1" library="q" package="HC49" value="20MHz" x="33.02" y="17.78" rot="R270" />
         <element name="R1" library="r" package="0202/7" value="100kΩ" x="31.75" y="38.1" rot="R270" />

Commit message: ...
Parts:
- R11: value 1k -> 1kΩ
- R8, R9: value 100 -> 100Ω
Changed lines of the file:
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@@
         <element name="R7" library="r" package="0202/10" value="10kΩ" x="10.16" y="10.16" />
         <element name="J3" library="pinconn" package="CONN-5P" value="PIC-ICSP" x="35.56" y="48.26" />
-        <element name="R8" library="r" package="0202/5" value="100" x="48.26" y="45.72" rot="R270" />
-        <element name="R9" library="r" package="0202/5" value="100" x="48.26" y="40.64" rot="R180" />
+        <element name="R8" library="r" package="0202/5" value="100Ω" x="48.26" y="45.72" rot="R270" />
+        <element name="R9" library="r" package="0202/5" value="100Ω" x="48.26" y="40.64" rot="R180" />
         <element name="J1" library="pinconn" package="CONN-8P" value="HD44780-4BIT-8PIN" x="53.34" y="22.86" rot="R90" />
-        <element name="R11" library="r" package="0202/5" value="1k" x="35.56" y="10.16" />
+        <element name="R11" library="r" package="0202/5" value="1kΩ" x="35.56" y="10.16" />
         <element name="LED1" library="led" package="LED3MM" value="TLLG4400" x="27.94" y="13.97" smashed="yes" rot="R90">
           <attribute name="MF" value="VISHAY SEMICONDUCTOR" x="27.94" y="13.97" size="0.8128" layer="27" rot="R90" display="off" />
