File: eagle/LCmeter0-LCD-8pinlcd-PIC-COMP.brd (EAGLE design)
At the start: 58.4 x 50.8 mm, 34 parts, among them IC1 PIC16F876A-X/SP, J1 HD44780-4BIT-8PIN, J2 PIC-UART, J3 PIC-ICSP, K2 DS2Y, Q1 20MHz, T1 BC547CBE-A, X1 FREQ, X2 L/C

Commit message: ...
Other:
- board size 58.4 x 50.8 mm -> 61 x 53.3 mm
Changed lines of the file:
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@@
 <board>
 <plain>
-<wire x1="-1.27" y1="-1.27" x2="57.15" y2="-1.27" width="0" layer="20"/>
-<wire x1="57.15" y1="-1.27" x2="57.15" y2="49.53" width="0" layer="20"/>
-<wire x1="57.15" y1="49.53" x2="-1.27" y2="49.53" width="0" layer="20"/>
-<wire x1="-1.27" y1="49.53" x2="-1.27" y2="-1.27" width="0" layer="20"/>
+<wire x1="-2.54" y1="-2.54" x2="58.42" y2="-2.54" width="0" layer="20"/>
+<wire x1="58.42" y1="-2.54" x2="58.42" y2="50.8" width="0" layer="20"/>
+<wire x1="58.42" y1="50.8" x2="-2.54" y2="50.8" width="0" layer="20"/>
+<wire x1="-2.54" y1="50.8" x2="-2.54" y2="-2.54" width="0" layer="20"/>
 <text x="55.88" y="40.64" size="0.8128" layer="21" rot="R90" align="center">D7</text>
 <text x="55.88" y="38.1" size="0.8128" layer="21" rot="R90" align="center">D6</text>
@@
 <text x="55.88" y="30.48" size="0.8128" layer="21" rot="R90" align="center">E</text>
 <text x="55.88" y="27.94" size="0.8128" layer="21" rot="R90" align="center">RS</text>
-<text x="-2.54" y="0" size="1.27" layer="20" align="center-right">1</text>
-<text x="-2.54" y="2.54" size="1.27" layer="20" align="center-right">2</text>
-<text x="-2.54" y="5.08" size="1.27" layer="20" align="center-right">3</text>
-<text x="-2.54" y="7.62" size="1.27" layer="20" align="center-right">4</text>
-<text x="-2.54" y="10.16" size="1.27" layer="20" align="center-right">5</text>
-<text x="-2.54" y="12.7" size="1.27" layer="20" align="center-right">6</text>
-<text x="-2.54" y="15.24" size="1.27" layer="20" align="center-right">7</text>
-<text x="-2.54" y="17.78" size="1.27" layer="20" align="center-right">8</text>
-<text x="-2.54" y="20.32" size="1.27" layer="20" align="center-right">9</text>
-<text x="-2.54" y="22.86" size="1.27" layer="20" align="center-right">10</text>
-<text x="-2.54" y="25.4" size="1.27" layer="20" align="center-right">11</text>
-<text x="-2.54" y="27.94" size="1.27" layer="20" align="center-right">12</text>
-<text x="-2.54" y="30.48" size="1.27" layer="20" align="center-right">13</text>
-<text x="-2.54" y="33.02" size="1.27" layer="20" align="center-right">14</text>
-<text x="-2.54" y="35.56" size="1.27" layer="20" align="center-right">15</text>
-<text x="-2.54" y="38.1" size="1.27" layer="20" align="center-right">16</text>
-<text x="-2.54" y="40.64" size="1.27" layer="20" align="center-right">17</text>
-<text x="-2.54" y="43.18" size="1.27" layer="20" align="center-right">18</text>
-<text x="-2.54" y="45.72" size="1.27" layer="20" align="center-right">19</text>
-<text x="-2.54" y="48.26" size="1.27" layer="20" align="center-right">20</text>
-<text x="0" y="-2.54" size="1.27" layer="20" align="top-center">1</text>
-<text x="2.54" y="-2.54" size="1.27" layer="20" align="top-center">2</text>
-<text x="5.08" y="-2.54" size="1.27" layer="20" align="top-center">3</text>
-<text x="7.62" y="-2.54" size="1.27" layer="20" align="top-center">4</text>
-<text x="10.16" y="-2.54" size="1.27" layer="20" align="top-center">5</text>
-<text x="12.7" y="-2.54" size="1.27" layer="20" align="top-center">6</text>
-<text x="15.24" y="-2.54" size="1.27" layer="20" align="top-center">7</text>
-<text x="17.78" y="-2.54" size="1.27" layer="20" align="top-center">8</text>
-<text x="20.32" y="-2.54" size="1.27" layer="20" align="top-center">9</text>
-<text x="22.86" y="-2.54" size="1.27" layer="20" align="top-center">10</text>
-<text x="25.4" y="-2.54" size="1.27" layer="20" align="top-center">11</text>
-<text x="27.94" y="-2.54" size="1.27" layer="20" align="top-center">12</text>
-<text x="30.48" y="-2.54" size="1.27" layer="20" align="top-center">13</text>
-<text x="33.02" y="-2.54" size="1.27" layer="20" align="top-center">14</text>
-<text x="35.56" y="-2.54" size="1.27" layer="20" align="top-center">15</text>
-<text x="38.1" y="-2.54" size="1.27" layer="20" align="top-center">16</text>
-<text x="40.64" y="-2.54" size="1.27" layer="20" align="top-center">17</text>
-<text x="43.18" y="-2.54" size="1.27" layer="20" align="top-center">18</text>
-<text x="45.72" y="-2.54" size="1.27" layer="20" align="top-center">19</text>
-<text x="48.26" y="-2.54" size="1.27" layer="20" align="top-center">20</text>
-<text x="50.8" y="-2.54" size="1.27" layer="20" align="top-center">21</text>
-<text x="53.34" y="-2.54" size="1.27" layer="20" align="top-center">22</text>
-<text x="55.88" y="-2.54" size="1.27" layer="20" align="top-center">23</text>
+<text x="-3.81" y="-2.54" size="1.27" layer="20" align="center-right">1</text>
+<text x="-3.81" y="0" size="1.27" layer="20" align="center-right">2</text>
+<text x="-3.81" y="2.54" size="1.27" layer="20" align="center-right">3</text>
+<text x="-3.81" y="5.08" size="1.27" layer="20" align="center-right">4</text>
+<text x="-3.81" y="7.62" size="1.27" layer="20" align="center-right">5</text>
+<text x="-3.81" y="10.16" size="1.27" layer="20" align="center-right">6</text>
+<text x="-3.81" y="12.7" size="1.27" layer="20" align="center-right">7</text>
+<text x="-3.81" y="15.24" size="1.27" layer="20" align="center-right">8</text>
+<text x="-3.81" y="17.78" size="1.27" layer="20" align="center-right">9</text>
+<text x="-3.81" y="20.32" size="1.27" layer="20" align="center-right">10</text>
+<text x="-3.81" y="22.86" size="1.27" layer="20" align="center-right">11</text>
+<text x="-3.81" y="25.4" size="1.27" layer="20" align="center-right">12</text>
+<text x="-3.81" y="27.94" size="1.27" layer="20" align="center-right">13</text>
+<text x="-3.81" y="30.48" size="1.27" layer="20" align="center-right">14</text>
+<text x="-3.81" y="33.02" size="1.27" layer="20" align="center-right">15</text>
+<text x="-3.81" y="35.56" size="1.27" layer="20" align="center-right">16</text>
+<text x="-3.81" y="38.1" size="1.27" layer="20" align="center-right">17</text>
+<text x="-3.81" y="40.64" size="1.27" layer="20" align="center-right">18</text>
+<text x="-3.81" y="43.18" size="1.27" layer="20" align="center-right">19</text>
+<text x="-3.81" y="45.72" size="1.27" layer="20" align="center-right">20</text>
+<text x="0" y="-3.81" size="1.27" layer="20" align="top-center">1</text>
+<text x="2.54" y="-3.81" size="1.27" layer="20" align="top-center">2</text>
+<text x="5.08" y="-3.81" size="1.27" layer="20" align="top-center">3</text>
+<text x="7.62" y="-3.81" size="1.27" layer="20" align="top-center">4</text>
+<text x="10.16" y="-3.81" size="1.27" layer="20" align="top-center">5</text>
+<text x="12.7" y="-3.81" size="1.27" layer="20" align="top-center">6</text>
+<text x="15.24" y="-3.81" size="1.27" layer="20" align="top-center">7</text>
+<text x="17.78" y="-3.81" size="1.27" layer="20" align="top-center">8</text>
+<text x="20.32" y="-3.81" size="1.27" layer="20" align="top-center">9</text>
+<text x="22.86" y="-3.81" size="1.27" layer="20" align="top-center">10</text>
+<text x="25.4" y="-3.81" size="1.27" layer="20" align="top-center">11</text>
+<text x="27.94" y="-3.81" size="1.27" layer="20" align="top-center">12</text>
+<text x="30.48" y="-3.81" size="1.27" layer="20" align="top-center">13</text>
+<text x="33.02" y="-3.81" size="1.27" layer="20" align="top-center">14</text>
+<text x="35.56" y="-3.81" size="1.27" layer="20" align="top-center">15</text>
+<text x="38.1" y="-3.81" size="1.27" layer="20" align="top-center">16</text>
+<text x="40.64" y="-3.81" size="1.27" layer="20" align="top-center">17</text>
+<text x="43.18" y="-3.81" size="1.27" layer="20" align="top-center">18</text>
+<text x="45.72" y="-3.81" size="1.27" layer="20" align="top-center">19</text>
+<text x="48.26" y="-3.81" size="1.27" layer="20" align="top-center">20</text>
+<text x="50.8" y="-3.81" size="1.27" layer="20" align="top-center">21</text>
+<text x="53.34" y="-3.81" size="1.27" layer="20" align="top-center">22</text>
+<text x="55.88" y="-3.81" size="1.27" layer="20" align="top-center">23</text>
 <hole x="0" y="48.26" drill="1.5"/>
 <hole x="55.88" y="48.26" drill="1.5"/>
@@
 <wire x1="5.08" y1="35.56" x2="5.08" y2="43.18" width="0.6096" layer="16"/>
 <wire x1="5.08" y1="43.18" x2="7.62" y2="43.18" width="0.6096" layer="16"/>
-<wire x1="5.08" y1="35.56" x2="3.81" y2="34.29" width="0.4064" layer="16"/>
-<wire x1="3.81" y1="34.29" x2="3.81" y2="31.75" width="0.4064" layer="16"/>
-<wire x1="3.81" y1="31.75" x2="2.54" y2="30.48" width="0.4064" layer="16"/>
+<wire x1="5.08" y1="35.56" x2="3.81" y2="34.29" width="0.254" layer="16"/>
+<wire x1="3.81" y1="34.29" x2="3.81" y2="31.75" width="0.254" layer="16"/>
+<wire x1="3.81" y1="31.75" x2="2.54" y2="30.48" width="0.254" layer="16"/>
 </signal>
 <signal name="OSC1">

Commit message: ...
Parts:
- L1: value 100μH -> 68μH
Changed lines of the file:
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@@
 <element name="D1" library="d" package="DO34-7" value="1N4148" x="19.05" y="2.54" rot="R180"/>
 <element name="IC1" library="lc-meter" package="DIL28-3" value="PIC16F876A-X/SP" x="41.91" y="24.13" rot="R270"/>
-<element name="L1" library="r" package="L-09R" value="100μH" x="10.16" y="43.18"/>
+<element name="L1" library="r" package="L-09R" value="68μH" x="10.16" y="43.18"/>
 <element name="Q1" library="q" package="HC49" value="20MHz" x="33.02" y="17.78" rot="R270"/>
 <element name="R1" library="r" package="0202/7" value="100kΩ" x="31.75" y="38.1" rot="R270"/>

Commit message: ...
Parts:
- J4: value (none) -> J4
- R6: value 10kΩ -> 10k
- U$2: value PIC16F876A-X/SP -> PIC16F876A-X/SP-COMP-B-A
- moved R6 14.5 mm to (34.3, 2.54), turned to 90 degrees
- renumbered IC1 to U$2, JP1 to J4
Connections:
- net RC5 renamed N$8
- net RX renamed N$9
Routing:
- net N$8: track 2.54 -> 20.3 mm, vias 1 -> 0
- net N$6: track 20.3 -> 2.54 mm
- net N$5: track 2.54 -> 3.81 mm

Commit message: ...
Parts:
- removed X1: FREQ, con-molex:70543-02
- removed X2: L/C, con-molex:70543-02
- added J5, J7: CONN-2P-2P, pinconn:CONN-2P
- J4: device pinhead:1X02 -> pinconn:CONN-2P
- moved R6 14.5 mm to (48.3, 6.35), turned to 180 degrees
- moved J2 1.80 mm to (53.3, 12.7)
- moved J4 1.27 mm to (50.8, 2.54)
Connections:
- new net N$11: U$2.21, U$2.22
- net FREQ: now also J5.2, U$2.11; no longer X1.2
- net GND: now also J4.1, J5.1; no longer J4.2, X1.1
- net M+: now also J7.2; no longer X2.2
- net M-: now also J7.1; no longer X2.1
- net VCC: now also J4.2; no longer J4.1
Routing:
- net N$8: track 20.3 -> 2.54 mm
- net N$6: track 2.54 -> 20.3 mm
- net FREQ: track 35.6 -> 45.7 mm
- net N$11: track 0.00 -> 5.08 mm
- net GND: track 190.5 -> 185.4 mm
- net N$5: track 3.81 -> 2.54 mm

Commit message: ...
Parts:
- C1, C2: device c:C050-020X036 -> c:C050-025X060
- C3, C4: device c:E2,5-4 -> c:E2,5-5
- turned C1 to 90 degrees
- turned C2 to 90 degrees
- turned C4 to 180 degrees
- turned J2 to 270 degrees
Routing:
- net A3: track 44.5 -> 47.0 mm
- net N$2: track 35.6 -> 38.1 mm
- net VCC: vias 9 -> 8
Changed lines of the file:
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@@
 <layer number="27" name="tValues" color="7" fill="1" visible="yes" active="yes"/>
 <layer number="28" name="bValues" color="7" fill="1" visible="yes" active="yes"/>
-<layer number="29" name="tStop" color="7" fill="3" visible="yes" active="yes"/>
-<layer number="30" name="bStop" color="7" fill="6" visible="yes" active="yes"/>
-<layer number="31" name="tCream" color="7" fill="4" visible="yes" active="yes"/>
-<layer number="32" name="bCream" color="7" fill="5" visible="yes" active="yes"/>
-<layer number="33" name="tFinish" color="6" fill="3" visible="yes" active="yes"/>
-<layer number="34" name="bFinish" color="6" fill="6" visible="yes" active="yes"/>
-<layer number="35" name="tGlue" color="7" fill="4" visible="yes" active="yes"/>
-<layer number="36" name="bGlue" color="7" fill="5" visible="yes" active="yes"/>
-<layer number="37" name="tTest" color="7" fill="1" visible="yes" active="yes"/>
-<layer number="38" name="bTest" color="7" fill="1" visible="yes" active="yes"/>
-<layer number="39" name="tKeepout" color="4" fill="11" visible="yes" active="yes"/>
-<layer number="40" name="bKeepout" color="1" fill="11" visible="yes" active="yes"/>
-<layer number="41" name="tRestrict" color="4" fill="10" visible="yes" active="yes"/>
-<layer number="42" name="bRestrict" color="1" fill="10" visible="yes" active="yes"/>
-<layer number="43" name="vRestrict" color="2" fill="10" visible="yes" active="yes"/>
-<layer number="44" name="Drills" color="7" fill="1" visible="yes" active="yes"/>
-<layer number="45" name="Holes" color="7" fill="1" visible="yes" active="yes"/>
+<layer number="29" name="tStop" color="7" fill="3" visible="no" active="yes"/>
+<layer number="30" name="bStop" color="7" fill="6" visible="no" active="yes"/>
+<layer number="31" name="tCream" color="7" fill="4" visible="no" active="yes"/>
+<layer number="32" name="bCream" color="7" fill="5" visible="no" active="yes"/>
+<layer number="33" name="tFinish" color="6" fill="3" visible="no" active="yes"/>
+<layer number="34" name="bFinish" color="6" fill="6" visible="no" active="yes"/>
+<layer number="35" name="tGlue" color="7" fill="4" visible="no" active="yes"/>
+<layer number="36" name="bGlue" color="7" fill="5" visible="no" active="yes"/>
+<layer number="37" name="tTest" color="7" fill="1" visible="no" active="yes"/>
+<layer number="38" name="bTest" color="7" fill="1" visible="no" active="yes"/>
+<layer number="39" name="tKeepout" color="4" fill="11" visible="no" active="yes"/>
+<layer number="40" name="bKeepout" color="1" fill="11" visible="no" active="yes"/>
+<layer number="41" name="tRestrict" color="4" fill="10" visible="no" active="yes"/>
+<layer number="42" name="bRestrict" color="1" fill="10" visible="no" active="yes"/>
+<layer number="43" name="vRestrict" color="2" fill="10" visible="no" active="yes"/>
+<layer number="44" name="Drills" color="7" fill="1" visible="no" active="yes"/>
+<layer number="45" name="Holes" color="7" fill="1" visible="no" active="yes"/>
 <layer number="46" name="Milling" color="3" fill="1" visible="yes" active="yes"/>
 <layer number="47" name="Measures" color="7" fill="1" visible="yes" active="yes"/>
@@
 <layer number="98" name="Guide" color="6" fill="1" visible="no" active="no"/>
 <layer number="99" name="SpiceOrder" color="5" fill="1" visible="no" active="no"/>
-<layer number="250" name="trash" color="7" fill="1" visible="yes" active="yes"/>
+<layer number="250" name="trash" color="7" fill="1" visible="no" active="yes"/>
 </layers>
 <board>
@@
 </autorouter>
 <elements>
-<element name="C1" library="c" package="C050-020X036" value="1nF" x="15.24" y="35.56"/>
-<element name="C2" library="c" package="C050-020X036" value="1nF" x="12.7" y="35.56"/>
-<element name="C3" library="c" package="E2,5-4" value="10μF" x="21.59" y="38.1"/>
-<element name="C4" library="c" package="E2,5-4" value="10μF" x="21.59" y="33.02"/>
+<element name="C1" library="c" package="C050-025X060" value="1nF" x="15.24" y="35.56" rot="R90"/>
+<element name="C2" library="c" package="C050-025X060" value="1nF" x="12.7" y="35.56" rot="R90"/>
+<element name="C3" library="c" package="E2,5-5" value="10μF" x="21.59" y="38.1" smashed="yes">
+<attribute name="NAME" x="21.59" y="41.148" size="1.27" layer="25" align="bottom-center"/>
+<attribute name="VALUE" x="24.003" y="35.687" size="1.27" layer="27"/>
+</element>
+<element name="C4" library="c" package="E2,5-5" value="10μF" x="21.59" y="33.02" smashed="yes" rot="R180">
+<attribute name="NAME" x="21.59" y="29.972" size="1.27" layer="25" align="top-center"/>
+<attribute name="VALUE" x="24.003" y="30.607" size="1.27" layer="27"/>
+</element>
 <element name="C5" library="c" package="C025-020X036" value="33pF" x="26.67" y="17.78" rot="R90"/>
 <element name="C6" library="c" package="C025-020X036" value="33pF" x="26.67" y="20.32" rot="R90"/>
 <element name="C7" library="c" package="E2,5-6" value="100μF" x="52.07" y="7.62" rot="R180"/>
 <element name="C9" library="rcl" package="C025-024X044" value="100nF" x="50.8" y="19.05" smashed="yes" rot="R270">
-<attribute name="NAME" x="49.53" y="16.51" size="1.27" layer="25" ratio="10" rot="R270"/>
-<attribute name="VALUE" x="48.133" y="20.828" size="1.27" layer="27" ratio="10" rot="R270"/>
+<attribute name="NAME" x="49.784" y="21.844" size="1.016" layer="25" ratio="10" rot="R90" align="top-left"/>
+<attribute name="VALUE" x="48.641" y="17.526" size="0.8128" layer="27" ratio="10" rot="R270" align="bottom-right"/>
 </element>
 <element name="D1" library="d" package="DO34-7" value="1N4148" x="19.05" y="2.54" rot="R180"/>
@@
 </element>
 <element name="J4" library="pinconn" package="CONN-2P" value="J4" x="50.8" y="2.54" rot="R180"/>
-<element name="J2" library="pinconn" package="PIC-UART" value="PIC-UART" x="53.34" y="12.7" rot="R90"/>
+<element name="J2" library="pinconn" package="PIC-UART" value="PIC-UART" x="53.34" y="12.7" rot="R270"/>
 <element name="U$1" library="sw" package="PB-1P1T" value="PB-1P-1T" x="22.86" y="45.72" rot="R180"/>
 <element name="U$2" library="lc-meter" package="DIL28-3" value="PIC16F876A-X/SP-COMP-B-A" x="41.91" y="24.13" rot="R270"/>
@@
 <via x="25.4" y="25.4" extent="1-16" drill="0.6" shape="square"/>
 <wire x1="25.4" y1="43.18" x2="25.4" y2="38.1" width="0.6096" layer="16"/>
-<wire x1="25.4" y1="38.1" x2="22.86" y2="38.1" width="0.6096" layer="16"/>
+<wire x1="25.4" y1="38.1" x2="20.32" y2="38.1" width="0.6096" layer="16"/>
 <contactref element="U$2" pad="5"/>
 </signal>
@@
 <contactref element="C3" pad="-"/>
 <contactref element="S1" pad="1"/>
-<wire x1="15.24" y1="38.1" x2="20.32" y2="38.1" width="0.6096" layer="16"/>
+<wire x1="15.24" y1="38.1" x2="22.86" y2="38.1" width="0.6096" layer="16"/>
 <wire x1="2.54" y1="35.56" x2="2.54" y2="45.72" width="0.6096" layer="16"/>
 <wire x1="2.54" y1="45.72" x2="12.7" y2="45.72" width="0.6096" layer="16"/>
@@
 <wire x1="10.16" y1="5.08" x2="12.7" y2="5.08" width="0.6096" layer="16"/>
 <wire x1="12.7" y1="5.08" x2="15.24" y2="5.08" width="0.6096" layer="16"/>
-<via x="50.8" y="20.32" extent="1-16" drill="0.6" shape="square"/>
 <via x="55.88" y="20.32" extent="1-16" drill="0.5"/>
 <via x="55.88" y="7.62" extent="1-16" drill="0.6" shape="square"/>

Commit message: ...
Parts:
- added D2: 1N4148-12, d:DO34-12
Connections:
- new net N$12: C7.+, D2.A, J4.2
- net VCC: now also D2.C; no longer C7.+, J4.2
Routing:
- net VCC: track 147.3 -> 127.0 mm, vias 8 -> 6
- net N$12: track 0.00 -> 7.62 mm
Changed lines of the file:
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@@
 <element name="J7" library="pinconn" package="CONN-2P" value="CONN-2P-2P" x="5.08" y="17.78" rot="R270"/>
 <element name="J5" library="pinconn" package="CONN-2P" value="CONN-2P-2P" x="5.08" y="5.08" rot="R270"/>
+<element name="D2" library="d" package="DO34-12" value="1N4148-12" x="55.88" y="13.97" rot="R270"/>
 </elements>
 <signals>
@@
 <contactref element="C6" pad="1"/>
 <contactref element="C4" pad="-"/>
-<contactref element="C7" pad="-"/>
-<contactref element="C9" pad="2"/>
 <contactref element="T1" pad="E"/>
 <wire x1="48.26" y1="22.86" x2="48.26" y2="17.78" width="0.6096" layer="1"/>
-<wire x1="53.34" y1="17.78" x2="50.8" y2="17.78" width="0.6096" layer="16"/>
 <wire x1="48.26" y1="17.78" x2="45.72" y2="17.78" width="0.6096" layer="16"/>
 <wire x1="25.4" y1="17.78" x2="25.4" y2="20.32" width="0.6096" layer="16"/>
@@
 <contactref element="J2" pad="19"/>
 <wire x1="53.34" y1="17.78" x2="55.88" y2="17.78" width="0.6096" layer="16"/>
-<wire x1="50.8" y1="7.62" x2="50.8" y2="10.16" width="0.6096" layer="16"/>
 <wire x1="50.8" y1="10.16" x2="55.88" y2="10.16" width="0.6096" layer="16"/>
 <wire x1="55.88" y1="10.16" x2="55.88" y2="17.78" width="0.6096" layer="16"/>
@@
 <wire x1="22.86" y1="22.86" x2="25.4" y2="22.86" width="0.6096" layer="16"/>
 <wire x1="48.26" y1="22.86" x2="53.34" y2="22.86" width="0.6096" layer="16"/>
-<wire x1="50.8" y1="17.78" x2="48.26" y2="17.78" width="0.6096" layer="16"/>
 <wire x1="22.86" y1="22.86" x2="20.32" y2="22.86" width="0.6096" layer="16"/>
 <wire x1="20.32" y1="22.86" x2="20.32" y2="33.02" width="0.6096" layer="16"/>
@@
 <wire x1="5.08" y1="0" x2="5.08" y2="5.08" width="0.6096" layer="16"/>
 <contactref element="J4" pad="1"/>
-<wire x1="50.8" y1="7.62" x2="50.8" y2="0" width="0.6096" layer="16"/>
-<wire x1="50.8" y1="0" x2="50.8" y2="2.54" width="0" layer="19" extent="16-16"/>
+<contactref element="C7" pad="-"/>
+<wire x1="50.8" y1="2.54" x2="50.8" y2="10.16" width="0.4064" layer="16"/>
+<contactref element="C9" pad="2"/>
+<wire x1="53.34" y1="17.78" x2="50.8" y2="17.78" width="0.6096" layer="16"/>
+<wire x1="50.8" y1="17.78" x2="48.26" y2="17.78" width="0.6096" layer="16"/>
+<wire x1="50.8" y1="10.16" x2="50.8" y2="7.62" width="0" layer="19" extent="16-16"/>
+<wire x1="50.8" y1="0" x2="50.8" y2="2.54" width="0.6096" layer="16"/>
 </signal>
 <signal name="N$7">
@@
 <contactref element="R3" pad="2"/>
 <contactref element="R5" pad="2"/>
-<contactref element="C9" pad="1"/>
-<contactref element="C7" pad="+"/>
 <contactref element="K2" pad="16"/>
 <contactref element="D1" pad="A"/>
 <wire x1="15.24" y1="2.54" x2="15.24" y2="5.08" width="0.6096" layer="16"/>
-<wire x1="55.88" y1="7.62" x2="55.88" y2="20.32" width="0.6096" layer="1"/>
-<wire x1="45.72" y1="20.32" x2="50.8" y2="20.32" width="0.6096" layer="16"/>
 <wire x1="55.88" y1="20.32" x2="55.88" y2="25.4" width="0.6096" layer="16"/>
 <contactref element="R7" pad="1"/>
 <wire x1="10.16" y1="5.08" x2="12.7" y2="5.08" width="0.6096" layer="16"/>
 <wire x1="12.7" y1="5.08" x2="15.24" y2="5.08" width="0.6096" layer="16"/>
-<via x="55.88" y="20.32" extent="1-16" drill="0.5"/>
-<via x="55.88" y="7.62" extent="1-16" drill="0.6" shape="square"/>
 <via x="12.7" y="15.24" extent="1-16" drill="0.6" shape="square"/>
 <wire x1="12.7" y1="15.24" x2="12.7" y2="5.08" width="0.6096" layer="1"/>
@@
 <wire x1="55.88" y1="25.4" x2="53.34" y2="25.4" width="0.6096" layer="16"/>
 <contactref element="J1" pad="2"/>
-<wire x1="55.88" y1="7.62" x2="53.34" y2="7.62" width="0.6096" layer="16"/>
 <contactref element="J2" pad="20"/>
 <wire x1="53.34" y1="20.32" x2="55.88" y2="20.32" width="0.6096" layer="16"/>
@@
 <wire x1="43.18" y1="43.18" x2="38.1" y2="43.18" width="0.6096" layer="1"/>
 <via x="38.1" y="43.18" extent="1-16" drill="0.6" shape="square"/>
-<wire x1="53.34" y1="20.32" x2="50.8" y2="20.32" width="0.6096" layer="16"/>
 <contactref element="R10" pad="1"/>
 <wire x1="27.94" y1="40.64" x2="30.48" y2="40.64" width="0.6096" layer="16"/>
 <contactref element="U$2" pad="20"/>
-<contactref element="J4" pad="2"/>
-<wire x1="53.34" y1="7.62" x2="53.34" y2="2.54" width="0.6096" layer="16"/>
+<contactref element="D2" pad="C"/>
+<wire x1="45.72" y1="20.32" x2="53.34" y2="20.32" width="0.6096" layer="16"/>
+<contactref element="C9" pad="1"/>
+<wire x1="53.34" y1="20.32" x2="50.8" y2="20.32" width="0" layer="19" extent="1-1"/>
 </signal>
 <signal name="D4">
@@
 <wire x1="45.72" y1="25.4" x2="48.26" y2="25.4" width="0.6096" layer="16"/>
 </signal>
+<signal name="N$12">
+<contactref element="J4" pad="2"/>
+<contactref element="C7" pad="+"/>
+<contactref element="D2" pad="A"/>
+<wire x1="55.88" y1="7.62" x2="53.34" y2="7.62" width="0.6096" layer="16"/>
+<wire x1="53.34" y1="7.62" x2="53.34" y2="2.54" width="0.6096" layer="16"/>
+</signal>
 </signals>
