File: eagle/LCmeter0-LCD-8pinlcd-PIC-COMP.brd (EAGLE design)
At the start: 61 x 53.3 mm, 35 parts, among them J1 HD44780-4BIT-8PIN, J2 PIC-UART, J3 PIC-ICSP, J4 J4, J5 CONN-2P-2P, J7 CONN-2P-2P, K2 DS2Y, Q1 20MHz, T1 BC547CBE-A

Commit message: ...
Parts:
- added C8: 22pF, c:C050-020X036
- C7: device c:E2,5-6 -> c:E2,5-5
- R8: device r:0202/5 -> r:0202/7
- moved R9 8.03 mm to (55.9, 43.2)
- moved R8 3.81 mm to (48.3, 41.9), turned to 180 degrees
Connections:
- net N$1 renamed PGC
- removed net N$3: J3.5, R9.1
- new net PGD: C8.2, J3.5, R9.1
- net D6: now also R8.2; no longer R9.2
- net D7: now also R9.2; no longer R8.2
- net GND: now also C8.1
Routing:
- net GND: track 185.4 -> 208.3 mm, vias 4 -> 6
- net PGD: track 0.00 -> 12.7 mm
- net N$3: track 7.62 -> 0.00 mm
- net PGC: track 5.08 -> 7.62 mm
- net D7: track 12.7 -> 10.2 mm
- net D6: track 10.2 -> 7.62 mm
Changed lines of the file:
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@@
 <element name="C5" library="c" package="C025-020X036" value="33pF" x="26.67" y="17.78" rot="R90"/>
 <element name="C6" library="c" package="C025-020X036" value="33pF" x="26.67" y="20.32" rot="R90"/>
-<element name="C7" library="c" package="E2,5-6" value="100μF" x="52.07" y="7.62" rot="R180"/>
+<element name="C7" library="c" package="E2,5-5" value="100μF" x="52.07" y="7.62" rot="R180"/>
 <element name="C9" library="rcl" package="C025-024X044" value="100nF" x="50.8" y="19.05" smashed="yes" rot="R270">
 <attribute name="NAME" x="49.784" y="21.844" size="1.016" layer="25" ratio="10" rot="R90" align="top-left"/>
@@
 <element name="R7" library="r" package="0202/10" value="10kΩ" x="10.16" y="10.16"/>
 <element name="J3" library="pinconn" package="CONN-5P" value="PIC-ICSP" x="35.56" y="48.26"/>
-<element name="R8" library="r" package="0202/5" value="100" x="48.26" y="45.72" rot="R270"/>
-<element name="R9" library="r" package="0202/5" value="100" x="48.26" y="40.64" rot="R180"/>
+<element name="R8" library="r" package="0202/7" value="100" x="48.26" y="41.91" rot="R180"/>
+<element name="R9" library="r" package="0202/5" value="100" x="55.88" y="43.18" rot="R180"/>
 <element name="J1" library="pinconn" package="CONN-8P" value="HD44780-4BIT-8PIN" x="53.34" y="22.86" rot="R90"/>
 <element name="LED1" library="led" package="LED3MM" value="TLLG4400" x="27.94" y="13.97" smashed="yes" rot="R90">
@@
 <element name="J5" library="pinconn" package="CONN-2P" value="CONN-2P-2P" x="5.08" y="5.08" rot="R270"/>
 <element name="D2" library="d" package="DO34-12" value="1N4148-12" x="55.88" y="13.97" rot="R270"/>
+<element name="C8" library="c" package="C050-020X036" value="22pF" x="53.34" y="45.72" rot="R180"/>
 </elements>
 <signals>
@@
 <via x="48.26" y="17.78" extent="1-16" drill="0.6" shape="square"/>
 <wire x1="22.86" y1="22.86" x2="25.4" y2="22.86" width="0.6096" layer="16"/>
-<wire x1="48.26" y1="22.86" x2="53.34" y2="22.86" width="0.6096" layer="16"/>
+<wire x1="48.26" y1="22.86" x2="50.8" y2="22.86" width="0.6096" layer="16"/>
+<wire x1="50.8" y1="22.86" x2="53.34" y2="22.86" width="0.6096" layer="16"/>
 <wire x1="22.86" y1="22.86" x2="20.32" y2="22.86" width="0.6096" layer="16"/>
 <wire x1="20.32" y1="22.86" x2="20.32" y2="33.02" width="0.6096" layer="16"/>
@@
 <wire x1="53.34" y1="17.78" x2="50.8" y2="17.78" width="0.6096" layer="16"/>
 <wire x1="50.8" y1="17.78" x2="48.26" y2="17.78" width="0.6096" layer="16"/>
-<wire x1="50.8" y1="10.16" x2="50.8" y2="7.62" width="0" layer="19" extent="16-16"/>
 <wire x1="50.8" y1="0" x2="50.8" y2="2.54" width="0.6096" layer="16"/>
+<contactref element="C8" pad="1"/>
+<via x="50.8" y="43.18" extent="1-16" drill="0.6" shape="square"/>
+<wire x1="50.8" y1="43.18" x2="50.8" y2="22.86" width="0.6096" layer="1"/>
+<via x="50.8" y="22.86" extent="1-16" drill="0.6" shape="square"/>
+<wire x1="50.8" y1="7.62" x2="50.8" y2="10.16" width="0" layer="19" extent="16-16"/>
+<wire x1="53.34" y1="43.18" x2="50.8" y2="43.18" width="0.6096" layer="16"/>
 </signal>
 <signal name="N$7">
@@
 </signal>
 <signal name="D6">
+<contactref element="J1" pad="7"/>
+<wire x1="53.34" y1="38.1" x2="48.26" y2="38.1" width="0.6096" layer="16"/>
+<contactref element="U$2" pad="27"/>
+<contactref element="R8" pad="2"/>
 <wire x1="45.72" y1="38.1" x2="48.26" y2="38.1" width="0.6096" layer="16"/>
+</signal>
+<signal name="D7">
+<contactref element="J1" pad="8"/>
+<wire x1="55.88" y1="40.64" x2="53.34" y2="40.64" width="0.6096" layer="16"/>
+<wire x1="53.34" y1="40.64" x2="45.72" y2="40.64" width="0.6096" layer="16"/>
+<contactref element="U$2" pad="28"/>
 <contactref element="R9" pad="2"/>
-<contactref element="J1" pad="7"/>
-<wire x1="53.34" y1="38.1" x2="45.72" y2="38.1" width="0.6096" layer="16"/>
-<contactref element="U$2" pad="27"/>
-</signal>
-<signal name="D7">
-<contactref element="R8" pad="2"/>
-<wire x1="50.8" y1="45.72" x2="50.8" y2="40.64" width="0.6096" layer="16"/>
-<contactref element="J1" pad="8"/>
-<wire x1="53.34" y1="40.64" x2="50.8" y2="40.64" width="0.6096" layer="16"/>
-<wire x1="50.8" y1="40.64" x2="45.72" y2="40.64" width="0.6096" layer="16"/>
-<contactref element="U$2" pad="28"/>
 </signal>
 <signal name="C2_CON">
@@
 <wire x1="5.08" y1="7.62" x2="33.02" y2="7.62" width="0.6096" layer="16"/>
 </signal>
-<signal name="N$1">
+<signal name="PGC">
 <contactref element="J3" pad="4"/>
 <contactref element="R8" pad="1"/>
 <wire x1="43.18" y1="48.26" x2="43.18" y2="45.72" width="0.6096" layer="16"/>
-<wire x1="43.18" y1="45.72" x2="45.72" y2="45.72" width="0.6096" layer="16"/>
-</signal>
-<signal name="N$3">
+<wire x1="43.18" y1="45.72" x2="48.26" y2="45.72" width="0.6096" layer="16"/>
+</signal>
+<signal name="PGD">
 <contactref element="R9" pad="1"/>
 <contactref element="J3" pad="5"/>
-<wire x1="45.72" y1="48.26" x2="48.26" y2="48.26" width="0.6096" layer="16"/>
-<wire x1="48.26" y1="48.26" x2="48.26" y2="43.18" width="0.6096" layer="16"/>
+<wire x1="45.72" y1="48.26" x2="53.34" y2="48.26" width="0.6096" layer="16"/>
+<contactref element="C8" pad="2"/>
+<wire x1="53.34" y1="48.26" x2="53.34" y2="45.72" width="0.6096" layer="16"/>
+<wire x1="53.34" y1="45.72" x2="55.88" y2="45.72" width="0.6096" layer="16"/>
 </signal>
 <signal name="N$5">

Commit message: ...
Parts:
- C3, C4: device c:E2,5-5 -> c:E2,5-4
- turned C4 to 0 degrees
- turned D1 to 0 degrees
Connections:
- net /RELAY: now also D1.A; no longer D1.C
- net VCC: now also D1.C; no longer D1.A
Routing:
- net A3: track 47.0 -> 44.5 mm
- net N$2: track 38.1 -> 35.6 mm
Changed lines of the file:
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@@
 <element name="C1" library="c" package="C050-025X060" value="1nF" x="15.24" y="35.56" rot="R90"/>
 <element name="C2" library="c" package="C050-025X060" value="1nF" x="12.7" y="35.56" rot="R90"/>
-<element name="C3" library="c" package="E2,5-5" value="10μF" x="21.59" y="38.1" smashed="yes">
-<attribute name="NAME" x="21.59" y="41.148" size="1.27" layer="25" align="bottom-center"/>
-<attribute name="VALUE" x="24.003" y="35.687" size="1.27" layer="27"/>
-</element>
-<element name="C4" library="c" package="E2,5-5" value="10μF" x="21.59" y="33.02" smashed="yes" rot="R180">
-<attribute name="NAME" x="21.59" y="29.972" size="1.27" layer="25" align="top-center"/>
-<attribute name="VALUE" x="24.003" y="30.607" size="1.27" layer="27"/>
+<element name="C3" library="c" package="E2,5-4" value="10μF" x="21.59" y="38.1" smashed="yes">
+<attribute name="NAME" x="20.066" y="40.132" size="1.016" layer="25" align="bottom-center"/>
+<attribute name="VALUE" x="22.86" y="35.56" size="0.8128" layer="27"/>
+</element>
+<element name="C4" library="c" package="E2,5-4" value="10μF" x="21.59" y="33.02" smashed="yes">
+<attribute name="NAME" x="20.066" y="35.052" size="1.016" layer="25" rot="R180" align="top-center"/>
+<attribute name="VALUE" x="22.86" y="30.48" size="0.8128" layer="27"/>
 </element>
 <element name="C5" library="c" package="C025-020X036" value="33pF" x="26.67" y="17.78" rot="R90"/>
 <element name="C6" library="c" package="C025-020X036" value="33pF" x="26.67" y="20.32" rot="R90"/>
-<element name="C7" library="c" package="E2,5-5" value="100μF" x="52.07" y="7.62" rot="R180"/>
+<element name="C7" library="c" package="E2,5-5" value="100μF" x="52.07" y="7.62" smashed="yes" rot="R180">
+<attribute name="NAME" x="50.673" y="10.16" size="0.8128" layer="25" align="bottom-right"/>
+<attribute name="VALUE" x="54.229" y="5.969" size="0.8128" layer="27" align="top-left"/>
+</element>
 <element name="C9" library="rcl" package="C025-024X044" value="100nF" x="50.8" y="19.05" smashed="yes" rot="R270">
-<attribute name="NAME" x="49.784" y="21.844" size="1.016" layer="25" ratio="10" rot="R90" align="top-left"/>
+<attribute name="NAME" x="50.038" y="16.51" size="1.016" layer="25" ratio="10" rot="R270" align="top-left"/>
 <attribute name="VALUE" x="48.641" y="17.526" size="0.8128" layer="27" ratio="10" rot="R270" align="bottom-right"/>
 </element>
-<element name="D1" library="d" package="DO34-7" value="1N4148" x="19.05" y="2.54" rot="R180"/>
+<element name="D1" library="d" package="DO34-7" value="1N4148" x="19.05" y="2.54"/>
 <element name="L1" library="r" package="L-09R" value="68μH" x="10.16" y="43.18"/>
 <element name="Q1" library="q" package="HC49" value="20MHz" x="33.02" y="17.78" rot="R270"/>
@@
 <attribute name="OC_FARNELL" value="1612435" x="27.94" y="13.97" size="0.8128" layer="27" rot="R90" display="off"/>
 <attribute name="NAME" x="27.94" y="11.557" size="0.8128" layer="25" ratio="10" rot="R180" align="bottom-center"/>
-<attribute name="VALUE" x="27.94" y="10.541" size="0.8128" layer="27" ratio="10" rot="R180" align="bottom-center"/>
 </element>
 <element name="J4" library="pinconn" package="CONN-2P" value="J4" x="50.8" y="2.54" rot="R180"/>
@@
 <element name="J7" library="pinconn" package="CONN-2P" value="CONN-2P-2P" x="5.08" y="17.78" rot="R270"/>
 <element name="J5" library="pinconn" package="CONN-2P" value="CONN-2P-2P" x="5.08" y="5.08" rot="R270"/>
-<element name="D2" library="d" package="DO34-12" value="1N4148-12" x="55.88" y="13.97" rot="R270"/>
+<element name="D2" library="d" package="DO34-12" value="1N4148-12" x="55.88" y="13.97" smashed="yes" rot="R270">
+<attribute name="NAME" x="57.023" y="13.843" size="0.8128" layer="25" ratio="10" rot="R90" align="top-center"/>
+</element>
 <element name="C8" library="c" package="C050-020X036" value="22pF" x="53.34" y="45.72" rot="R180"/>
 </elements>
@@
 <via x="25.4" y="25.4" extent="1-16" drill="0.6" shape="square"/>
 <wire x1="25.4" y1="43.18" x2="25.4" y2="38.1" width="0.6096" layer="16"/>
-<wire x1="25.4" y1="38.1" x2="20.32" y2="38.1" width="0.6096" layer="16"/>
+<wire x1="25.4" y1="38.1" x2="22.86" y2="38.1" width="0.6096" layer="16"/>
 <contactref element="U$2" pad="5"/>
 </signal>
@@
 <contactref element="C3" pad="-"/>
 <contactref element="S1" pad="1"/>
-<wire x1="15.24" y1="38.1" x2="22.86" y2="38.1" width="0.6096" layer="16"/>
+<wire x1="15.24" y1="38.1" x2="20.32" y2="38.1" width="0.6096" layer="16"/>
 <wire x1="2.54" y1="35.56" x2="2.54" y2="45.72" width="0.6096" layer="16"/>
 <wire x1="2.54" y1="45.72" x2="12.7" y2="45.72" width="0.6096" layer="16"/>
@@
 <contactref element="J4" pad="1"/>
 <contactref element="C7" pad="-"/>
-<wire x1="50.8" y1="2.54" x2="50.8" y2="10.16" width="0.4064" layer="16"/>
+<wire x1="50.8" y1="2.54" x2="50.8" y2="7.62" width="0.6096" layer="16"/>
 <contactref element="C9" pad="2"/>
 <wire x1="53.34" y1="17.78" x2="50.8" y2="17.78" width="0.6096" layer="16"/>
@@
 <wire x1="50.8" y1="43.18" x2="50.8" y2="22.86" width="0.6096" layer="1"/>
 <via x="50.8" y="22.86" extent="1-16" drill="0.6" shape="square"/>
-<wire x1="50.8" y1="7.62" x2="50.8" y2="10.16" width="0" layer="19" extent="16-16"/>
 <wire x1="53.34" y1="43.18" x2="50.8" y2="43.18" width="0.6096" layer="16"/>
+<wire x1="50.8" y1="10.16" x2="50.8" y2="7.62" width="0.6096" layer="16"/>
 </signal>
 <signal name="N$7">
@@
 <contactref element="R5" pad="2"/>
 <contactref element="K2" pad="16"/>
-<contactref element="D1" pad="A"/>
-<wire x1="15.24" y1="2.54" x2="15.24" y2="5.08" width="0.6096" layer="16"/>
 <wire x1="55.88" y1="20.32" x2="55.88" y2="25.4" width="0.6096" layer="16"/>
 <contactref element="R7" pad="1"/>
@@
 <contactref element="U$2" pad="20"/>
 <contactref element="D2" pad="C"/>
-<wire x1="45.72" y1="20.32" x2="53.34" y2="20.32" width="0.6096" layer="16"/>
+<wire x1="45.72" y1="20.32" x2="50.8" y2="20.32" width="0.6096" layer="16"/>
 <contactref element="C9" pad="1"/>
-<wire x1="53.34" y1="20.32" x2="50.8" y2="20.32" width="0" layer="19" extent="1-1"/>
+<contactref element="D1" pad="C"/>
+<wire x1="15.24" y1="2.54" x2="15.24" y2="5.08" width="0.6096" layer="16"/>
+<wire x1="50.8" y1="20.32" x2="53.34" y2="20.32" width="0.6096" layer="16"/>
 </signal>
 <signal name="D4">
@@
 </signal>
 <signal name="/RELAY">
-<contactref element="D1" pad="C"/>
 <contactref element="K2" pad="1"/>
 <contactref element="T1" pad="C"/>
 <wire x1="22.86" y1="5.08" x2="25.4" y2="5.08" width="0.6096" layer="16"/>
-<wire x1="22.86" y1="2.54" x2="22.86" y2="5.08" width="0.6096" layer="16"/>
+<contactref element="D1" pad="A"/>
+<wire x1="22.86" y1="5.08" x2="22.86" y2="2.54" width="0.6096" layer="16"/>
 </signal>
 <signal name="/MCLR">
