File: eagle/LCmeter0-LCD-8pinlcd-PIC-COMP.sch (EAGLE design)
At the start: 34 parts, among them IC1 PIC16F876A-X/SP-COMP-B-A, J1 HD44780-4BIT-8PIN, J2 PIC-UART, J3 PIC-ICSP, K2 DS2Y, Q1 20MHz, T1 BC547CBE-A, X1 FREQ, X2 L/C

Commit message: ...
Parts:
- J4: value (none) -> J4
- R6: value 10kΩ -> 10k
- renumbered IC1 to U$2
Connections:
- net /RELAIS renamed N$8
- net RX renamed N$9
- net TX renamed N$10
- removed net LED: LED1.A, U$2.RC3
- removed net N$6 (its old number): LED1.C, R11.1
- new net N$4: LED1.A, R11.2
- new net N$5: R11.1, U$2.RC3
- net GND: now also LED1.C; no longer R11.2
Other:
- moved on the sheet: LED1, R11, R6

Commit message: ...
Parts:
- removed X1: FREQ, con-molex:C-GRID-02-70543
- removed X2: L/C, con-molex:C-GRID-02-70543
- added J5, J7: CONN-2P-2P, pinconn:CONN-2P-2P
- J4: device pinhead:PINHD-1X2 -> pinconn:CONN-2P-2P
Connections:
- new net N$11: U$2.RB0, U$2.RB1
- net FREQ: now also J5.2, U$2.RC0; no longer X1-2.S
- net GND: now also J4.1, J5.1; no longer J4.2, X1-1.S
- net M+: now also J7.2; no longer X2-2.S
- net M-: now also J7.1; no longer X2-1.S
- net VCC: now also J4.2; no longer J4.1
Changed lines of the file:
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@@
 </variantdefs>
 <classes>
-<class number="0" name="default" width="0" drill="0">
+<class number="0" name="default" width="0.6096" drill="0">
 </class>
 </classes>
@@
 <part name="P+7" library="supply1" deviceset="VCC" device=""/>
 <part name="S1" library="sw" deviceset="SL-SW-2P-2T" device=""/>
-<part name="X2" library="con-molex" deviceset="C-GRID-02" device="-70543" value="L/C"/>
-<part name="X1" library="con-molex" deviceset="C-GRID-02" device="-70543" value="FREQ"/>
 <part name="GND1" library="supply1" deviceset="GND" device=""/>
 <part name="R7" library="r" deviceset="R" device="0202/10" value="10kΩ"/>
@@
 <part name="P+8" library="supply1" deviceset="VCC" device=""/>
 <part name="GND13" library="supply1" deviceset="GND" device=""/>
-<part name="J4" library="pinhead" deviceset="PINHD-1X2" device="" value="J4"/>
+<part name="J4" library="pinconn" deviceset="CONN-2P" device="-2P" value="J4"/>
 <part name="J2" library="pinconn" deviceset="PIC-UART" device=""/>
 <part name="GND15" library="supply1" deviceset="GND" device=""/>
@@
 <part name="R6" library="r" deviceset="R" device="0202/7" value="10k"/>
 <part name="R11" library="r" deviceset="R" device="0202/5" value="1k"/>
+<part name="J7" library="pinconn" deviceset="CONN-2P" device="-2P"/>
+<part name="J5" library="pinconn" deviceset="CONN-2P" device="-2P"/>
 </parts>
 <sheets>
@@
 <attribute name="NAME" x="-5.08" y="29.21" size="1.778" layer="95"/>
 </instance>
-<instance part="X2" gate="-2" x="-22.86" y="27.94" rot="R180"/>
-<instance part="X2" gate="-1" x="-22.86" y="22.86" rot="R180"/>
-<instance part="X1" gate="-2" x="-22.86" y="2.54" rot="R180"/>
-<instance part="X1" gate="-1" x="-22.86" y="-1.27" rot="R180"/>
 <instance part="GND1" gate="1" x="-17.78" y="-7.62"/>
 <instance part="R7" gate="G$1" x="152.4" y="-27.94" rot="MR180"/>
@@
 <instance part="R6" gate="G$1" x="66.04" y="-15.24" rot="R90"/>
 <instance part="R11" gate="G$1" x="83.82" y="0" rot="R90"/>
+<instance part="J7" gate="G$1" x="-22.86" y="25.4" rot="MR0"/>
+<instance part="J5" gate="G$1" x="-22.86" y="0" rot="MR0"/>
 </instances>
 <busses>
@@
 </segment>
 <segment>
-<pinref part="X1" gate="-1" pin="S"/>
 <pinref part="GND1" gate="1" pin="GND"/>
-<wire x1="-20.32" y1="-1.27" x2="-17.78" y2="-1.27" width="0.1524" layer="91"/>
-<wire x1="-17.78" y1="-1.27" x2="-17.78" y2="-5.08" width="0.1524" layer="91"/>
+<wire x1="-20.32" y1="0" x2="-17.78" y2="0" width="0.1524" layer="91"/>
+<wire x1="-17.78" y1="0" x2="-17.78" y2="-5.08" width="0.1524" layer="91"/>
+<pinref part="J5" gate="G$1" pin="1"/>
 </segment>
 <segment>
@@
 <segment>
 <pinref part="GND13" gate="1" pin="GND"/>
-<pinref part="J4" gate="G$1" pin="2"/>
-<wire x1="167.64" y1="-33.02" x2="167.64" y2="-27.94" width="0.1524" layer="91"/>
-<wire x1="167.64" y1="-27.94" x2="175.26" y2="-27.94" width="0.1524" layer="91"/>
+<wire x1="167.64" y1="-33.02" x2="167.64" y2="-29.21" width="0.1524" layer="91"/>
+<pinref part="J4" gate="G$1" pin="1"/>
+<wire x1="175.26" y1="-27.94" x2="167.64" y2="-27.94" width="0.1524" layer="91"/>
+<wire x1="167.64" y1="-27.94" x2="167.64" y2="-29.21" width="0.1524" layer="91"/>
 </segment>
 <segment>
@@
 <pinref part="P+8" gate="VCC" pin="VCC"/>
 <wire x1="167.64" y1="-25.4" x2="167.64" y2="-22.86" width="0.1524" layer="91"/>
-<pinref part="J4" gate="G$1" pin="1"/>
-<wire x1="175.26" y1="-25.4" x2="167.64" y2="-25.4" width="0.1524" layer="91"/>
+<pinref part="J4" gate="G$1" pin="2"/>
+<wire x1="167.64" y1="-25.4" x2="175.26" y2="-25.4" width="0.1524" layer="91"/>
 </segment>
 <segment>
@@
 <segment>
 <wire x1="-20.32" y1="27.94" x2="-8.89" y2="27.94" width="0.1524" layer="91"/>
-<pinref part="X2" gate="-2" pin="S"/>
 <pinref part="S1" gate="G$1" pin="P"/>
+<pinref part="J7" gate="G$1" pin="2"/>
 </segment>
 </net>
@@
 <segment>
 <pinref part="S1" gate="G$1" pin="P1"/>
-<wire x1="-20.32" y1="22.86" x2="-12.7" y2="22.86" width="0.1524" layer="91"/>
-<wire x1="-12.7" y1="22.86" x2="-12.7" y2="17.78" width="0.1524" layer="91"/>
+<wire x1="-12.7" y1="25.4" x2="-12.7" y2="17.78" width="0.1524" layer="91"/>
 <wire x1="-12.7" y1="17.78" x2="-8.89" y2="17.78" width="0.1524" layer="91"/>
-<pinref part="X2" gate="-1" pin="S"/>
+<wire x1="-20.32" y1="25.4" x2="-12.7" y2="25.4" width="0.1524" layer="91"/>
+<pinref part="J7" gate="G$1" pin="1"/>
 </segment>
 </net>
 <net name="FREQ" class="0">
 <segment>
-<pinref part="X1" gate="-2" pin="S"/>
 <wire x1="-20.32" y1="2.54" x2="-12.7" y2="2.54" width="0.1524" layer="91"/>
 <label x="-17.78" y="2.54" size="1.778" layer="95"/>
 <wire x1="-12.7" y1="2.54" x2="-12.7" y2="-30.48" width="0.1524" layer="91"/>
 <wire x1="-12.7" y1="-30.48" x2="91.44" y2="-30.48" width="0.1524" layer="91"/>
-<wire x1="91.44" y1="7.62" x2="91.44" y2="-30.48" width="0.1524" layer="91"/>
 <label x="91.44" y="0" size="1.778" layer="95" rot="R270"/>
 <pinref part="U$2" gate="G$1" pin="RC2"/>
+<wire x1="91.44" y1="5.08" x2="91.44" y2="-30.48" width="0.1524" layer="91"/>
+<wire x1="91.44" y1="7.62" x2="91.44" y2="5.08" width="0.1524" layer="91"/>
+<pinref part="U$2" gate="G$1" pin="RC0"/>
+<wire x1="91.44" y1="5.08" x2="81.28" y2="5.08" width="0.1524" layer="91"/>
+<wire x1="81.28" y1="5.08" x2="81.28" y2="7.62" width="0.1524" layer="91"/>
+<junction x="91.44" y="5.08"/>
+<pinref part="J5" gate="G$1" pin="2"/>
 </segment>
 </net>
@@
 </segment>
 </net>
+<net name="N$11" class="0">
+<segment>
+<pinref part="U$2" gate="G$1" pin="RB0"/>
+<wire x1="142.24" y1="43.18" x2="142.24" y2="50.8" width="0.1524" layer="91"/>
+<wire x1="142.24" y1="50.8" x2="147.32" y2="50.8" width="0.1524" layer="91"/>
+<pinref part="U$2" gate="G$1" pin="RB1"/>
+<wire x1="147.32" y1="50.8" x2="147.32" y2="43.18" width="0.1524" layer="91"/>
+<wire x1="142.24" y1="50.8" x2="142.24" y2="58.42" width="0.1524" layer="91"/>
+<junction x="142.24" y="50.8"/>
+</segment>
+</net>

Commit message: ...
Parts:
- C1, C2: device c:C050-020X036 -> c:C025-025X060
- C3, C4: device c:CPOLE2,5-4 -> c:CPOLE2.5-5
Changed lines of the file:
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@@
 <part name="R4" library="r" deviceset="R" device="0202/7" value="47kΩ"/>
 <part name="R10" library="r" deviceset="R" device="0202/7" value="4.7kΩ"/>
-<part name="C1" library="c" deviceset="C" device="050-020X036" value="1nF"/>
-<part name="C2" library="c" deviceset="C" device="050-020X036" value="1nF"/>
-<part name="C3" library="c" deviceset="CPOL" device="E2,5-4" value="10μF"/>
-<part name="C4" library="c" deviceset="CPOL" device="E2,5-4" value="10μF"/>
+<part name="C1" library="c" deviceset="C" device="025-025X060" value="1nF"/>
+<part name="C2" library="c" deviceset="C" device="025-025X060" value="1nF"/>
+<part name="C3" library="c" deviceset="CPOL" device="E2.5-5" value="10μF"/>
+<part name="C4" library="c" deviceset="CPOL" device="E2.5-5" value="10μF"/>
 <part name="C5" library="c" deviceset="C" device="025-020X036" value="33pF"/>
 <part name="C6" library="c" deviceset="C" device="025-020X036" value="33pF"/>

Commit message: ...
Parts:
- added D2: 1N4148-12, d:1N4148-12
Connections:
- new net N$12: C7.+, D2.A, J4.2
- net VCC: now also D2.C; no longer C7.+, J4.2
Other:
- moved on the sheet: C7, C9, J4
Changed lines of the file:
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@@
 <part name="C9" library="rcl" deviceset="C-EU" device="025-024X044" value="100nF"/>
 <part name="GND2" library="supply1" deviceset="GND" device=""/>
-<part name="GND4" library="supply1" deviceset="GND" device=""/>
 <part name="GND5" library="supply1" deviceset="GND" device=""/>
 <part name="GND6" library="supply1" deviceset="GND" device=""/>
@@
 <part name="LED1" library="led" deviceset="TLLG4400" device=""/>
 <part name="GND10" library="supply1" deviceset="GND" device=""/>
-<part name="P+8" library="supply1" deviceset="VCC" device=""/>
 <part name="GND13" library="supply1" deviceset="GND" device=""/>
 <part name="J4" library="pinconn" deviceset="CONN-2P" device="-2P" value="J4"/>
@@
 <part name="J7" library="pinconn" deviceset="CONN-2P" device="-2P"/>
 <part name="J5" library="pinconn" deviceset="CONN-2P" device="-2P"/>
+<part name="D2" library="d" deviceset="1N4148" device="-12" value="1N4148-12"/>
 </parts>
 <sheets>
@@
 <instance part="C5" gate="G$1" x="177.8" y="-2.54" rot="MR180"/>
 <instance part="C6" gate="G$1" x="167.64" y="-2.54" rot="R180"/>
-<instance part="C7" gate="G$1" x="199.39" y="-20.32" smashed="yes" rot="R270">
-<attribute name="NAME" x="199.517" y="-18.288" size="1.27" layer="95" rot="R180" align="top-center"/>
-<attribute name="VALUE" x="199.517" y="-22.86" size="1.27" layer="96" rot="R180" align="bottom-center"/>
-</instance>
-<instance part="C9" gate="G$1" x="200.66" y="-30.48" smashed="yes" rot="R270">
-<attribute name="NAME" x="199.39" y="-27.94" size="1.4224" layer="95" align="bottom-center"/>
-<attribute name="VALUE" x="199.39" y="-33.02" size="1.27" layer="96" align="top-center"/>
+<instance part="C7" gate="G$1" x="185.42" y="-22.86" smashed="yes">
+<attribute name="NAME" x="183.388" y="-22.733" size="1.27" layer="95" rot="R270" align="top-center"/>
+<attribute name="VALUE" x="187.96" y="-22.733" size="1.27" layer="96" rot="R270" align="bottom-center"/>
+</instance>
+<instance part="C9" gate="G$1" x="200.66" y="-21.59" smashed="yes">
+<attribute name="NAME" x="198.12" y="-22.86" size="1.4224" layer="95" rot="R90" align="bottom-center"/>
+<attribute name="VALUE" x="203.2" y="-22.86" size="1.27" layer="96" rot="R90" align="top-center"/>
 </instance>
 <instance part="GND2" gate="1" x="58.42" y="5.08"/>
-<instance part="GND4" gate="1" x="190.5" y="-35.56"/>
 <instance part="GND5" gate="1" x="22.86" y="-2.54"/>
 <instance part="GND6" gate="1" x="35.56" y="-2.54"/>
@@
 <instance part="L1" gate="G$1" x="12.7" y="25.4" rot="R90"/>
 <instance part="Q1" gate="G$1" x="172.72" y="5.08"/>
-<instance part="P+3" gate="VCC" x="208.28" y="-12.7" smashed="yes">
-<attribute name="VALUE" x="208.28" y="-11.43" size="1.778" layer="96" align="bottom-center"/>
+<instance part="P+3" gate="VCC" x="200.66" y="-12.7" smashed="yes">
+<attribute name="VALUE" x="200.66" y="-11.43" size="1.778" layer="96" align="bottom-center"/>
 </instance>
 <instance part="P+4" gate="VCC" x="43.18" y="63.5" smashed="yes">
@@
 <instance part="LED1" gate="G$1" x="72.39" y="0" rot="MR90"/>
 <instance part="GND10" gate="1" x="66.04" y="-5.08"/>
-<instance part="P+8" gate="VCC" x="167.64" y="-20.32" smashed="yes">
-<attribute name="VALUE" x="167.64" y="-19.05" size="1.778" layer="96" align="bottom-center"/>
-</instance>
-<instance part="GND13" gate="1" x="167.64" y="-35.56"/>
-<instance part="J4" gate="G$1" x="177.8" y="-27.94"/>
+<instance part="GND13" gate="1" x="200.66" y="-35.56" rot="MR0"/>
+<instance part="J4" gate="G$1" x="175.26" y="-27.94" rot="MR0"/>
 <instance part="J2" gate="1" x="134.62" y="-11.43"/>
 <instance part="GND15" gate="1" x="121.92" y="-21.59"/>
@@
 <instance part="J7" gate="G$1" x="-22.86" y="25.4" rot="MR0"/>
 <instance part="J5" gate="G$1" x="-22.86" y="0" rot="MR0"/>
+<instance part="D2" gate="G$1" x="193.04" y="-17.78" rot="R270"/>
 </instances>
 <busses>
@@
 <pinref part="GND2" gate="1" pin="GND"/>
 <wire x1="58.42" y1="10.16" x2="58.42" y2="7.62" width="0.1524" layer="91"/>
-</segment>
-<segment>
-<pinref part="GND4" gate="1" pin="GND"/>
-<pinref part="C7" gate="G$1" pin="-"/>
-<pinref part="C9" gate="G$1" pin="2"/>
-<wire x1="190.5" y1="-30.48" x2="190.5" y2="-20.32" width="0.1524" layer="91"/>
-<wire x1="190.5" y1="-20.32" x2="195.58" y2="-20.32" width="0.1524" layer="91"/>
-<wire x1="190.5" y1="-33.02" x2="190.5" y2="-30.48" width="0.1524" layer="91"/>
-<wire x1="190.5" y1="-30.48" x2="195.58" y2="-30.48" width="0.1524" layer="91"/>
-<junction x="190.5" y="-30.48"/>
 </segment>
 <segment>
@@
 <segment>
 <pinref part="GND13" gate="1" pin="GND"/>
-<wire x1="167.64" y1="-33.02" x2="167.64" y2="-29.21" width="0.1524" layer="91"/>
+<wire x1="200.66" y1="-33.02" x2="200.66" y2="-27.94" width="0.1524" layer="91"/>
 <pinref part="J4" gate="G$1" pin="1"/>
-<wire x1="175.26" y1="-27.94" x2="167.64" y2="-27.94" width="0.1524" layer="91"/>
-<wire x1="167.64" y1="-27.94" x2="167.64" y2="-29.21" width="0.1524" layer="91"/>
+<wire x1="200.66" y1="-27.94" x2="185.42" y2="-27.94" width="0.1524" layer="91"/>
+<wire x1="177.8" y1="-27.94" x2="185.42" y2="-27.94" width="0.1524" layer="91"/>
+<wire x1="185.42" y1="-27.94" x2="185.42" y2="-26.67" width="0.1524" layer="91"/>
+<pinref part="C7" gate="G$1" pin="-"/>
+<junction x="185.42" y="-27.94"/>
+<pinref part="C9" gate="G$1" pin="2"/>
+<wire x1="200.66" y1="-26.67" x2="200.66" y2="-27.94" width="0.1524" layer="91"/>
+<junction x="200.66" y="-27.94"/>
 </segment>
 <segment>
@@
 <pinref part="P+5" gate="VCC" pin="VCC"/>
 <wire x1="124.46" y1="55.88" x2="124.46" y2="58.42" width="0.1524" layer="91"/>
-</segment>
-<segment>
-<pinref part="C7" gate="G$1" pin="+"/>
-<pinref part="C9" gate="G$1" pin="1"/>
-<wire x1="203.2" y1="-20.32" x2="208.28" y2="-20.32" width="0.1524" layer="91"/>
-<wire x1="208.28" y1="-20.32" x2="208.28" y2="-30.48" width="0.1524" layer="91"/>
-<wire x1="208.28" y1="-30.48" x2="203.2" y2="-30.48" width="0.1524" layer="91"/>
-<pinref part="P+3" gate="VCC" pin="VCC"/>
-<wire x1="208.28" y1="-20.32" x2="208.28" y2="-15.24" width="0.1524" layer="91"/>
-<junction x="208.28" y="-20.32"/>
 </segment>
 <segment>
@@
 </segment>
 <segment>
-<pinref part="P+8" gate="VCC" pin="VCC"/>
-<wire x1="167.64" y1="-25.4" x2="167.64" y2="-22.86" width="0.1524" layer="91"/>
-<pinref part="J4" gate="G$1" pin="2"/>
-<wire x1="167.64" y1="-25.4" x2="175.26" y2="-25.4" width="0.1524" layer="91"/>
-</segment>
-<segment>
 <pinref part="J2" gate="1" pin="VDD"/>
 <pinref part="P+9" gate="VCC" pin="VCC"/>
@@
 <wire x1="132.08" y1="58.42" x2="132.08" y2="43.18" width="0.1524" layer="91"/>
 <pinref part="U$2" gate="G$1" pin="VDD"/>
+</segment>
+<segment>
+<pinref part="D2" gate="G$1" pin="C"/>
+<wire x1="195.58" y1="-17.78" x2="200.66" y2="-17.78" width="0.1524" layer="91"/>
+<wire x1="200.66" y1="-17.78" x2="200.66" y2="-15.24" width="0.1524" layer="91"/>
+<pinref part="P+3" gate="VCC" pin="VCC"/>
+<pinref part="C9" gate="G$1" pin="1"/>
+<wire x1="200.66" y1="-19.05" x2="200.66" y2="-17.78" width="0.1524" layer="91"/>
+<junction x="200.66" y="-17.78"/>
 </segment>
 </net>
@@
 </segment>
 </net>
+<net name="N$12" class="0">
+<segment>
+<wire x1="180.34" y1="-17.78" x2="185.42" y2="-17.78" width="0.1524" layer="91"/>
+<pinref part="J4" gate="G$1" pin="2"/>
+<wire x1="185.42" y1="-17.78" x2="190.5" y2="-17.78" width="0.1524" layer="91"/>
+<wire x1="180.34" y1="-17.78" x2="180.34" y2="-25.4" width="0.1524" layer="91"/>
+<wire x1="180.34" y1="-25.4" x2="177.8" y2="-25.4" width="0.1524" layer="91"/>
+<pinref part="C7" gate="G$1" pin="+"/>
+<wire x1="185.42" y1="-19.05" x2="185.42" y2="-17.78" width="0.1524" layer="91"/>
+<junction x="185.42" y="-17.78"/>
+<pinref part="D2" gate="G$1" pin="A"/>
+</segment>
+</net>

Commit message: ...
Parts:
- added C8: 22pF, c:C050-020X036
- C7: device c:CPOLE2.5-6 -> c:CPOLE2.5-5
- R8: device r:R0202/5 -> r:R0202/7
Connections:
- net N$1 renamed PGC
- removed net N$3: J3.PGD, R9.1
- new net PGD: C8.2, J3.PGD, R9.1
- net D6: now also R8.2; no longer R9.2
- net D7: now also R9.2; no longer R8.2
- net GND: now also C8.1
Other:
- moved on the sheet: J1, J3, R10, R8, R9

Commit message: ...
Parts:
- C3, C4: device c:CPOLE2.5-5 -> c:CPOLE2,5-4
Connections:
- net /RELAY: now also D1.A; no longer D1.C
- net VCC: now also D1.C; no longer D1.A
Other:
- moved on the sheet: D1
Changed lines of the file:
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@@
 <part name="C1" library="c" deviceset="C" device="025-025X060" value="1nF"/>
 <part name="C2" library="c" deviceset="C" device="025-025X060" value="1nF"/>
-<part name="C3" library="c" deviceset="CPOL" device="E2.5-5" value="10μF"/>
-<part name="C4" library="c" deviceset="CPOL" device="E2.5-5" value="10μF"/>
+<part name="C3" library="c" deviceset="CPOL" device="E2,5-4" value="10μF"/>
+<part name="C4" library="c" deviceset="CPOL" device="E2,5-4" value="10μF"/>
 <part name="C5" library="c" deviceset="C" device="025-020X036" value="33pF"/>
 <part name="C6" library="c" deviceset="C" device="025-020X036" value="33pF"/>
@@
 <instance part="GND6" gate="1" x="35.56" y="-2.54"/>
 <instance part="GND7" gate="1" x="43.18" y="12.7" rot="MR0"/>
-<instance part="D1" gate="G$1" x="50.8" y="0" rot="R180"/>
+<instance part="D1" gate="G$1" x="50.8" y="0" rot="MR0"/>
 <instance part="L1" gate="G$1" x="12.7" y="25.4" rot="R90"/>
 <instance part="Q1" gate="G$1" x="172.72" y="5.08"/>
@@
 <junction x="58.42" y="45.72"/>
 <label x="88.9" y="45.72" size="1.778" layer="95"/>
-<label x="58.42" y="35.56" size="1.778" layer="95"/>
 <wire x1="58.42" y1="45.72" x2="93.98" y2="45.72" width="0.1524" layer="91"/>
 <wire x1="93.98" y1="45.72" x2="104.14" y2="45.72" width="0.1524" layer="91"/>
@@
 <segment>
 <wire x1="50.8" y1="10.16" x2="50.8" y2="7.62" width="0.1524" layer="91"/>
-<pinref part="D1" gate="G$1" pin="A"/>
-<wire x1="50.8" y1="7.62" x2="50.8" y2="2.54" width="0.1524" layer="91"/>
 <wire x1="43.18" y1="5.08" x2="43.18" y2="7.62" width="0.1524" layer="91"/>
 <wire x1="43.18" y1="7.62" x2="50.8" y2="7.62" width="0.1524" layer="91"/>
-<junction x="50.8" y="7.62"/>
 <pinref part="K2" gate="1" pin="-"/>
 <pinref part="P+7" gate="VCC" pin="VCC"/>
+<pinref part="D1" gate="G$1" pin="C"/>
+<wire x1="50.8" y1="2.54" x2="50.8" y2="7.62" width="0.1524" layer="91"/>
+<junction x="50.8" y="7.62"/>
 </segment>
 <segment>
@@
 <pinref part="T1" gate="G$1" pin="C"/>
 <label x="52.07" y="-15.24" size="1.778" layer="95" rot="MR0"/>
-<pinref part="D1" gate="G$1" pin="C"/>
-<wire x1="50.8" y1="-2.54" x2="50.8" y2="-7.62" width="0.1524" layer="91"/>
 <wire x1="50.8" y1="-10.16" x2="50.8" y2="-7.62" width="0.1524" layer="91"/>
 <wire x1="50.8" y1="-7.62" x2="43.18" y2="-7.62" width="0.1524" layer="91"/>
 <wire x1="43.18" y1="-5.08" x2="43.18" y2="-7.62" width="0.1524" layer="91"/>
 <pinref part="K2" gate="1" pin="+"/>
+<pinref part="D1" gate="G$1" pin="A"/>
+<wire x1="50.8" y1="-2.54" x2="50.8" y2="-7.62" width="0.1524" layer="91"/>
 <junction x="50.8" y="-7.62"/>
 </segment>

Commit message: ...
Parts:
- S1: value SL-SW-2P-2T -> SL-SW-2P-2T-H; device sw:SL-SW-2P-2T -> sw:SL-SW-2P-2T-H
Changed lines of the file:
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@@
 <part name="GND8" library="supply1" deviceset="GND" device=""/>
 <part name="P+7" library="supply1" deviceset="VCC" device=""/>
-<part name="S1" library="sw" deviceset="SL-SW-2P-2T" device=""/>
+<part name="S1" library="sw" deviceset="SL-SW-2P-2T" device="-H" value="SL-SW-2P-2T-H"/>
 <part name="GND1" library="supply1" deviceset="GND" device=""/>
 <part name="R7" library="r" deviceset="R" device="0202/10" value="10kΩ"/>
