File: eagle/LCmeter0-LCD-8pinlcd-alt.brd (EAGLE design)
At the start: 58.4 x 50.8 mm, 34 parts, among them IC1 PIC16F876A-X/SP, J1 HD44780-4BIT-8PIN, J2 PIC-UART, K2 DS2Y, Q1 20MHz, SW1 SPST, T1 BC547CBE-A, X1 FREQ, X2 L/C

Commit message: ...
Parts:
- R1, R10, R3, R4: device r:0202/2V -> r:0202/7
- moved C3 9.16 mm to (20.3, 38.1)
- moved SW1 8.89 mm to (8.89, 45.7)
- moved C4 7.18 mm to (22.9, 30.5)
- moved C2 5.68 mm to (15.2, 33.0)
- moved C1 5.68 mm to (17.8, 33.0)
- moved R4 5.39 mm to (31.8, 33.0), turned to 270 degrees
- moved R5 4.02 mm to (31.8, 27.9), turned to 90 degrees
- moved R10 4.02 mm to (31.8, 40.6), turned to 90 degrees
- moved L1 3.59 mm to (11.4, 38.1)
- moved R1 2.54 mm to (31.8, 38.1)
- moved R3 2.54 mm to (31.8, 43.2)
- moved R2 1.80 mm to (31.8, 25.4), turned to 90 degrees
Routing:
- net A3: track 22.9 -> 49.5 mm
- net A1: track 7.62 -> 20.3 mm, vias 0 -> 2
- net GND: track 175.3 -> 186.7 mm, vias 4 -> 6
- net /MCLR: track 33.0 -> 44.4 mm
- net C2_CON: track 17.8 -> 25.4 mm
- net N$2: track 30.5 -> 38.1 mm
- net A0: track 25.4 -> 30.5 mm
- net A4: track 5.08 -> 2.54 mm
- net VCC: track 152.4 -> 149.9 mm, vias 11 -> 9

Commit message: ...
Parts:
- moved C9 5.08 mm to (50.8, 19.1)
- moved SW1 3.81 mm to (12.7, 45.7)
- renumbered U$1 to J3
Routing:
- net N$2: track 38.1 -> 30.5 mm
- net GND: track 186.7 -> 190.5 mm, vias 6 -> 2
- net /MCLR: track 44.4 -> 40.6 mm
- net VCC: track 149.9 -> 147.3 mm
Changed lines of the file:
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@@
 <element name="C6" library="c" package="C025-020X036" value="33pF" x="26.67" y="20.32" rot="R90"/>
 <element name="C7" library="c" package="E2,5-6" value="100μF" x="52.07" y="7.62" rot="R180"/>
-<element name="C9" library="rcl" package="C025-024X044" value="100nF" x="50.8" y="24.13" smashed="yes" rot="R270">
-<attribute name="NAME" x="49.53" y="21.59" size="1.27" layer="25" ratio="10" rot="R270"/>
-<attribute name="VALUE" x="48.133" y="25.908" size="1.27" layer="27" ratio="10" rot="R270"/>
+<element name="C9" library="rcl" package="C025-024X044" value="100nF" x="50.8" y="19.05" smashed="yes" rot="R270">
+<attribute name="NAME" x="49.53" y="16.51" size="1.27" layer="25" ratio="10" rot="R270"/>
+<attribute name="VALUE" x="48.133" y="20.828" size="1.27" layer="27" ratio="10" rot="R270"/>
 </element>
 <element name="D1" library="d" package="DO34-7" value="1N4148" x="19.05" y="2.54" rot="R180"/>
@@
 <element name="R4" library="r" package="0202/7" value="47kΩ" x="31.75" y="33.02" rot="R270"/>
 <element name="R5" library="r" package="0202/7" value="4.7kΩ" x="31.75" y="27.94" rot="R90"/>
-<element name="SW1" library="lc-meter" package="PB-5" value="SPST" x="8.89" y="45.72"/>
+<element name="SW1" library="lc-meter" package="PB-5" value="SPST" x="12.7" y="45.72"/>
 <element name="K2" library="relay" package="DS2Y" value="DS2Y" x="19.05" y="13.97" rot="R90">
 <attribute name="OC_NEWARK" value="13P3268" x="19.05" y="13.97" size="1.778" layer="27" rot="R90" display="off"/>
@@
 </element>
 <element name="R7" library="r" package="0202/10" value="10kΩ" x="10.16" y="10.16"/>
-<element name="U$1" library="pinconn" package="CONN-5P" value="PIC-ICSP" x="35.56" y="48.26"/>
+<element name="J3" library="pinconn" package="CONN-5P" value="PIC-ICSP" x="35.56" y="48.26"/>
 <element name="R8" library="r" package="0202/5" value="100" x="48.26" y="45.72" rot="R270"/>
 <element name="R9" library="r" package="0202/5" value="100" x="48.26" y="40.64" rot="R180"/>
@@
 <contactref element="C3" pad="-"/>
 <contactref element="S1" pad="1"/>
-<wire x1="15.24" y1="38.1" x2="17.78" y2="38.1" width="0.4064" layer="16"/>
-<wire x1="15.24" y1="35.56" x2="17.78" y2="35.56" width="0.4064" layer="16"/>
-<wire x1="17.78" y1="35.56" x2="17.78" y2="38.1" width="0.4064" layer="16"/>
 <wire x1="17.78" y1="38.1" x2="15.24" y2="38.1" width="0.4064" layer="16"/>
 <wire x1="15.24" y1="35.56" x2="17.78" y2="35.56" width="0.4064" layer="16"/>
@@
 <contactref element="IC1" pad="8"/>
 <contactref element="T1" pad="E"/>
-<wire x1="50.8" y1="22.86" x2="48.26" y2="22.86" width="0.4064" layer="16"/>
 <wire x1="48.26" y1="22.86" x2="48.26" y2="17.78" width="0.4064" layer="1"/>
-<wire x1="50.8" y1="17.78" x2="48.26" y2="17.78" width="0.4064" layer="16"/>
+<wire x1="53.34" y1="17.78" x2="50.8" y2="17.78" width="0.4064" layer="16"/>
 <wire x1="48.26" y1="17.78" x2="45.72" y2="17.78" width="0.4064" layer="16"/>
 <wire x1="25.4" y1="17.78" x2="25.4" y2="20.32" width="0.4064" layer="16"/>
@@
 <wire x1="50.8" y1="0" x2="50.8" y2="2.54" width="0.4064" layer="16"/>
 <wire x1="50.8" y1="2.54" x2="50.8" y2="7.62" width="0.4064" layer="16"/>
-<wire x1="53.34" y1="22.86" x2="50.8" y2="22.86" width="0.4064" layer="16"/>
 <wire x1="25.4" y1="0" x2="2.54" y2="0" width="0.4064" layer="16"/>
-<contactref element="U$1" pad="1"/>
+<contactref element="J3" pad="1"/>
 <contactref element="SW1" pad="3"/>
 <contactref element="J1" pad="1"/>
@@
 <contactref element="JP1" pad="2"/>
 <contactref element="J2" pad="19"/>
-<wire x1="53.34" y1="17.78" x2="50.8" y2="17.78" width="0.4064" layer="16"/>
+<wire x1="53.34" y1="17.78" x2="55.88" y2="17.78" width="0.4064" layer="16"/>
 <wire x1="50.8" y1="7.62" x2="50.8" y2="10.16" width="0.4064" layer="16"/>
-<via x="50.8" y="10.16" extent="1-16" drill="0.6" shape="square"/>
-<wire x1="50.8" y1="10.16" x2="50.8" y2="17.78" width="0.4064" layer="1"/>
-<via x="50.8" y="17.78" extent="1-16" drill="0.6" shape="square"/>
+<wire x1="50.8" y1="10.16" x2="55.88" y2="10.16" width="0.4064" layer="16"/>
+<wire x1="55.88" y1="10.16" x2="55.88" y2="17.78" width="0.4064" layer="16"/>
 <via x="48.26" y="22.86" extent="1-16" drill="0.6" shape="square"/>
 <via x="48.26" y="17.78" extent="1-16" drill="0.6" shape="square"/>
 <wire x1="35.56" y1="48.26" x2="20.32" y2="48.26" width="0.4064" layer="16"/>
-<wire x1="20.32" y1="48.26" x2="11.43" y2="48.26" width="0.4064" layer="16"/>
+<wire x1="20.32" y1="48.26" x2="15.24" y2="48.26" width="0.4064" layer="16"/>
 <wire x1="17.78" y1="30.48" x2="20.32" y2="30.48" width="0.4064" layer="16"/>
 <wire x1="20.32" y1="30.48" x2="20.32" y2="22.86" width="0.4064" layer="16"/>
 <wire x1="20.32" y1="22.86" x2="22.86" y2="22.86" width="0.4064" layer="16"/>
 <wire x1="22.86" y1="22.86" x2="25.4" y2="22.86" width="0.4064" layer="16"/>
-<wire x1="20.32" y1="30.48" x2="20.32" y2="43.18" width="0.4064" layer="16"/>
-<via x="20.32" y="43.18" extent="1-16" drill="0.6" shape="square"/>
-<wire x1="20.32" y1="43.18" x2="20.32" y2="48.26" width="0.4064" layer="1"/>
-<via x="20.32" y="48.26" extent="1-16" drill="0.6" shape="square"/>
+<wire x1="20.32" y1="30.48" x2="20.32" y2="48.26" width="0.4064" layer="16"/>
+<wire x1="48.26" y1="22.86" x2="53.34" y2="22.86" width="0.4064" layer="16"/>
+<wire x1="50.8" y1="17.78" x2="48.26" y2="17.78" width="0.4064" layer="16"/>
 </signal>
 <signal name="N$7">
@@
 <wire x1="15.24" y1="2.54" x2="15.24" y2="5.08" width="0.4064" layer="16"/>
 <wire x1="55.88" y1="7.62" x2="55.88" y2="20.32" width="0.4064" layer="1"/>
-<wire x1="45.72" y1="20.32" x2="53.34" y2="20.32" width="0.4064" layer="16"/>
+<wire x1="45.72" y1="20.32" x2="50.8" y2="20.32" width="0.4064" layer="16"/>
 <wire x1="55.88" y1="20.32" x2="55.88" y2="25.4" width="0.4064" layer="16"/>
 <contactref element="IC1" pad="20"/>
@@
 <wire x1="10.16" y1="5.08" x2="12.7" y2="5.08" width="0.4064" layer="16"/>
 <wire x1="12.7" y1="5.08" x2="15.24" y2="5.08" width="0.4064" layer="16"/>
-<via x="50.8" y="25.4" extent="1-16" drill="0.6" shape="square"/>
+<via x="50.8" y="20.32" extent="1-16" drill="0.6" shape="square"/>
 <via x="55.88" y="20.32" extent="1-16" drill="0.6" shape="square"/>
 <via x="55.88" y="7.62" extent="1-16" drill="0.6" shape="square"/>
@@
 <wire x1="12.7" y1="15.24" x2="12.7" y2="5.08" width="0.4064" layer="1"/>
 <via x="12.7" y="5.08" extent="1-16" drill="0.6" shape="square"/>
-<contactref element="U$1" pad="2"/>
+<contactref element="J3" pad="2"/>
 <wire x1="55.88" y1="25.4" x2="53.34" y2="25.4" width="0.4064" layer="16"/>
 <contactref element="J1" pad="2"/>
-<wire x1="53.34" y1="25.4" x2="50.8" y2="25.4" width="0.4064" layer="16"/>
 <contactref element="JP1" pad="1"/>
 <wire x1="53.34" y1="2.54" x2="53.34" y2="7.62" width="0.4064" layer="16"/>
@@
 <wire x1="43.18" y1="43.18" x2="38.1" y2="43.18" width="0.4064" layer="1"/>
 <via x="38.1" y="43.18" extent="1-16" drill="0.6" shape="square"/>
+<wire x1="53.34" y1="20.32" x2="50.8" y2="20.32" width="0.4064" layer="16"/>
 </signal>
 <signal name="D4">
@@
 <contactref element="R10" pad="1"/>
 <contactref element="IC1" pad="1"/>
-<contactref element="U$1" pad="3"/>
+<contactref element="J3" pad="3"/>
 <contactref element="SW1" pad="1"/>
 <wire x1="35.56" y1="40.64" x2="38.1" y2="40.64" width="0.4064" layer="16"/>
@@
 <wire x1="40.64" y1="40.64" x2="40.64" y2="45.72" width="0.4064" layer="16"/>
 <wire x1="40.64" y1="45.72" x2="40.64" y2="48.26" width="0.4064" layer="16"/>
-<wire x1="11.43" y1="43.18" x2="11.43" y2="45.72" width="0.4064" layer="16"/>
-<wire x1="11.43" y1="45.72" x2="35.56" y2="45.72" width="0.4064" layer="16"/>
-<via x="35.56" y="45.72" extent="1-16" drill="0.6" shape="square"/>
-<wire x1="35.56" y1="45.72" x2="40.64" y2="45.72" width="0.4064" layer="1"/>
+<wire x1="15.24" y1="43.18" x2="15.24" y2="45.72" width="0.4064" layer="16"/>
+<wire x1="15.24" y1="45.72" x2="17.78" y2="45.72" width="0.4064" layer="16"/>
+<via x="17.78" y="45.72" extent="1-16" drill="0.6" shape="square"/>
+<wire x1="17.78" y1="45.72" x2="40.64" y2="45.72" width="0.4064" layer="1"/>
 <via x="40.64" y="45.72" extent="1-16" drill="0.6" shape="square"/>
 </signal>
@@
 </signal>
 <signal name="N$1">
-<contactref element="U$1" pad="4"/>
+<contactref element="J3" pad="4"/>
 <contactref element="R8" pad="1"/>
 <wire x1="43.18" y1="48.26" x2="43.18" y2="45.72" width="0.4064" layer="16"/>
@@
 <signal name="N$3">
 <contactref element="R9" pad="1"/>
-<contactref element="U$1" pad="5"/>
+<contactref element="J3" pad="5"/>
 <wire x1="45.72" y1="48.26" x2="48.26" y2="48.26" width="0.4064" layer="16"/>
 <wire x1="48.26" y1="48.26" x2="48.26" y2="43.18" width="0.4064" layer="16"/>

Commit message: ...
Parts:
- IC1: device lc-meter:DIL28-3 -> mcu:DIL28-3
- SW1: device lc-meter:PB-5 -> mcu:PB-5
Changed lines of the file:
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@@
 </element>
 <element name="D1" library="d" package="DO34-7" value="1N4148" x="19.05" y="2.54" rot="R180"/>
-<element name="IC1" library="lc-meter" package="DIL28-3" value="PIC16F876A-X/SP" x="41.91" y="24.13" rot="R270"/>
+<element name="IC1" library="mcu" package="DIL28-3" value="PIC16F876A-X/SP" x="41.91" y="24.13" rot="R270"/>
 <element name="L1" library="r" package="L-02/7" value="100μH" x="11.43" y="38.1" rot="R90"/>
 <element name="Q1" library="q" package="HC49" value="20MHz" x="33.02" y="17.78" rot="R270"/>
@@
 <element name="R4" library="r" package="0202/7" value="47kΩ" x="31.75" y="33.02" rot="R270"/>
 <element name="R5" library="r" package="0202/7" value="4.7kΩ" x="31.75" y="27.94" rot="R90"/>
-<element name="SW1" library="lc-meter" package="PB-5" value="SPST" x="12.7" y="45.72"/>
+<element name="SW1" library="mcu" package="PB-5" value="SPST" x="12.7" y="45.72"/>
 <element name="K2" library="relay" package="DS2Y" value="DS2Y" x="19.05" y="13.97" rot="R90">
 <attribute name="OC_NEWARK" value="13P3268" x="19.05" y="13.97" size="1.778" layer="27" rot="R90" display="off"/>
