File: eagle/LCmeter0-LCD-8pinlcd-alt.sch (EAGLE design)
At the start: 34 parts, among them IC1 PIC16F876A-X/SP, J1 HD44780-4BIT-8PIN, J2 PIC-UART, K2 DS2Y, Q1 20MHz, SW1 SPST, T1 BC547CBE-A, X1 FREQ, X2 L/C

Commit message: ...
Parts:
- R1, R10, R3, R4: device r:R0202/2V -> r:R0202/7
Changed lines of the file:
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@@
 <setting verticaltext="up"/>
 </settings>
-<grid distance="50" unitdist="mil" unit="inch" style="dots" multiple="2" display="yes" altdistance="10" altunitdist="mil" altunit="inch"/>
+<grid distance="50" unitdist="mil" unit="inch" style="lines" multiple="2" display="yes" altdistance="10" altunitdist="mil" altunit="inch"/>
 <layers>
 <layer number="1" name="Top" color="4" fill="1" visible="yes" active="no"/>
@@
 <parts>
 <part name="IC1" library="lc-meter" deviceset="PIC16F876A-X/SP" device=""/>
-<part name="R1" library="r" deviceset="R" device="0202/2V" value="100kΩ"/>
+<part name="R1" library="r" deviceset="R" device="0202/7" value="100kΩ"/>
 <part name="R2" library="r" deviceset="R" device="0202/7" value="100kΩ"/>
-<part name="R3" library="r" deviceset="R" device="0202/2V" value="100kΩ"/>
-<part name="R4" library="r" deviceset="R" device="0202/2V" value="47kΩ"/>
-<part name="R10" library="r" deviceset="R" device="0202/2V" value="4.7kΩ"/>
+<part name="R3" library="r" deviceset="R" device="0202/7" value="100kΩ"/>
+<part name="R4" library="r" deviceset="R" device="0202/7" value="47kΩ"/>
+<part name="R10" library="r" deviceset="R" device="0202/7" value="4.7kΩ"/>
 <part name="C1" library="c" deviceset="C" device="050-020X036" value="1nF"/>
 <part name="C2" library="c" deviceset="C" device="050-020X036" value="1nF"/>

Commit message: ...
Parts:
- renumbered U$1 to J3
Changed lines of the file:
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@@
 <part name="GND1" library="supply1" deviceset="GND" device=""/>
 <part name="R7" library="r" deviceset="R" device="0202/10" value="10kΩ"/>
-<part name="U$1" library="pinconn" deviceset="PIC-ICSP" device=""/>
+<part name="J3" library="pinconn" deviceset="PIC-ICSP" device=""/>
 <part name="P+1" library="supply1" deviceset="VCC" device=""/>
 <part name="GND9" library="supply1" deviceset="GND" device=""/>
@@
 <instance part="GND1" gate="1" x="-58.42" y="-7.62"/>
 <instance part="R7" gate="G$1" x="142.24" y="7.62" rot="MR180"/>
-<instance part="U$1" gate="G$1" x="172.72" y="68.58"/>
+<instance part="J3" gate="G$1" x="172.72" y="68.58"/>
 <instance part="P+1" gate="VCC" x="152.4" y="81.28" smashed="yes">
 <attribute name="VALUE" x="152.4" y="82.55" size="1.778" layer="96" align="bottom-center"/>
@@
 </segment>
 <segment>
-<pinref part="U$1" gate="G$1" pin="VSS"/>
+<pinref part="J3" gate="G$1" pin="VSS"/>
 <pinref part="GND9" gate="1" pin="GND"/>
 <wire x1="165.1" y1="71.12" x2="147.32" y2="71.12" width="0.1524" layer="91"/>
@@
 <segment>
 <pinref part="P+1" gate="VCC" pin="VCC"/>
-<pinref part="U$1" gate="G$1" pin="VDD"/>
+<pinref part="J3" gate="G$1" pin="VDD"/>
 <wire x1="152.4" y1="78.74" x2="152.4" y2="73.66" width="0.1524" layer="91"/>
 <wire x1="152.4" y1="73.66" x2="165.1" y2="73.66" width="0.1524" layer="91"/>
@@
 </segment>
 <segment>
-<pinref part="U$1" gate="G$1" pin="MCLR"/>
+<pinref part="J3" gate="G$1" pin="MCLR"/>
 <wire x1="165.1" y1="68.58" x2="147.32" y2="68.58" width="0.1524" layer="91"/>
 <label x="147.32" y="68.58" size="1.778" layer="95"/>
@@
 <net name="N$1" class="0">
 <segment>
-<pinref part="U$1" gate="G$1" pin="PGC"/>
+<pinref part="J3" gate="G$1" pin="PGC"/>
 <pinref part="R8" gate="G$1" pin="1"/>
 <wire x1="162.56" y1="66.04" x2="165.1" y2="66.04" width="0.1524" layer="91"/>
@@
 <segment>
 <pinref part="R9" gate="G$1" pin="1"/>
-<pinref part="U$1" gate="G$1" pin="PGD"/>
+<pinref part="J3" gate="G$1" pin="PGD"/>
 <wire x1="162.56" y1="63.5" x2="165.1" y2="63.5" width="0.1524" layer="91"/>
 </segment>

Commit message: ...
Parts:
- IC1: device lc-meter:PIC16F876A-X/SP -> mcu:PIC16F876A-X/SP
- SW1: device lc-meter:PB-SPST -> mcu:PB-SPST
Changed lines of the file:
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@@
 </classes>
 <parts>
-<part name="IC1" library="lc-meter" deviceset="PIC16F876A-X/SP" device=""/>
+<part name="IC1" library="mcu" deviceset="PIC16F876A-X/SP" device=""/>
 <part name="R1" library="r" deviceset="R" device="0202/7" value="100kΩ"/>
 <part name="R2" library="r" deviceset="R" device="0202/7" value="100kΩ"/>
@@
 <part name="P+5" library="supply1" deviceset="VCC" device=""/>
 <part name="GND14" library="supply1" deviceset="GND" device=""/>
-<part name="SW1" library="lc-meter" deviceset="PB-SPST" device="" value="SPST"/>
+<part name="SW1" library="mcu" deviceset="PB-SPST" device="" value="SPST"/>
 <part name="K2" library="relay" deviceset="DS2Y-S-DC*" device="" technology="5V" value="DS2Y"/>
 <part name="P+6" library="supply1" deviceset="VCC" device=""/>
