File: eagle/LCmeter0-hd44780.sch (EAGLE design)
At the start: 26 parts, among them J1 22-27-2021-02, K1 DS2Y

Commit message: ...
Parts:
- removed U$4: S-DPDT, lc-meter:S-DPDT
- added S1: 9450-2, switch-misc:9450-2
Connections:
- net L/C: now also S12.S; no longer U$4.2-3
- net N$23: now also S11.O; no longer U$4.1-2
- net N$24: now also S11.S, S12.O; no longer U$4.1-3, U$4.2-2
- net N$5: now also S11.P; no longer U$4.1-1
- net N$8: now also S12.P; no longer U$4.2-1

Commit message: ...
Parts:
- U$2: device lc-meter:PB-5-2 -> mcu:PB-5-2
- U$3: device lc-meter:PIC16F876A-X/SP-COMP-B -> mcu:PIC16F876A-X/SP-COMP-B
Changed lines of the file:
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@@
 <part name="LCD" library="con-lsta" deviceset="FE08-1" device=""/>
 <part name="GND12" library="supply1" deviceset="GND" device=""/>
-<part name="U$3" library="lc-meter" deviceset="PIC16F876A-X/SP-COMP-B" device=""/>
+<part name="U$3" library="mcu" deviceset="PIC16F876A-X/SP-COMP-B" device=""/>
 <part name="ICSP" library="con-lsta" deviceset="FE05-1" device=""/>
 <part name="GND6" library="supply1" deviceset="GND" device=""/>
@@
 <part name="C4" library="resistor" deviceset="C-EU" device="025-024X044"/>
 <part name="C5" library="rcl" deviceset="CPOL-US" device="E2,5-6E"/>
-<part name="U$2" library="lc-meter" deviceset="PB-5-2" device=""/>
+<part name="U$2" library="mcu" deviceset="PB-5-2" device=""/>
 <part name="J1" library="con-molex" deviceset="22-?-02" device="27-2021"/>
 <part name="S1" library="switch-misc" deviceset="9450-2" device=""/>

Commit message: ...
Parts:
- C4: value (none) -> C-EU025-024X044; device resistor:C-EU025-024X044 -> r:C-EU025-024X044
- D1: device diode:1N4148DO35-7 -> d:1N4148DO35-7
- Q1: value (none) -> CRYSTALHC49S; device crystal:CRYSTALHC49S -> q:CRYSTALHC49S
- T1: value (none) -> BC548-NPN-TO92-CBE; device transistor:BC548-NPN-TO92-CBE -> t:BC548-NPN-TO92-CBE
Changed lines of the file:
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@@
 <part name="GND3" library="supply1" deviceset="GND" device=""/>
 <part name="P+1" library="supply1" deviceset="+5V" device=""/>
-<part name="Q1" library="crystal" deviceset="CRYSTAL" device="HC49S"/>
+<part name="Q1" library="q" deviceset="CRYSTAL" device="HC49S"/>
 <part name="GND4" library="supply1" deviceset="GND" device=""/>
 <part name="GND5" library="supply1" deviceset="GND" device=""/>
@@
 <part name="P+3" library="supply1" deviceset="+5V" device=""/>
 <part name="GND7" library="supply1" deviceset="GND" device=""/>
-<part name="D1" library="diode" deviceset="1N4148" device="DO35-7" value="1N4148"/>
-<part name="T1" library="transistor" deviceset="*-NPN-" device="TO92-CBE" technology="BC548"/>
+<part name="D1" library="d" deviceset="1N4148" device="DO35-7" value="1N4148"/>
+<part name="T1" library="t" deviceset="*-NPN-" device="TO92-CBE" technology="BC548"/>
 <part name="K1" library="relay" deviceset="DS2Y-S-DC*" device="" technology="5V" value="DS2Y"/>
 <part name="GND8" library="supply1" deviceset="GND" device=""/>
@@
 <part name="P+8" library="supply1" deviceset="+5V" device=""/>
 <part name="GND13" library="supply1" deviceset="GND" device=""/>
-<part name="C4" library="resistor" deviceset="C-EU" device="025-024X044"/>
+<part name="C4" library="r" deviceset="C-EU" device="025-024X044"/>
 <part name="C5" library="rcl" deviceset="CPOL-US" device="E2,5-6E"/>
 <part name="U$2" library="mcu" deviceset="PB-5-2" device=""/>
