File: eagle/LCmeter0-nokia3310.sch (EAGLE design)
At the start: 29 parts, among them K1 DS2Y

Commit message: ...
Parts:
- U$1: device lc-meter:PB-SPST -> mcu:PB-SPST
- U$2: device lc-meter:PIC16F876A-X/SP-COMP -> mcu:PIC16F876A-X/SP-COMP
- U$3: device lc-meter:NOKIA-3310-64X64 -> mcu:NOKIA-3310-64X64
- U$4: device lc-meter:S-DPDT -> mcu:S-DPDT
Changed lines of the file:
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@@
 </classes>
 <parts>
-<part name="U$2" library="lc-meter" deviceset="PIC16F876A-X/SP-COMP" device=""/>
+<part name="U$2" library="mcu" deviceset="PIC16F876A-X/SP-COMP" device=""/>
 <part name="R1" library="rcl" deviceset="R-EU_" device="0204/7" value="100k"/>
 <part name="R2" library="rcl" deviceset="R-EU_" device="0204/2V" value="100k"/>
@@
 <part name="C7" library="rcl" deviceset="C-EU" device="050-025X075" value="22pF"/>
 <part name="R11" library="rcl" deviceset="R-EU_" device="0204/2V" value="4.7k"/>
-<part name="U$1" library="lc-meter" deviceset="PB-SPST" device=""/>
+<part name="U$1" library="mcu" deviceset="PB-SPST" device=""/>
 <part name="GND1" library="supply1" deviceset="GND" device=""/>
 <part name="GND2" library="supply1" deviceset="GND" device=""/>
 <part name="GND3" library="supply1" deviceset="GND" device=""/>
-<part name="U$3" library="lc-meter" deviceset="NOKIA-3310-64X64" device=""/>
+<part name="U$3" library="mcu" deviceset="NOKIA-3310-64X64" device=""/>
 <part name="+3V1" library="supply1" deviceset="+3V3" device=""/>
 <part name="P+1" library="supply1" deviceset="+5V" device=""/>
@@
 <part name="GND10" library="supply1" deviceset="GND" device=""/>
 <part name="L2" library="rcl" deviceset="L-US" device="IR-2" value="100uH"/>
-<part name="U$4" library="lc-meter" deviceset="S-DPDT" device=""/>
+<part name="U$4" library="mcu" deviceset="S-DPDT" device=""/>
 <part name="GND11" library="supply1" deviceset="GND" device=""/>
 <part name="P+5" library="supply1" deviceset="+5V" device=""/>

Commit message: ...
Parts:
- D1: device diode:1N4148DO35-7 -> d:1N4148DO35-7
- Q1: value (none) -> CRYSTALHC49S; device crystal:CRYSTALHC49S -> q:CRYSTALHC49S
- T1: value (none) -> BC548-NPN-TO92-CBE; device transistor:BC548-NPN-TO92-CBE -> t:BC548-NPN-TO92-CBE
Changed lines of the file:
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@@
 <part name="+3V1" library="supply1" deviceset="+3V3" device=""/>
 <part name="P+1" library="supply1" deviceset="+5V" device=""/>
-<part name="Q1" library="crystal" deviceset="CRYSTAL" device="HC49S"/>
+<part name="Q1" library="q" deviceset="CRYSTAL" device="HC49S"/>
 <part name="GND4" library="supply1" deviceset="GND" device=""/>
 <part name="GND5" library="supply1" deviceset="GND" device=""/>
@@
 <part name="P+3" library="supply1" deviceset="+5V" device=""/>
 <part name="GND7" library="supply1" deviceset="GND" device=""/>
-<part name="D1" library="diode" deviceset="1N4148" device="DO35-7" value="1N4148"/>
-<part name="T1" library="transistor" deviceset="*-NPN-" device="TO92-CBE" technology="BC548"/>
+<part name="D1" library="d" deviceset="1N4148" device="DO35-7" value="1N4148"/>
+<part name="T1" library="t" deviceset="*-NPN-" device="TO92-CBE" technology="BC548"/>
 <part name="K1" library="relay" deviceset="DS2Y-S-DC*" device="" technology="5V" value="DS2Y"/>
 <part name="GND8" library="supply1" deviceset="GND" device=""/>
