File: eagle/LCmeter0-perfboard-new.sch (EAGLE design)
At the start: 25 parts, among them IC1 PIC16F876A-X/SP, K2 DS2Y, Q1 20MHz, Q2 BC548, SW1 SPST, SW2 DPDT

Commit message: ...
Parts:
- IC1: device lc-meter:PIC16F876A-X/SP -> mcu:PIC16F876A-X/SP
- SW1: device lc-meter:PB-SPST -> mcu:PB-SPST
- SW2: device lc-meter:S-DPDT -> mcu:S-DPDT
Changed lines of the file:
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@@
 </classes>
 <parts>
-<part name="IC1" library="lc-meter" deviceset="PIC16F876A-X/SP" device=""/>
+<part name="IC1" library="mcu" deviceset="PIC16F876A-X/SP" device=""/>
 <part name="R1" library="rcl" deviceset="R-EU_" device="0204/7" value="100kΩ"/>
 <part name="R2" library="resistor" deviceset="R-EU_" device="0204/2V" value="100kΩ"/>
@@
 <part name="P+5" library="supply1" deviceset="VCC" device=""/>
 <part name="GND14" library="supply1" deviceset="GND" device=""/>
-<part name="SW2" library="lc-meter" deviceset="S-DPDT" device="" value="DPDT"/>
-<part name="SW1" library="lc-meter" deviceset="PB-SPST" device="" value="SPST"/>
+<part name="SW2" library="mcu" deviceset="S-DPDT" device="" value="DPDT"/>
+<part name="SW1" library="mcu" deviceset="PB-SPST" device="" value="SPST"/>
 <part name="K2" library="relay" deviceset="DS2Y-S-DC*" device="" technology="5V" value="DS2Y"/>
 <part name="P+6" library="supply1" deviceset="VCC" device=""/>

Commit message: ...
Parts:
- D1: device diode:1N4148DO35-7 -> d:1N4148DO35-7
- Q1: device crystal:CRYSTALHC49S -> q:CRYSTALHC49S
- Q2: device transistor-npn:BC548 -> t:BC548
- R10, R5: device resistor:R-EU_0207/10 -> r:R-EU_0207/10
- R2, R3, R4, R6: device resistor:R-EU_0204/2V -> r:R-EU_0204/2V
Changed lines of the file:
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@@
 <part name="IC1" library="mcu" deviceset="PIC16F876A-X/SP" device=""/>
 <part name="R1" library="rcl" deviceset="R-EU_" device="0204/7" value="100kΩ"/>
-<part name="R2" library="resistor" deviceset="R-EU_" device="0204/2V" value="100kΩ"/>
-<part name="R3" library="resistor" deviceset="R-EU_" device="0204/2V" value="100kΩ"/>
-<part name="R4" library="resistor" deviceset="R-EU_" device="0204/2V" value="47kΩ"/>
-<part name="R10" library="resistor" deviceset="R-EU_" device="0207/10" value="4.7kΩ"/>
+<part name="R2" library="r" deviceset="R-EU_" device="0204/2V" value="100kΩ"/>
+<part name="R3" library="r" deviceset="R-EU_" device="0204/2V" value="100kΩ"/>
+<part name="R4" library="r" deviceset="R-EU_" device="0204/2V" value="47kΩ"/>
+<part name="R10" library="r" deviceset="R-EU_" device="0207/10" value="4.7kΩ"/>
 <part name="C1" library="rcl" deviceset="C-EU" device="050-024X044" value="1nF"/>
 <part name="C2" library="rcl" deviceset="C-EU" device="050-024X044" value="1nF"/>
@@
 <part name="GND6" library="supply1" deviceset="GND" device=""/>
 <part name="GND7" library="supply1" deviceset="GND" device=""/>
-<part name="D1" library="diode" deviceset="1N4148" device="DO35-7" value="1N4148"/>
+<part name="D1" library="d" deviceset="1N4148" device="DO35-7" value="1N4148"/>
 <part name="L1" library="rcl" deviceset="L-US" device="0204/5" value="100μH"/>
-<part name="Q1" library="crystal" deviceset="CRYSTAL" device="HC49S" value="20MHz"/>
+<part name="Q1" library="q" deviceset="CRYSTAL" device="HC49S" value="20MHz"/>
 <part name="P+1" library="supply1" deviceset="VCC" device=""/>
 <part name="GND11" library="supply1" deviceset="GND" device=""/>
@@
 <part name="P+4" library="supply1" deviceset="VCC" device=""/>
 <part name="GND12" library="supply1" deviceset="GND" device=""/>
-<part name="R5" library="resistor" deviceset="R-EU_" device="0207/10" value="4.7kΩ"/>
+<part name="R5" library="r" deviceset="R-EU_" device="0207/10" value="4.7kΩ"/>
 <part name="P+5" library="supply1" deviceset="VCC" device=""/>
 <part name="GND14" library="supply1" deviceset="GND" device=""/>
@@
 <part name="K2" library="relay" deviceset="DS2Y-S-DC*" device="" technology="5V" value="DS2Y"/>
 <part name="P+6" library="supply1" deviceset="VCC" device=""/>
-<part name="Q2" library="transistor-npn" deviceset="BC548*" device=""/>
+<part name="Q2" library="t" deviceset="BC548*" device=""/>
 <part name="GND8" library="supply1" deviceset="GND" device=""/>
-<part name="R6" library="resistor" deviceset="R-EU_" device="0204/2V" value="10kΩ"/>
+<part name="R6" library="r" deviceset="R-EU_" device="0204/2V" value="10kΩ"/>
 <part name="LCD1" library="con-lstb" deviceset="MA08-1" device="" value="HD44780"/>
 <part name="P+7" library="supply1" deviceset="VCC" device=""/>
