File: eagle/LCmeter0-perfboard2.brd (EAGLE design)
At the start: 51.1 x 49.5 mm, 25 parts, among them IC1 PIC16F876A-X/SP, K2 DS2Y, Q1 20MHz, Q2 BC548, SW1 SPST, SW2 DPDT

Commit message: ...
Parts:
- IC1: device lc-meter:DIL28-3 -> mcu:DIL28-3
- SW1: device lc-meter:PB-5 -> mcu:PB-5
- SW2: device lc-meter:DPDT -> mcu:DPDT
Changed lines of the file:
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@@
 </element>
 <element name="D1" library="diode" package="DO35-7" value="1N4148" x="8.89" y="2.54" rot="R180"/>
-<element name="IC1" library="lc-meter" package="DIL28-3" value="PIC16F876A-X/SP" x="31.75" y="24.13" rot="R270"/>
+<element name="IC1" library="mcu" package="DIL28-3" value="PIC16F876A-X/SP" x="31.75" y="24.13" rot="R270"/>
 <element name="L1" library="rcl" package="0204/5" value="100μH" x="-5.08" y="35.56" rot="R90"/>
 <element name="Q1" library="crystal" package="HC49/S" value="20MHz" x="22.86" y="20.32" rot="R270">
@@
 <element name="R4" library="resistor" package="0204V" value="47kΩ" x="25.4" y="36.83" rot="R90"/>
 <element name="R5" library="rcl" package="0204/7" value="4.7kΩ" x="21.59" y="27.94" rot="R180"/>
-<element name="SW2" library="lc-meter" package="DPDT" value="DPDT" x="-1.27" y="25.4" rot="R90"/>
-<element name="SW1" library="lc-meter" package="PB-5" value="SPST" x="-2.54" y="10.16"/>
+<element name="SW2" library="mcu" package="DPDT" value="DPDT" x="-1.27" y="25.4" rot="R90"/>
+<element name="SW1" library="mcu" package="PB-5" value="SPST" x="-2.54" y="10.16"/>
 <element name="K2" library="relay" package="DS2Y" value="DS2Y" x="6.35" y="13.97" rot="R90">
 <attribute name="OC_NEWARK" value="13P3268" x="6.35" y="13.97" size="1.778" layer="27" rot="R90" display="off"/>

Commit message: ...
Parts:
- D1: device diode:DO35-7 -> d:DO35-7
- Q1: device crystal:HC49/S -> q:HC49/S
- Q2: device transistor-npn:TO92-EBC -> t:TO92-EBC
- R10: device resistor:0207/10 -> r:0207/10
- R2, R3, R4: device resistor:0204V -> r:0204V
Changed lines of the file:
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@@
 <attribute name="VALUE" x="35.433" y="20.828" size="1.27" layer="27" ratio="10" rot="R270"/>
 </element>
-<element name="D1" library="diode" package="DO35-7" value="1N4148" x="8.89" y="2.54" rot="R180"/>
+<element name="D1" library="d" package="DO35-7" value="1N4148" x="8.89" y="2.54" rot="R180"/>
 <element name="IC1" library="mcu" package="DIL28-3" value="PIC16F876A-X/SP" x="31.75" y="24.13" rot="R270"/>
 <element name="L1" library="rcl" package="0204/5" value="100μH" x="-5.08" y="35.56" rot="R90"/>
-<element name="Q1" library="crystal" package="HC49/S" value="20MHz" x="22.86" y="20.32" rot="R270">
+<element name="Q1" library="q" package="HC49/S" value="20MHz" x="22.86" y="20.32" rot="R270">
 <attribute name="OC_NEWARK" value="unknown" x="22.86" y="20.32" size="1.778" layer="27" rot="R270" display="off"/>
 <attribute name="MPN" value="" x="22.86" y="20.32" size="1.778" layer="27" rot="R270" display="off"/>
@@
 </element>
 <element name="R1" library="rcl" package="0204/7" value="100kΩ" x="16.51" y="38.1"/>
-<element name="R10" library="resistor" package="0207/10" value="4.7kΩ" x="20.32" y="40.64" smashed="yes" rot="R180">
+<element name="R10" library="r" package="0207/10" value="4.7kΩ" x="20.32" y="40.64" smashed="yes" rot="R180">
 <attribute name="NAME" x="22.4536" y="39.4716" size="1.27" layer="25" ratio="10" rot="R180"/>
 <attribute name="VALUE" x="22.4536" y="42.9514" size="1.27" layer="27" ratio="10" rot="R180"/>
 </element>
-<element name="R2" library="resistor" package="0204V" value="100kΩ" x="12.7" y="34.29" rot="R90"/>
-<element name="R3" library="resistor" package="0204V" value="100kΩ" x="12.7" y="41.91" rot="R90"/>
-<element name="R4" library="resistor" package="0204V" value="47kΩ" x="25.4" y="36.83" rot="R90"/>
+<element name="R2" library="r" package="0204V" value="100kΩ" x="12.7" y="34.29" rot="R90"/>
+<element name="R3" library="r" package="0204V" value="100kΩ" x="12.7" y="41.91" rot="R90"/>
+<element name="R4" library="r" package="0204V" value="47kΩ" x="25.4" y="36.83" rot="R90"/>
 <element name="R5" library="rcl" package="0204/7" value="4.7kΩ" x="21.59" y="27.94" rot="R180"/>
 <element name="SW2" library="mcu" package="DPDT" value="DPDT" x="-1.27" y="25.4" rot="R90"/>
@@
 <attribute name="OC_FARNELL" value="unknown" x="6.35" y="13.97" size="1.778" layer="27" rot="R90" display="off"/>
 </element>
-<element name="Q2" library="transistor-npn" package="TO92-EBC" value="BC548" x="16.51" y="5.08" rot="R90"/>
+<element name="Q2" library="t" package="TO92-EBC" value="BC548" x="16.51" y="5.08" rot="R90"/>
 <element name="R6" library="rcl" package="0207/10" value="10kΩ" x="25.4" y="5.08" rot="R180"/>
 <element name="LCD1" library="con-lstb" package="MA08-1" value="HD44780" x="43.18" y="31.75" rot="R90">
