File: eagle/LCmeter0.brd (EAGLE design)
At the start: 63.5 x 50.5 mm, 25 parts, among them IC1 PIC16F876A-X/SP, K2 DS2Y, Q1 20MHz, Q2 BC548, SW1 SPST

Commit message: ...
Parts:
- IC1: device lc-meter:DIL28-3 -> mcu:DIL28-3
- SW1: device lc-meter:PB-5 -> mcu:PB-5
Changed lines of the file:
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@@
 </element>
 <element name="D1" library="diode" package="DO35-7" value="1N4148" x="27.94" y="8.89" rot="R90"/>
-<element name="IC1" library="lc-meter" package="DIL28-3" value="PIC16F876A-X/SP" x="44.45" y="26.67" rot="R270"/>
+<element name="IC1" library="mcu" package="DIL28-3" value="PIC16F876A-X/SP" x="44.45" y="26.67" rot="R270"/>
 <element name="L1" library="rcl" package="0207/10" value="100μH" x="17.78" y="30.48" rot="R90"/>
 <element name="Q1" library="crystal" package="HC49U70" value="20MHz" x="33.02" y="20.32">
@@
 <attribute name="VALUE" x="36.195" y="42.1894" size="1.27" layer="27" ratio="10" rot="R90"/>
 </element>
-<element name="SW1" library="lc-meter" package="PB-5" value="SPST" x="10.16" y="40.64"/>
+<element name="SW1" library="mcu" package="PB-5" value="SPST" x="10.16" y="40.64"/>
 <element name="K2" library="relay" package="DS2Y" value="DS2Y" x="21.59" y="13.97" rot="R90">
 <attribute name="OC_NEWARK" value="13P3268" x="21.59" y="13.97" size="1.778" layer="27" rot="R90" display="off"/>

Commit message: ...
Parts:
- D1: device diode:DO35-7 -> d:DO35-7
- Q1: device crystal:HC49U70 -> q:HC49U70
- Q2: device transistor-npn:TO92-EBC -> t:TO92-EBC
- R1, R2, R4: device resistor:0207/10 -> r:0207/10
- R10, R3, R5: device resistor:0204V -> r:0204V
Changed lines of the file:
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@@
 <attribute name="VALUE" x="55.753" y="23.368" size="1.27" layer="27" ratio="10" rot="R270"/>
 </element>
-<element name="D1" library="diode" package="DO35-7" value="1N4148" x="27.94" y="8.89" rot="R90"/>
+<element name="D1" library="d" package="DO35-7" value="1N4148" x="27.94" y="8.89" rot="R90"/>
 <element name="IC1" library="mcu" package="DIL28-3" value="PIC16F876A-X/SP" x="44.45" y="26.67" rot="R270"/>
 <element name="L1" library="rcl" package="0207/10" value="100μH" x="17.78" y="30.48" rot="R90"/>
-<element name="Q1" library="crystal" package="HC49U70" value="20MHz" x="33.02" y="20.32">
+<element name="Q1" library="q" package="HC49U70" value="20MHz" x="33.02" y="20.32">
 <attribute name="OC_NEWARK" value="unknown" x="33.02" y="20.32" size="1.778" layer="27" display="off"/>
 <attribute name="MPN" value="" x="33.02" y="20.32" size="1.778" layer="27" display="off"/>
@@
 <attribute name="OC_FARNELL" value="unknown" x="33.02" y="20.32" size="1.778" layer="27" display="off"/>
 </element>
-<element name="R1" library="resistor" package="0207/10" value="100kΩ" x="30.48" y="40.64" smashed="yes">
+<element name="R1" library="r" package="0207/10" value="100kΩ" x="30.48" y="40.64" smashed="yes">
 <attribute name="NAME" x="30.48" y="40.64" size="1.27" layer="25" ratio="10" align="center"/>
 <attribute name="VALUE" x="28.2194" y="40.005" size="1.27" layer="27" ratio="10"/>
 </element>
-<element name="R10" library="resistor" package="0204V" value="4.7kΩ" x="38.1" y="44.45" smashed="yes" rot="R90">
+<element name="R10" library="r" package="0204V" value="4.7kΩ" x="38.1" y="44.45" smashed="yes" rot="R90">
 <attribute name="NAME" x="38.1" y="45.72" size="1.27" layer="25" ratio="10" rot="R90" align="center"/>
 <attribute name="VALUE" x="38.735" y="42.1894" size="1.27" layer="27" ratio="10" rot="R90"/>
 </element>
-<element name="R2" library="resistor" package="0207/10" value="100kΩ" x="25.4" y="33.02" smashed="yes" rot="R90">
+<element name="R2" library="r" package="0207/10" value="100kΩ" x="25.4" y="33.02" smashed="yes" rot="R90">
 <attribute name="NAME" x="25.4" y="33.02" size="1.27" layer="25" ratio="10" rot="R90" align="center"/>
 <attribute name="VALUE" x="26.035" y="30.7594" size="1.27" layer="27" ratio="10" rot="R90"/>
 </element>
-<element name="R3" library="resistor" package="0204V" value="100kΩ" x="25.4" y="44.45" smashed="yes" rot="R90">
+<element name="R3" library="r" package="0204V" value="100kΩ" x="25.4" y="44.45" smashed="yes" rot="R90">
 <attribute name="NAME" x="25.4" y="45.72" size="1.27" layer="25" ratio="10" rot="R90" align="center"/>
 <attribute name="VALUE" x="26.035" y="42.1894" size="1.27" layer="27" ratio="10" rot="R90"/>
 </element>
-<element name="R4" library="resistor" package="0207/10" value="47kΩ" x="35.56" y="33.02" smashed="yes" rot="R90">
+<element name="R4" library="r" package="0207/10" value="47kΩ" x="35.56" y="33.02" smashed="yes" rot="R90">
 <attribute name="NAME" x="35.56" y="33.02" size="1.27" layer="25" ratio="10" rot="R90" align="center"/>
 <attribute name="VALUE" x="36.195" y="30.7594" size="1.27" layer="27" ratio="10" rot="R90"/>
 </element>
-<element name="R5" library="resistor" package="0204V" value="4.7kΩ" x="35.56" y="44.45" smashed="yes" rot="R90">
+<element name="R5" library="r" package="0204V" value="4.7kΩ" x="35.56" y="44.45" smashed="yes" rot="R90">
 <attribute name="NAME" x="35.56" y="46.355" size="1.27" layer="25" ratio="10" rot="R90" align="center"/>
 <attribute name="VALUE" x="36.195" y="42.1894" size="1.27" layer="27" ratio="10" rot="R90"/>
@@
 <attribute name="OC_FARNELL" value="unknown" x="21.59" y="13.97" size="1.778" layer="27" rot="R90" display="off"/>
 </element>
-<element name="Q2" library="transistor-npn" package="TO92-EBC" value="BC548" x="54.61" y="7.62" rot="R180"/>
+<element name="Q2" library="t" package="TO92-EBC" value="BC548" x="54.61" y="7.62" rot="R180"/>
 <element name="R6" library="rcl" package="0207/10" value="" x="55.88" y="12.7"/>
 <element name="CON1" library="con-lstb" package="MA07-2" value="" x="57.15" y="35.56" rot="R90">
