File: eagle/LCmeter0.sch (EAGLE design)
At the start: 25 parts, among them IC1 PIC16F876A-X/SP, K2 DS2Y, Q1 20MHz, Q2 BC548, SW1 SPST, SW2 DPDT

Commit message: ...
Parts:
- removed SV1: DIL-12, con-lsta:FE12-1
- added CON1: (no value), con-lstb:MA07-2
Connections:
- removed net B0: IC1.RB0/INT, SV1.8
- removed net B1: IC1.RB1, SV1.7
- net B2: now also CON1.4; no longer SV1.6
- net B3: now also CON1.6; no longer SV1.5
- net B4: now also CON1.11; no longer SV1.4
- net B5: now also CON1.12; no longer SV1.3
- net B6: now also CON1.13; no longer SV1.2
- net B7: now also CON1.14; no longer SV1.1
- net N$3: now also CON1.2; no longer SV1.9
- net RX: no longer SV1.11
- net TX: no longer SV1.12
- net VSS: now also CON1.1, CON1.5; no longer SV1.10

Commit message: ...
Parts:
- removed SW2: DPDT, lc-meter:S-DPDT
- added S1: TL46PO, switch:TL46PO
Connections:
- net /LC: now also S1.S1; no longer SW2.2-3
- net N$2: now also S1.O; no longer SW2.1-2
- net N$7: now also S1.O1, S1.S; no longer SW2.1-3, SW2.2-2
Changed lines of the file:
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@@
 <setting verticaltext="up"/>
 </settings>
-<grid distance="0.05" unitdist="inch" unit="inch" style="lines" multiple="2" display="no" altdistance="0.025" altunitdist="inch" altunit="inch"/>
+<grid distance="0.05" unitdist="inch" unit="inch" style="lines" multiple="2" display="no" altdistance="0.01" altunitdist="inch" altunit="inch"/>
 <layers>
 <layer number="1" name="Top" color="4" fill="1" visible="yes" active="no"/>
@@
 <part name="P+5" library="supply1" deviceset="VCC" device=""/>
 <part name="GND14" library="supply1" deviceset="GND" device=""/>
-<part name="SW2" library="lc-meter" deviceset="S-DPDT" device="" value="DPDT"/>
 <part name="SW1" library="lc-meter" deviceset="PB-SPST" device="" value="SPST"/>
 <part name="K2" library="relay" deviceset="DS2Y-S-DC*" device="" technology="5V" value="DS2Y"/>
@@
 <part name="R6" library="rcl" deviceset="R-EU_" device="0207/10"/>
 <part name="CON1" library="con-lstb" deviceset="MA07-2" device=""/>
+<part name="S1" library="switch" deviceset="TL46PO" device=""/>
 </parts>
 <sheets>
@@
 </instance>
 <instance part="GND14" gate="1" x="153.67" y="-7.62"/>
-<instance part="SW2" gate="G$1" x="-46.99" y="27.94" smashed="yes" rot="R270">
-<attribute name="NAME" x="-52.705" y="13.97" size="1.778" layer="95"/>
-<attribute name="VALUE" x="-52.705" y="11.43" size="1.778" layer="96"/>
-</instance>
 <instance part="SW1" gate="G$1" x="139.7" y="1.27" smashed="yes">
 <attribute name="NAME" x="143.51" y="1.27" size="1.778" layer="95" rot="R90" align="top-center"/>
@@
 <instance part="R6" gate="G$1" x="114.3" y="2.54"/>
 <instance part="CON1" gate="G$1" x="187.96" y="31.75"/>
+<instance part="S1" gate="BEF1" x="-53.34" y="27.94" rot="R270"/>
 </instances>
 <busses>
@@
 <wire x1="-11.43" y1="30.48" x2="-8.89" y2="30.48" width="0.1524" layer="91"/>
 <junction x="-11.43" y="30.48"/>
-<pinref part="SW2" gate="G$1" pin="1-2"/>
-<wire x1="-41.91" y1="30.48" x2="-19.05" y2="30.48" width="0.1524" layer="91"/>
+<wire x1="-48.26" y1="30.48" x2="-19.05" y2="30.48" width="0.1524" layer="91"/>
 <junction x="-19.05" y="30.48"/>
 <junction x="-19.05" y="25.4"/>
+<pinref part="S1" gate="BEF1" pin="O"/>
 </segment>
 </net>
@@
 <pinref part="L1" gate="G$1" pin="1"/>
 <wire x1="-36.83" y1="25.4" x2="-39.37" y2="25.4" width="0.1524" layer="91"/>
-<pinref part="SW2" gate="G$1" pin="1-3"/>
-<wire x1="-41.91" y1="25.4" x2="-39.37" y2="25.4" width="0.1524" layer="91"/>
+<wire x1="-48.26" y1="25.4" x2="-39.37" y2="25.4" width="0.1524" layer="91"/>
 <junction x="-39.37" y="25.4"/>
-<pinref part="SW2" gate="G$1" pin="2-2"/>
-<wire x1="-41.91" y1="20.32" x2="-39.37" y2="20.32" width="0.1524" layer="91"/>
+<wire x1="-48.26" y1="20.32" x2="-39.37" y2="20.32" width="0.1524" layer="91"/>
+<pinref part="S1" gate="BEF1" pin="S"/>
+<pinref part="S1" gate="BEF1" pin="O1"/>
 </segment>
 </net>
@@
 <net name="/LC" class="0">
 <segment>
-<pinref part="SW2" gate="G$1" pin="2-3"/>
-<wire x1="-41.91" y1="15.24" x2="-35.56" y2="15.24" width="0.1524" layer="91"/>
+<wire x1="-48.26" y1="15.24" x2="-35.56" y2="15.24" width="0.1524" layer="91"/>
 <label x="-40.64" y="15.24" size="1.778" layer="95"/>
-</segment>
-<segment>
+<pinref part="S1" gate="BEF1" pin="S1"/>
+</segment>
+<segment>

Commit message: ...
Parts:
- IC1: device lc-meter:PIC16F876A-X/SP -> mcu:PIC16F876A-X/SP
- SW1: device lc-meter:PB-SPST -> mcu:PB-SPST
Changed lines of the file:
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@@
 </classes>
 <parts>
-<part name="IC1" library="lc-meter" deviceset="PIC16F876A-X/SP" device=""/>
+<part name="IC1" library="mcu" deviceset="PIC16F876A-X/SP" device=""/>
 <part name="R1" library="resistor" deviceset="R-EU_" device="0207/10" value="100kΩ"/>
 <part name="R2" library="resistor" deviceset="R-EU_" device="0207/10" value="100kΩ"/>
@@
 <part name="P+5" library="supply1" deviceset="VCC" device=""/>
 <part name="GND14" library="supply1" deviceset="GND" device=""/>
-<part name="SW1" library="lc-meter" deviceset="PB-SPST" device="" value="SPST"/>
+<part name="SW1" library="mcu" deviceset="PB-SPST" device="" value="SPST"/>
 <part name="K2" library="relay" deviceset="DS2Y-S-DC*" device="" technology="5V" value="DS2Y"/>
 <part name="P+6" library="supply1" deviceset="VCC" device=""/>

Commit message: ...
Parts:
- D1: device diode:1N4148DO35-7 -> d:1N4148DO35-7
- Q1: device crystal:CRYSTALHC49U70 -> q:CRYSTALHC49U70
- Q2: device transistor-npn:BC548 -> t:BC548
- R1, R2, R4: device resistor:R-EU_0207/10 -> r:R-EU_0207/10
- R10, R3, R5: device resistor:R-EU_0204/2V -> r:R-EU_0204/2V
Changed lines of the file:
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@@
 <parts>
 <part name="IC1" library="mcu" deviceset="PIC16F876A-X/SP" device=""/>
-<part name="R1" library="resistor" deviceset="R-EU_" device="0207/10" value="100kΩ"/>
-<part name="R2" library="resistor" deviceset="R-EU_" device="0207/10" value="100kΩ"/>
-<part name="R3" library="resistor" deviceset="R-EU_" device="0204/2V" value="100kΩ"/>
-<part name="R4" library="resistor" deviceset="R-EU_" device="0207/10" value="47kΩ"/>
-<part name="R10" library="resistor" deviceset="R-EU_" device="0204/2V" value="4.7kΩ"/>
+<part name="R1" library="r" deviceset="R-EU_" device="0207/10" value="100kΩ"/>
+<part name="R2" library="r" deviceset="R-EU_" device="0207/10" value="100kΩ"/>
+<part name="R3" library="r" deviceset="R-EU_" device="0204/2V" value="100kΩ"/>
+<part name="R4" library="r" deviceset="R-EU_" device="0207/10" value="47kΩ"/>
+<part name="R10" library="r" deviceset="R-EU_" device="0204/2V" value="4.7kΩ"/>
 <part name="C1" library="rcl" deviceset="C-EU" device="050-025X075" value="1nF"/>
 <part name="C2" library="rcl" deviceset="C-EU" device="050-025X075" value="1nF"/>
@@
 <part name="GND6" library="supply1" deviceset="GND" device=""/>
 <part name="GND7" library="supply1" deviceset="GND" device=""/>
-<part name="D1" library="diode" deviceset="1N4148" device="DO35-7" value="1N4148"/>
+<part name="D1" library="d" deviceset="1N4148" device="DO35-7" value="1N4148"/>
 <part name="L1" library="rcl" deviceset="L-US" device="0207/10" value="100μH"/>
-<part name="Q1" library="crystal" deviceset="CRYSTAL" device="HC49U70" value="20MHz"/>
+<part name="Q1" library="q" deviceset="CRYSTAL" device="HC49U70" value="20MHz"/>
 <part name="P+1" library="supply1" deviceset="VCC" device=""/>
 <part name="GND11" library="supply1" deviceset="GND" device=""/>
@@
 <part name="P+4" library="supply1" deviceset="VCC" device=""/>
 <part name="GND12" library="supply1" deviceset="GND" device=""/>
-<part name="R5" library="resistor" deviceset="R-EU_" device="0204/2V" value="4.7kΩ"/>
+<part name="R5" library="r" deviceset="R-EU_" device="0204/2V" value="4.7kΩ"/>
 <part name="P+5" library="supply1" deviceset="VCC" device=""/>
 <part name="GND14" library="supply1" deviceset="GND" device=""/>
@@
 <part name="K2" library="relay" deviceset="DS2Y-S-DC*" device="" technology="5V" value="DS2Y"/>
 <part name="P+6" library="supply1" deviceset="VCC" device=""/>
-<part name="Q2" library="transistor-npn" deviceset="BC548*" device=""/>
+<part name="Q2" library="t" deviceset="BC548*" device=""/>
 <part name="GND8" library="supply1" deviceset="GND" device=""/>
 <part name="R6" library="rcl" deviceset="R-EU_" device="0207/10"/>
