File: eagle/LCmeter0-perfboard.brd (EAGLE design)
At the start: 48.6 x 49.5 mm, 25 parts, among them IC1 PIC16F876A-X/SP, K2 DS2Y, Q1 20MHz, Q2 BC548, SW1 SPST, SW2 DPDT

Commit message: ...
Parts:
- IC1: device lc-meter:DIL28-3 -> mcu:DIL28-3
- SW1: device lc-meter:PB-5 -> mcu:PB-5
- SW2: device lc-meter:DPDT -> mcu:DPDT
Changed lines of the file:
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@@
 </element>
 <element name="D1" library="diode" package="DO35-7" value="1N4148" x="8.89" y="2.54" rot="R180"/>
-<element name="IC1" library="lc-meter" package="DIL28-3" value="PIC16F876A-X/SP" x="31.75" y="26.67" rot="R270"/>
+<element name="IC1" library="mcu" package="DIL28-3" value="PIC16F876A-X/SP" x="31.75" y="26.67" rot="R270"/>
 <element name="L1" library="rcl" package="0204/5" value="100μH" x="12.7" y="35.56"/>
 <element name="Q1" library="crystal" package="HC49/S" value="20MHz" x="22.86" y="20.32" rot="R270">
@@
 <attribute name="VALUE" x="26.035" y="44.7294" size="1.27" layer="27" ratio="10" rot="R90"/>
 </element>
-<element name="SW2" library="lc-meter" package="DPDT" value="DPDT" x="6.35" y="33.02" rot="R90"/>
-<element name="SW1" library="lc-meter" package="PB-5" value="SPST" x="7.62" y="43.18"/>
+<element name="SW2" library="mcu" package="DPDT" value="DPDT" x="6.35" y="33.02" rot="R90"/>
+<element name="SW1" library="mcu" package="PB-5" value="SPST" x="7.62" y="43.18"/>
 <element name="K2" library="relay" package="DS2Y" value="DS2Y" x="6.35" y="13.97" rot="R90">
 <attribute name="OC_NEWARK" value="13P3268" x="6.35" y="13.97" size="1.778" layer="27" rot="R90" display="off"/>

Commit message: ...
Parts:
- D1: device diode:DO35-7 -> d:DO35-7
- Q1: device crystal:HC49/S -> q:HC49/S
- Q2: device transistor-npn:TO92-EBC -> t:TO92-EBC
- R1, R10, R2, R3, R4, R5: device resistor:0204V -> r:0204V
Changed lines of the file:
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@@
 <attribute name="VALUE" x="43.053" y="20.828" size="1.27" layer="27" ratio="10" rot="R270"/>
 </element>
-<element name="D1" library="diode" package="DO35-7" value="1N4148" x="8.89" y="2.54" rot="R180"/>
+<element name="D1" library="d" package="DO35-7" value="1N4148" x="8.89" y="2.54" rot="R180"/>
 <element name="IC1" library="mcu" package="DIL28-3" value="PIC16F876A-X/SP" x="31.75" y="26.67" rot="R270"/>
 <element name="L1" library="rcl" package="0204/5" value="100μH" x="12.7" y="35.56"/>
-<element name="Q1" library="crystal" package="HC49/S" value="20MHz" x="22.86" y="20.32" rot="R270">
+<element name="Q1" library="q" package="HC49/S" value="20MHz" x="22.86" y="20.32" rot="R270">
 <attribute name="OC_NEWARK" value="unknown" x="22.86" y="20.32" size="1.778" layer="27" rot="R270" display="off"/>
 <attribute name="MPN" value="" x="22.86" y="20.32" size="1.778" layer="27" rot="R270" display="off"/>
@@
 <attribute name="OC_FARNELL" value="1667008" x="22.86" y="20.32" size="1.778" layer="27" rot="R270" display="off"/>
 </element>
-<element name="R1" library="resistor" package="0204V" value="100kΩ" x="20.32" y="41.91" rot="R270"/>
-<element name="R10" library="resistor" package="0204V" value="4.7kΩ" x="12.7" y="46.99" smashed="yes" rot="R90">
+<element name="R1" library="r" package="0204V" value="100kΩ" x="20.32" y="41.91" rot="R270"/>
+<element name="R10" library="r" package="0204V" value="4.7kΩ" x="12.7" y="46.99" smashed="yes" rot="R90">
 <attribute name="NAME" x="12.7" y="48.26" size="1.27" layer="25" ratio="10" rot="R90" align="center"/>
 <attribute name="VALUE" x="13.335" y="44.7294" size="1.27" layer="27" ratio="10" rot="R90"/>
 </element>
-<element name="R2" library="resistor" package="0204V" value="100kΩ" x="20.32" y="31.75" rot="R90"/>
-<element name="R3" library="resistor" package="0204V" value="100kΩ" x="20.32" y="46.99" smashed="yes" rot="MR90">
+<element name="R2" library="r" package="0204V" value="100kΩ" x="20.32" y="31.75" rot="R90"/>
+<element name="R3" library="r" package="0204V" value="100kΩ" x="20.32" y="46.99" smashed="yes" rot="MR90">
 <attribute name="NAME" x="20.32" y="48.26" size="1.27" layer="26" ratio="10" rot="MR90" align="center"/>
 <attribute name="VALUE" x="19.685" y="44.7294" size="1.27" layer="28" ratio="10" rot="MR90"/>
 </element>
-<element name="R4" library="resistor" package="0204V" value="47kΩ" x="22.86" y="39.37" rot="R90"/>
-<element name="R5" library="resistor" package="0204V" value="4.7kΩ" x="25.4" y="46.99" smashed="yes" rot="R90">
+<element name="R4" library="r" package="0204V" value="47kΩ" x="22.86" y="39.37" rot="R90"/>
+<element name="R5" library="r" package="0204V" value="4.7kΩ" x="25.4" y="46.99" smashed="yes" rot="R90">
 <attribute name="NAME" x="25.4" y="48.895" size="1.27" layer="25" ratio="10" rot="R90" align="center"/>
 <attribute name="VALUE" x="26.035" y="44.7294" size="1.27" layer="27" ratio="10" rot="R90"/>
@@
 <attribute name="OC_FARNELL" value="unknown" x="6.35" y="13.97" size="1.778" layer="27" rot="R90" display="off"/>
 </element>
-<element name="Q2" library="transistor-npn" package="TO92-EBC" value="BC548" x="16.51" y="5.08" rot="R90"/>
+<element name="Q2" library="t" package="TO92-EBC" value="BC548" x="16.51" y="5.08" rot="R90"/>
 <element name="R6" library="rcl" package="0207/10" value="10kΩ" x="25.4" y="5.08" rot="R180"/>
 <element name="LCD1" library="con-lstb" package="MA08-1" value="HD44780" x="43.18" y="34.29" rot="R90">

Commit message: ...
Parts:
- D1: device d:DO35-7 -> diode:DO35-7
- IC1: device mcu:DIL28-3 -> lc-meter:DIL28-3
- Q1: device q:HC49/S -> crystal:HC49/S
- Q2: device t:TO92-EBC -> transistor-npn:TO92-EBC
- R1, R5: device r:0204V -> rcl:0204/7
- R10: device r:0204V -> resistor:0207/10
- R2, R3, R4: device r:0204V -> resistor:0204V
- SW1: device mcu:PB-5 -> lc-meter:PB-5
- SW2: device mcu:DPDT -> lc-meter:DPDT
- moved SW1 34.5 mm to (-2.54, 10.2)
- moved R5 19.4 mm to (21.6, 27.9), turned to 180 degrees
- moved L1 17.8 mm to (-5.08, 35.6), turned to 90 degrees
- moved C2 16.1 mm to (0.00, 35.6)
- moved C4 13.7 mm to (10.2, 27.9)
- moved C1 11.4 mm to (2.54, 35.6)
- moved SW2 10.8 mm to (-1.27, 25.4)
- moved C3 10.5 mm to (7.62, 38.1), turned to 180 degrees
- moved R10 9.92 mm to (20.3, 40.6), turned to 180 degrees
- moved R3 9.16 mm to (12.7, 41.9), flipped to the top
- moved R2 8.03 mm to (12.7, 34.3)
- moved C9 7.62 mm to (38.1, 19.1)
- moved R1 5.39 mm to (16.5, 38.1), turned to 0 degrees
- moved C7 5.08 mm to (41.9, 7.62)
- moved R4 3.59 mm to (25.4, 36.8)
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Routing:
- net A3: track 22.9 -> 0.00 mm
- net A4: track 17.1 -> 0.00 mm
- net OSC1: track 0.00 -> 11.3 mm
- net VCC: track 75.2 -> 64.2 mm
- net OSC2: track 0.00 -> 9.02 mm
- net A1: track 7.62 -> 0.00 mm
- net RS: track 0.00 -> 7.62 mm
- net E: track 0.00 -> 7.62 mm
- net D7: track 0.00 -> 7.62 mm
- net D6: track 0.00 -> 7.62 mm
- net D5: track 0.00 -> 7.62 mm
- net D4: track 0.00 -> 7.62 mm
- net GND: track 57.0 -> 50.8 mm
- net /MCLR: track 0.00 -> 2.54 mm
- net A0: track 24.7 -> 25.4 mm
Other:
- board size 48.6 x 49.5 mm -> 51.1 x 49.5 mm
