File: eagle/LCmeter0-LCD3310-8pinlcd-PIC-COMP.brd (EAGLE design)
At the start: 43 parts, among them IC1 PIC16F876A, J2 PIC-UART, J3 PIC-ICSP, J4 J4, J5 CONN-2P2P/V, J6 NOKIA-5510-48X84, J7 CONN-2P2P/V, K2 DS2Y, Q1 20MHz, SW1 PB-1P-1T, T1 BC547

Commit message: ...
Parts:
- C10: device c:C025-015X024/V -> c:C050-020X036
- C8: device c:C050-020X036 -> c:C025-015X024
- R1: device r:0202/7 -> r:0204/10
- R10, R12, R13, R14, R15, R16, R17, R2, R3, R4, R5, R8: device r:0202/7 -> r:0202/7@1
- R6: device r:0202/7-V -> r:0204/7-V
- R7: device r:0202/10-V -> r:0204/10
- moved J3 5.08 mm to (40.6, 48.3)
- moved J4 3.81 mm to (54.6, 2.54), turned to 0 degrees
- moved C8 1.27 mm to (53.3, 47.0), turned to 90 degrees
- moved J7 1.27 mm to (5.08, 14.0)
- moved C3 1.27 mm to (21.6, 38.1)
- moved C4 1.27 mm to (21.6, 33.0)
- turned R7 to 90 degrees
- turned R9 to 270 degrees
Routing:
- net GND: track 200.7 -> 204.5 mm
- net VCC: track 129.5 -> 133.3 mm
- net N$12: track 10.2 -> 7.62 mm
- net FREQ: track 48.3 -> 49.5 mm
- net A3: track 44.5 -> 43.2 mm

Commit message: ...
Parts:
- L1: device r:L-09R -> r:L-8R
Changed lines of the file:
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@@
 </element>
 <element name="D1" library="d" package="DO34-7" value="1N4148" x="19.05" y="2.54"/>
-<element name="L1" library="r" package="L-09R" value="68μH" x="7.62" y="43.18"/>
+<element name="L1" library="r" package="L-8R" value="68μH" x="7.62" y="43.18"/>
 <element name="Q1" library="q" package="HC49" value="20MHz" x="33.02" y="17.78"/>
 <element name="R1" library="r" package="0204/10" value="100kΩ" x="31.75" y="38.1"/>

Commit message: ...
Parts:
- R11: value 1k -> 1kΩ
- R12, R8, R9: value 100 -> 100Ω
- R13, R14, R15, R16, R17, R6: value 10k -> 10kΩ
Changed lines of the file:
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@@
 <attribute name="NAME" x="39.37" y="46.355" size="0.8128" layer="25" align="top-left"/>
 </element>
-<element name="R8" library="r" package="0202/7@1" value="100" x="46.99" y="45.72"/>
-<element name="R9" library="r" package="0202/2V" value="100" x="46.99" y="43.18" rot="R270"/>
+<element name="R8" library="r" package="0202/7@1" value="100Ω" x="46.99" y="45.72"/>
+<element name="R9" library="r" package="0202/2V" value="100Ω" x="46.99" y="43.18" rot="R270"/>
 <element name="LED1" library="led" package="LED3MM" value="TLLG4400" x="27.94" y="13.97" smashed="yes" rot="R90">
 <attribute name="MF" value="VISHAY SEMICONDUCTOR" x="27.94" y="13.97" size="0.8128" layer="27" rot="R90" display="off"/>
@@
 <element name="SW1" library="sw" package="PB-1P1T" value="PB-1P-1T" x="22.86" y="45.72" rot="R180"/>
 <element name="IC1" library="mcu" package="DIL28-3/V" value="PIC16F876A" x="41.91" y="24.13"/>
-<element name="R6" library="r" package="0204/7-V" value="10k" x="48.26" y="6.35" rot="R180"/>
-<element name="R11" library="r" package="0202/5-V" value="1k" x="35.56" y="10.16"/>
+<element name="R6" library="r" package="0204/7-V" value="10kΩ" x="48.26" y="6.35" rot="R180"/>
+<element name="R11" library="r" package="0202/5-V" value="1kΩ" x="35.56" y="10.16"/>
 <element name="J7" library="pinconn" package="CONN-2P-V" value="CONN-2P2P/V" x="5.08" y="13.97"/>
 <element name="J5" library="pinconn" package="CONN-2P-V" value="CONN-2P2P/V" x="5.08" y="2.54"/>
@@
 </element>
 <element name="C10" library="c" package="C050-020X036" value="100nF" x="55.88" y="24.13"/>
-<element name="R12" library="r" package="0202/7@1" value="100" x="52.07" y="40.64" rot="R180"/>
-<element name="R13" library="r" package="0202/7@1" value="10k" x="52.07" y="38.1" rot="R180"/>
-<element name="R14" library="r" package="0202/7@1" value="10k" x="52.07" y="35.56" rot="R180"/>
-<element name="R15" library="r" package="0202/7@1" value="10k" x="52.07" y="33.02" rot="R180"/>
-<element name="R16" library="r" package="0202/7@1" value="10k" x="52.07" y="30.48" rot="R180"/>
-<element name="R17" library="r" package="0202/7@1" value="10k" x="52.07" y="27.94"/>
+<element name="R12" library="r" package="0202/7@1" value="100Ω" x="52.07" y="40.64" rot="R180"/>
+<element name="R13" library="r" package="0202/7@1" value="10kΩ" x="52.07" y="38.1" rot="R180"/>
+<element name="R14" library="r" package="0202/7@1" value="10kΩ" x="52.07" y="35.56" rot="R180"/>
+<element name="R15" library="r" package="0202/7@1" value="10kΩ" x="52.07" y="33.02" rot="R180"/>
+<element name="R16" library="r" package="0202/7@1" value="10kΩ" x="52.07" y="30.48" rot="R180"/>
+<element name="R17" library="r" package="0202/7@1" value="10kΩ" x="52.07" y="27.94"/>
 </elements>
 <signals>

Commit message: ...
Routing:
- net M+: track 20.3 -> 15.9 mm
- net GND: track 204.5 -> 201.6 mm
- net M-: track 20.3 -> 21.9 mm, vias 2 -> 0
- net A0: track 30.5 -> 29.0 mm
- net VCC: track 133.3 -> 132.3 mm
