File: eagle/LCmeter0-LCD3310-8pinlcd-PIC-COMP.sch (EAGLE design)
At the start: 36 parts, among them IC1 PIC16F876A, J1 HD44780-4BITLCD44780-8P, J2 PIC-UART, J3 PIC-ICSP, J4 J4, J5 CONN-2P2P/V, J7 CONN-2P2P/V, K2 DS2Y, Q1 20MHz, SW1 PB-1P-1T, T1 BC547

Commit message: ...
Parts:
- IC1: value PIC16F876A -> PIC16F876A-X/SP; device lc-meter:PIC16F876A-X/SP-COMP-B-A -> mcu:PIC16F876A-X/SP-COMPDIL28-3/V
- J1: value HD44780-4BITLCD44780-8P -> SPI-LCD3310; device pinconn:HD44780-4BITLCD44780-8P -> lcd:NOKIA-3310-64X64SPARKFUN
Connections:
- net /MCLR: no longer IC1.*MCLR/VPP
- net D4: now also J1.SCE; no longer J1.D4
- net D5: now also J1.GND; no longer J1.D5
- net D6: now also J1.VOUT; no longer J1.D6
- net D7: now also J1.RES; no longer J1.D7
- net E: now also J1.D_C; no longer J1.E
- net GND: now also J1.VDD; no longer J1.GND
- net RS: now also J1.SDIN; no longer J1.RS
- net VCC: now also IC1.RA2, J1.SCK; no longer IC1.VDD, J1.VCC
Other:
- moved on the sheet: C5, C6, C7, C8, C9, D2, J2, J3, J4, LED1, Q1, R10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

Commit message: ...
Parts:
- J1: value SPI-LCD3310 -> NOKIA-3310-64X64SPARKFUN
Changed lines of the file:
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@@
 <part name="C8" library="c" deviceset="C" device="050-020X036" value="22pF"/>
 <part name="GND3" library="supply1" deviceset="GND" device=""/>
-<part name="J1" library="lcd" deviceset="NOKIA-3310-64X64" device="SPARKFUN" value="SPI-LCD3310"/>
 <part name="IC1" library="mcu" deviceset="PIC16F876A-X/SP-COMP" device="DIL28-3/V" value="PIC16F876A-X/SP"/>
+<part name="J1" library="lcd" deviceset="NOKIA-3310-64X64" device="SPARKFUN"/>
 </parts>
 <sheets>
@@
 <instance part="C8" gate="G$1" x="261.62" y="45.72"/>
 <instance part="GND3" gate="1" x="269.24" y="12.7"/>
+<instance part="IC1" gate="1" x="137.16" y="25.4"/>
 <instance part="J1" gate="1" x="252.73" y="-31.75" rot="R180"/>
-<instance part="IC1" gate="1" x="137.16" y="25.4"/>
 </instances>
 <busses>
@@
 <junction x="180.34" y="-7.62"/>
 <junction x="236.22" y="-7.62"/>
-<pinref part="J1" gate="1" pin="VDD"/>
 <pinref part="IC1" gate="1" pin="VSS"/>
 <pinref part="IC1" gate="1" pin="VSS_2"/>
-</segment>
-<segment>
+<pinref part="J1" gate="1" pin="VDD"/>
+</segment>
+<segment>

Commit message: ...
Parts:
- J1: value NOKIA-3310-64X64SPARKFUN -> SPI-LCD3310
Connections:
- net /MCLR: now also IC1.*MCLR/VPP
- net VCC: now also IC1.VDD; no longer IC1.RA2
Changed lines of the file:
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@@
 <part name="GND3" library="supply1" deviceset="GND" device=""/>
 <part name="IC1" library="mcu" deviceset="PIC16F876A-X/SP-COMP" device="DIL28-3/V" value="PIC16F876A-X/SP"/>
-<part name="J1" library="lcd" deviceset="NOKIA-3310-64X64" device="SPARKFUN"/>
+<part name="J1" library="lcd" deviceset="NOKIA-3310-64X64" device="SPARKFUN" value="SPI-LCD3310"/>
 </parts>
 <sheets>
@@
 <attribute name="VALUE" x="165.1" y="-16.51" size="1.778" layer="96" align="bottom-center"/>
 </instance>
-<instance part="P+11" gate="VCC" x="144.78" y="60.96" smashed="yes">
-<attribute name="VALUE" x="144.78" y="62.23" size="1.778" layer="96" align="bottom-center"/>
+<instance part="P+11" gate="VCC" x="123.19" y="60.96" smashed="yes">
+<attribute name="VALUE" x="123.19" y="62.23" size="1.778" layer="96" align="bottom-center"/>
 </instance>
 <instance part="R6" gate="G$1" x="66.04" y="-15.24" rot="R90"/>
@@
 <wire x1="236.22" y1="-7.62" x2="236.22" y2="-12.7" width="0.1524" layer="91"/>
 <label x="139.7" y="-7.62" size="1.778" layer="95"/>
-<junction x="236.22" y="-7.62"/>
-<wire x1="236.22" y1="-7.62" x2="243.84" y2="-7.62" width="0.1524" layer="91"/>
-<wire x1="243.84" y1="-7.62" x2="243.84" y2="-12.7" width="0.1524" layer="91"/>
 <wire x1="139.7" y1="7.62" x2="139.7" y2="-7.62" width="0.1524" layer="91"/>
-<wire x1="139.7" y1="-7.62" x2="149.86" y2="-7.62" width="0.1524" layer="91"/>
-<wire x1="149.86" y1="-7.62" x2="149.86" y2="7.62" width="0.1524" layer="91"/>
 <wire x1="236.22" y1="-7.62" x2="180.34" y2="-7.62" width="0.1524" layer="91"/>
-<junction x="149.86" y="-7.62"/>
 <pinref part="C6" gate="G$1" pin="1"/>
 <wire x1="180.34" y1="-7.62" x2="170.18" y2="-7.62" width="0.1524" layer="91"/>
 <wire x1="170.18" y1="-7.62" x2="149.86" y2="-7.62" width="0.1524" layer="91"/>
+<wire x1="149.86" y1="-7.62" x2="139.7" y2="-7.62" width="0.1524" layer="91"/>
 <wire x1="170.18" y1="-5.08" x2="170.18" y2="-7.62" width="0.1524" layer="91"/>
 <junction x="170.18" y="-7.62"/>
@@
 <wire x1="180.34" y1="-5.08" x2="180.34" y2="-7.62" width="0.1524" layer="91"/>
 <junction x="180.34" y="-7.62"/>
+<pinref part="IC1" gate="1" pin="VSS"/>
+<wire x1="236.22" y1="-7.62" x2="243.84" y2="-7.62" width="0.1524" layer="91"/>
 <junction x="236.22" y="-7.62"/>
-<pinref part="IC1" gate="1" pin="VSS"/>
+<pinref part="J1" gate="1" pin="VDD"/>
+<wire x1="243.84" y1="-7.62" x2="243.84" y2="-12.7" width="0.1524" layer="91"/>
 <pinref part="IC1" gate="1" pin="VSS_2"/>
-<pinref part="J1" gate="1" pin="VDD"/>
+<wire x1="149.86" y1="7.62" x2="149.86" y2="-7.62" width="0.1524" layer="91"/>
+<junction x="149.86" y="-7.62"/>
 </segment>
 <segment>
@@
 <segment>
 <pinref part="C5" gate="G$1" pin="2"/>
-<wire x1="180.34" y1="7.62" x2="180.34" y2="5.08" width="0.1524" layer="91"/>
 <pinref part="Q1" gate="G$1" pin="1"/>
 <wire x1="180.34" y1="5.08" x2="180.34" y2="2.54" width="0.1524" layer="91"/>
 <wire x1="177.8" y1="5.08" x2="180.34" y2="5.08" width="0.1524" layer="91"/>
+<pinref part="IC1" gate="1" pin="OSC2"/>
+<wire x1="180.34" y1="7.62" x2="180.34" y2="5.08" width="0.1524" layer="91"/>
 <junction x="180.34" y="5.08"/>
-<pinref part="IC1" gate="1" pin="OSC2"/>
 </segment>
 </net>
@@
 <pinref part="R10" gate="G$1" pin="1"/>
 <wire x1="233.68" y1="30.48" x2="246.38" y2="30.48" width="0.1524" layer="91"/>
-<wire x1="246.38" y1="-12.7" x2="246.38" y2="27.94" width="0.1524" layer="91"/>
 <pinref part="J3" gate="G$1" pin="VDD"/>
 <wire x1="246.38" y1="27.94" x2="271.78" y2="27.94" width="0.1524" layer="91"/>
+<pinref part="P+6" gate="VCC" pin="VCC"/>
 <wire x1="246.38" y1="30.48" x2="246.38" y2="27.94" width="0.1524" layer="91"/>
-<junction x="246.38" y="27.94"/>
-<pinref part="P+6" gate="VCC" pin="VCC"/>
 <wire x1="246.38" y1="30.48" x2="246.38" y2="35.56" width="0.1524" layer="91"/>
 <junction x="246.38" y="30.48"/>
 <pinref part="J1" gate="1" pin="SCK"/>
+<wire x1="246.38" y1="-12.7" x2="246.38" y2="27.94" width="0.1524" layer="91"/>
+<junction x="246.38" y="27.94"/>
 </segment>
 <segment>
@@
 </segment>
 <segment>
-<pinref part="P+11" gate="VCC" pin="VCC"/>
-<wire x1="144.78" y1="58.42" x2="144.78" y2="43.18" width="0.1524" layer="91"/>
-<pinref part="IC1" gate="1" pin="RA2"/>
-</segment>
-<segment>
 <pinref part="D2" gate="G$1" pin="C"/>
 <wire x1="208.28" y1="-17.78" x2="213.36" y2="-17.78" width="0.1524" layer="91"/>
@@
 <junction x="213.36" y="-17.78"/>
 </segment>
+<segment>
+<pinref part="IC1" gate="1" pin="VDD"/>
+<pinref part="P+11" gate="VCC" pin="VCC"/>
+<wire x1="124.46" y1="43.18" x2="124.46" y2="57.15" width="0.1524" layer="91"/>
+<wire x1="124.46" y1="57.15" x2="123.19" y2="58.42" width="0.1524" layer="91"/>
+</segment>
 </net>
 <net name="D4" class="0">
 <segment>
-<wire x1="254" y1="-12.7" x2="254" y2="2.54" width="0.1524" layer="91"/>
 <wire x1="254" y1="2.54" x2="220.98" y2="2.54" width="0.1524" layer="91"/>
 <wire x1="220.98" y1="2.54" x2="218.44" y2="5.08" width="0.1524" layer="91"/>
 <label x="226.06" y="2.54" size="1.778" layer="95"/>
+<wire x1="254" y1="2.54" x2="254" y2="-12.7" width="0.1524" layer="91"/>
 <pinref part="J1" gate="1" pin="SCE"/>
 </segment>
@@
 <net name="E" class="0">
 <segment>
-<wire x1="251.46" y1="-12.7" x2="251.46" y2="0" width="0.1524" layer="91"/>
 <wire x1="251.46" y1="0" x2="220.98" y2="0" width="0.1524" layer="91"/>
 <wire x1="220.98" y1="0" x2="218.44" y2="2.54" width="0.1524" layer="91"/>
 <label x="226.06" y="0" size="1.778" layer="95"/>
 <pinref part="J1" gate="1" pin="D_C"/>
+<wire x1="251.46" y1="0" x2="251.46" y2="-12.7" width="0.1524" layer="91"/>
 </segment>
 <segment>
@@
 <net name="RS" class="0">
 <segment>
-<wire x1="248.92" y1="-12.7" x2="248.92" y2="-2.54" width="0.1524" layer="91"/>
 <wire x1="248.92" y1="-2.54" x2="220.98" y2="-2.54" width="0.1524" layer="91"/>
 <wire x1="220.98" y1="-2.54" x2="218.44" y2="0" width="0.1524" layer="91"/>
 <label x="226.06" y="-2.54" size="1.778" layer="95"/>
 <pinref part="J1" gate="1" pin="SDIN"/>
+<wire x1="248.92" y1="-2.54" x2="248.92" y2="-12.7" width="0.1524" layer="91"/>
 </segment>
 <segment>
@@
 <wire x1="271.78" y1="25.4" x2="220.98" y2="25.4" width="0.1524" layer="91"/>
 <wire x1="220.98" y1="25.4" x2="210.82" y2="25.4" width="0.1524" layer="91"/>
-<wire x1="201.93" y1="25.4" x2="210.82" y2="25.4" width="0.1524" layer="91"/>
+<wire x1="200.66" y1="25.4" x2="210.82" y2="25.4" width="0.1524" layer="91"/>
 <wire x1="210.82" y1="25.4" x2="210.82" y2="20.32" width="0.1524" layer="91"/>
 <junction x="220.98" y="25.4"/>
 <junction x="210.82" y="25.4"/>
+<pinref part="IC1" gate="1" pin="*MCLR/VPP"/>
 </segment>
 </net>
 <net name="D5" class="0">
 <segment>
-<wire x1="256.54" y1="-12.7" x2="256.54" y2="5.08" width="0.1524" layer="91"/>
 <wire x1="256.54" y1="5.08" x2="220.98" y2="5.08" width="0.1524" layer="91"/>
 <wire x1="220.98" y1="5.08" x2="218.44" y2="7.62" width="0.1524" layer="91"/>
 <label x="226.06" y="5.08" size="1.778" layer="95"/>
 <pinref part="J1" gate="1" pin="GND"/>
+<wire x1="256.54" y1="-12.7" x2="256.54" y2="5.08" width="0.1524" layer="91"/>
 </segment>
 <segment>
@@
 <net name="D6" class="0">
 <segment>
-<wire x1="259.08" y1="-12.7" x2="259.08" y2="7.62" width="0.1524" layer="91"/>
 <wire x1="259.08" y1="7.62" x2="220.98" y2="7.62" width="0.1524" layer="91"/>
 <wire x1="220.98" y1="7.62" x2="218.44" y2="10.16" width="0.1524" layer="91"/>
 <label x="226.06" y="7.62" size="1.778" layer="95"/>
 <pinref part="J1" gate="1" pin="VOUT"/>
+<wire x1="259.08" y1="-12.7" x2="259.08" y2="7.62" width="0.1524" layer="91"/>
+<wire x1="259.08" y1="8.89" x2="259.08" y2="7.62" width="0.1524" layer="91"/>
+<junction x="259.08" y="7.62"/>
 </segment>
 <segment>
@@
 <net name="D7" class="0">
 <segment>
-<wire x1="261.62" y1="-12.7" x2="261.62" y2="10.16" width="0.1524" layer="91"/>
 <wire x1="261.62" y1="10.16" x2="220.98" y2="10.16" width="0.1524" layer="91"/>
 <wire x1="220.98" y1="10.16" x2="218.44" y2="12.7" width="0.1524" layer="91"/>
 <label x="226.06" y="10.16" size="1.778" layer="95"/>
 <pinref part="J1" gate="1" pin="RES"/>
-</segment>
-<segment>
+<wire x1="261.62" y1="10.16" x2="261.62" y2="-12.7" width="0.1524" layer="91"/>
+</segment>
+<segment>

Commit message: ...
Parts:
- IC1: value PIC16F876A-X/SP -> PIC16F876A
- J1: value SPI-LCD3310 -> NOKIA-3310-64X64SPARKFUN
Changed lines of the file:
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@@
 <grid distance="50" unitdist="mil" unit="inch" style="dots" multiple="2" display="yes" altdistance="10" altunitdist="mil" altunit="inch"/>
 <layers>
-<layer number="1" name="Top" color="4" fill="1" visible="no" active="no"/>
-<layer number="2" name="Route2" color="1" fill="3" visible="no" active="no"/>
-<layer number="3" name="Route3" color="4" fill="3" visible="no" active="no"/>
-<layer number="4" name="Route4" color="1" fill="4" visible="no" active="no"/>
-<layer number="5" name="Route5" color="4" fill="4" visible="no" active="no"/>
-<layer number="6" name="Route6" color="1" fill="8" visible="no" active="no"/>
-<layer number="7" name="Route7" color="4" fill="8" visible="no" active="no"/>
-<layer number="8" name="Route8" color="1" fill="2" visible="no" active="no"/>
-<layer number="9" name="Route9" color="4" fill="2" visible="no" active="no"/>
-<layer number="10" name="Route10" color="1" fill="7" visible="no" active="no"/>
-<layer number="11" name="Route11" color="4" fill="7" visible="no" active="no"/>
-<layer number="12" name="Route12" color="1" fill="5" visible="no" active="no"/>
-<layer number="13" name="Route13" color="4" fill="5" visible="no" active="no"/>
-<layer number="14" name="Route14" color="1" fill="6" visible="no" active="no"/>
-<layer number="15" name="Route15" color="4" fill="6" visible="no" active="no"/>
-<layer number="16" name="Bottom" color="1" fill="1" visible="no" active="no"/>
-<layer number="17" name="Pads" color="2" fill="1" visible="no" active="no"/>
-<layer number="18" name="Vias" color="2" fill="1" visible="no" active="no"/>
-<layer number="19" name="Unrouted" color="6" fill="1" visible="no" active="no"/>
-<layer number="20" name="Dimension" color="15" fill="1" visible="no" active="no"/>
-<layer number="21" name="tPlace" color="7" fill="1" visible="no" active="no"/>
-<layer number="22" name="bPlace" color="7" fill="1" visible="no" active="no"/>
-<layer number="23" name="tOrigins" color="15" fill="1" visible="no" active="no"/>
-<layer number="24" name="bOrigins" color="15" fill="1" visible="no" active="no"/>
-<layer number="25" name="tNames" color="7" fill="1" visible="no" active="no"/>
-<layer number="26" name="bNames" color="7" fill="1" visible="no" active="no"/>
-<layer number="27" name="tValues" color="7" fill="1" visible="no" active="no"/>
-<layer number="28" name="bValues" color="7" fill="1" visible="no" active="no"/>
+<layer number="1" name="Top" color="4" fill="1" visible="yes" active="no"/>
+<layer number="2" name="Route2" color="1" fill="3" visible="yes" active="no"/>
+<layer number="3" name="Route3" color="4" fill="3" visible="yes" active="no"/>
+<layer number="4" name="Route4" color="1" fill="4" visible="yes" active="no"/>
+<layer number="5" name="Route5" color="4" fill="4" visible="yes" active="no"/>
+<layer number="6" name="Route6" color="1" fill="8" visible="yes" active="no"/>
+<layer number="7" name="Route7" color="4" fill="8" visible="yes" active="no"/>
+<layer number="8" name="Route8" color="1" fill="2" visible="yes" active="no"/>
+<layer number="9" name="Route9" color="4" fill="2" visible="yes" active="no"/>
+<layer number="10" name="Route10" color="1" fill="7" visible="yes" active="no"/>
+<layer number="11" name="Route11" color="4" fill="7" visible="yes" active="no"/>
+<layer number="12" name="Route12" color="1" fill="5" visible="yes" active="no"/>
+<layer number="13" name="Route13" color="4" fill="5" visible="yes" active="no"/>
+<layer number="14" name="Route14" color="1" fill="6" visible="yes" active="no"/>
+<layer number="15" name="Route15" color="4" fill="6" visible="yes" active="no"/>
+<layer number="16" name="Bottom" color="1" fill="1" visible="yes" active="no"/>
+<layer number="17" name="Pads" color="2" fill="1" visible="yes" active="no"/>
+<layer number="18" name="Vias" color="2" fill="1" visible="yes" active="no"/>
+<layer number="19" name="Unrouted" color="6" fill="1" visible="yes" active="no"/>
+<layer number="20" name="Dimension" color="15" fill="1" visible="yes" active="no"/>
+<layer number="21" name="tPlace" color="7" fill="1" visible="yes" active="no"/>
+<layer number="22" name="bPlace" color="7" fill="1" visible="yes" active="no"/>
+<layer number="23" name="tOrigins" color="15" fill="1" visible="yes" active="no"/>
+<layer number="24" name="bOrigins" color="15" fill="1" visible="yes" active="no"/>
+<layer number="25" name="tNames" color="7" fill="1" visible="yes" active="no"/>
+<layer number="26" name="bNames" color="7" fill="1" visible="yes" active="no"/>
+<layer number="27" name="tValues" color="7" fill="1" visible="yes" active="no"/>
+<layer number="28" name="bValues" color="7" fill="1" visible="yes" active="no"/>
 <layer number="29" name="tStop" color="7" fill="3" visible="no" active="no"/>
 <layer number="30" name="bStop" color="7" fill="6" visible="no" active="no"/>
@@
 <layer number="35" name="tGlue" color="7" fill="4" visible="no" active="no"/>
 <layer number="36" name="bGlue" color="7" fill="5" visible="no" active="no"/>
-<layer number="37" name="tTest" color="7" fill="1" visible="no" active="no"/>
-<layer number="38" name="bTest" color="7" fill="1" visible="no" active="no"/>
+<layer number="37" name="tTest" color="7" fill="1" visible="yes" active="no"/>
+<layer number="38" name="bTest" color="7" fill="1" visible="yes" active="no"/>
 <layer number="39" name="tKeepout" color="4" fill="11" visible="no" active="no"/>
 <layer number="40" name="bKeepout" color="1" fill="11" visible="no" active="no"/>
@@
 <layer number="44" name="Drills" color="7" fill="1" visible="no" active="no"/>
 <layer number="45" name="Holes" color="7" fill="1" visible="no" active="no"/>
-<layer number="46" name="Milling" color="3" fill="1" visible="no" active="no"/>
-<layer number="47" name="Measures" color="7" fill="1" visible="no" active="no"/>
-<layer number="48" name="Document" color="7" fill="1" visible="no" active="no"/>
-<layer number="49" name="Reference" color="7" fill="1" visible="no" active="no"/>
-<layer number="51" name="tDocu" color="7" fill="1" visible="no" active="no"/>
-<layer number="52" name="bDocu" color="7" fill="1" visible="no" active="no"/>
+<layer number="46" name="Milling" color="3" fill="1" visible="yes" active="no"/>
+<layer number="47" name="Measures" color="7" fill="1" visible="yes" active="no"/>
+<layer number="48" name="Document" color="7" fill="1" visible="yes" active="no"/>
+<layer number="49" name="Reference" color="7" fill="1" visible="yes" active="no"/>
+<layer number="51" name="tDocu" color="7" fill="1" visible="yes" active="no"/>
+<layer number="52" name="bDocu" color="7" fill="1" visible="yes" active="no"/>
 <layer number="90" name="Modules" color="5" fill="10" visible="yes" active="yes"/>
 <layer number="91" name="Nets" color="2" fill="1" visible="yes" active="yes"/>
@@
 <part name="C8" library="c" deviceset="C" device="050-020X036" value="22pF"/>
 <part name="GND3" library="supply1" deviceset="GND" device=""/>
-<part name="IC1" library="mcu" deviceset="PIC16F876A-X/SP-COMP" device="DIL28-3/V" value="PIC16F876A-X/SP"/>
-<part name="J1" library="lcd" deviceset="NOKIA-3310-64X64" device="SPARKFUN" value="SPI-LCD3310"/>
+<part name="IC1" library="mcu" deviceset="PIC16F876A-X/SP-COMP" device="DIL28-3/V" value="PIC16F876A"/>
+<part name="J1" library="lcd" deviceset="NOKIA-3310-64X64" device="SPARKFUN" value="NOKIA-3310-64X64SPARKFUN"/>
 </parts>
 <sheets>

Commit message: ...
Parts:
- removed J1: NOKIA-3310-64X64SPARKFUN, lcd:NOKIA-3310-64X64SPARKFUN
- added C10: 100nF, c:C025-015X024
- added J6: NOKIA-5510-48X84, lcd:NOKIA-5510-48X84
- added R12: 100, r:R0202/7
- added R13, R14, R15, R16, R17: 10k, r:R0202/7
- C7: device c:CPOLE2.5-5 -> c:CPOLE5-5
- D2: device d:1N414834-12V -> d:1N414834-10V
- R7: device r:R0202/10 -> r:R0202/10-V
- R9: device r:R0202/5-V -> r:R0202/2V
Connections:
- removed net D4: IC1.RB4, J1.SCE
- removed net D5: IC1.RB5, J1.GND
- removed net D6: IC1.RB6, J1.VOUT, R8.2
- removed net D7: IC1.RB7, J1.RES, R9.2
- removed net E: IC1.RB3, J1.D_C
- removed net RS: IC1.RB2, J1.SDIN
- new net N$13: J6.SDIN, R14.1
- new net N$14: J6.SCLK, R13.1
- new net N$15: J6.RES, R16.1
- new net N$16: J6.SCE, R17.1
- new net N$17: IC1.RB1
- new net N$3: J6.LED, R12.1
- new net N$4: J6.D_C, R15.1
- new net RB2: IC1.RB2, R17.2
- new net RB3: IC1.RB3, R16.2
- new net RB4: IC1.RB4, R15.2
- new net RB5: IC1.RB5, R14.2
- new net RB6: IC1.RB6, R13.2, R8.2
- new net RB7: IC1.RB7, R12.2, R9.2
- net GND: now also C10.1, J6.GND; no longer J1.VDD
- net N$11: no longer IC1.RB1
- net VCC: now also C10.2, J6.VCC; no longer J1.SCK
