File: eagle/CapMeter-LCD-16F876A.brd (EAGLE design)
At the start: 33 x 40.6 mm, 14 parts, among them IC1 PIC16F876A-X/SP-COMPDIL28-3/V, J1 CONN-2P2P/H, Q1 20MHz

Commit message: ...
Parts:
- added U$1: LCD-8PIN, lcd:1X8
Connections:
- new net D4: IC1.25, U$1.5
- new net D5: IC1.26, U$1.6
- new net D6: IC1.27, U$1.7
- new net D7: IC1.28, U$1.8
- new net E: IC1.24, U$1.4
- new net RS: IC1.23, U$1.3
Changed lines of the file:
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@@
 <layer number="98" name="Guide" color="6" fill="1" visible="no" active="no"/>
 <layer number="99" name="SpiceOrder" color="7" fill="1" visible="no" active="no"/>
+<layer number="100" name="LCD" color="13" fill="1" visible="no" active="yes"/>
 <layer number="250" name="trash" color="7" fill="1" visible="yes" active="yes"/>
 </layers>
@@
 <element name="J1" library="pinconn" package="CONN-2P" value="CONN-2P2P/H" x="29.21" y="5.08"/>
 <element name="C2" library="c" package="C025-020X036" value="100nF" x="27.94" y="13.97" rot="R270"/>
+<element name="U$1" library="lcd" package="1X8" value="LCD-8PIN" x="30.48" y="26.67" rot="R90"/>
 </elements>
 <signals>
@@
 <wire x1="12.7" y1="7.62" x2="16.51" y2="7.62" width="0.6096" layer="16"/>
 </signal>
+<signal name="D7">
+<contactref element="U$1" pad="8"/>
+<contactref element="IC1" pad="28"/>
+<wire x1="30.48" y1="35.56" x2="24.13" y2="35.56" width="0" layer="19" extent="1-1"/>
+</signal>
+<signal name="D6">
+<contactref element="U$1" pad="7"/>
+<contactref element="IC1" pad="27"/>
+<wire x1="30.48" y1="33.02" x2="24.13" y2="33.02" width="0" layer="19" extent="1-1"/>
+</signal>
+<signal name="D5">
+<contactref element="U$1" pad="6"/>
+<contactref element="IC1" pad="26"/>
+<wire x1="30.48" y1="30.48" x2="24.13" y2="30.48" width="0" layer="19" extent="1-1"/>
+</signal>
+<signal name="D4">
+<contactref element="U$1" pad="5"/>
+<contactref element="IC1" pad="25"/>
+<wire x1="30.48" y1="27.94" x2="24.13" y2="27.94" width="0" layer="19" extent="1-1"/>
+</signal>
+<signal name="E">
+<contactref element="U$1" pad="4"/>
+<contactref element="IC1" pad="24"/>
+<wire x1="30.48" y1="25.4" x2="24.13" y2="25.4" width="0" layer="19" extent="1-1"/>
+</signal>
+<signal name="RS">
+<contactref element="U$1" pad="3"/>
+<contactref element="IC1" pad="23"/>
+<wire x1="30.48" y1="22.86" x2="24.13" y2="22.86" width="0" layer="19" extent="1-1"/>
+</signal>
 </signals>

Commit message: ...
Routing:
- net RS: track 0.00 -> 6.35 mm
- net E: track 0.00 -> 6.35 mm
- net D7: track 0.00 -> 6.35 mm
- net D6: track 0.00 -> 6.35 mm
- net D5: track 0.00 -> 6.35 mm
- net D4: track 0.00 -> 6.35 mm
- net GND: track 71.1 -> 73.7 mm
- net N$3: track 22.9 -> 25.4 mm
Changed lines of the file:
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@@
 <contactref element="C1" pad="2"/>
 <contactref element="TEST-" pad="1"/>
-<wire x1="2.54" y1="30.48" x2="2.54" y2="22.86" width="0.6096" layer="16"/>
 <wire x1="2.54" y1="15.24" x2="2.54" y2="22.86" width="0.6096" layer="16"/>
 <wire x1="2.54" y1="22.86" x2="12.7" y2="22.86" width="0.6096" layer="16"/>
@@
 <wire x1="27.94" y1="12.7" x2="27.94" y2="5.08" width="0.6096" layer="16"/>
 <wire x1="5.08" y1="38.1" x2="5.08" y2="33.02" width="0.6096" layer="16"/>
-<wire x1="2.54" y1="33.02" x2="5.08" y2="33.02" width="0.6096" layer="16"/>
-<wire x1="5.08" y1="33.02" x2="5.08" y2="30.48" width="0.6096" layer="16"/>
 <wire x1="27.94" y1="12.7" x2="24.13" y2="12.7" width="0.6096" layer="16"/>
-<wire x1="2.54" y1="30.48" x2="2.54" y2="33.02" width="0" layer="19" extent="16-16"/>
-<wire x1="2.54" y1="27.94" x2="2.54" y2="30.48" width="0" layer="19" extent="16-16"/>
+<wire x1="2.54" y1="27.94" x2="2.54" y2="22.86" width="0.6096" layer="16"/>
+<wire x1="5.08" y1="30.48" x2="5.08" y2="33.02" width="0.6096" layer="16"/>
+<wire x1="5.08" y1="33.02" x2="2.54" y2="33.02" width="0.6096" layer="16"/>
+<wire x1="2.54" y1="33.02" x2="2.54" y2="27.94" width="0.6096" layer="16"/>
 </signal>
 <signal name="N$3">
@@
 <wire x1="19.05" y1="25.4" x2="19.05" y2="38.1" width="0.6096" layer="16"/>
 <wire x1="19.05" y1="38.1" x2="15.24" y2="38.1" width="0.6096" layer="16"/>
-<wire x1="12.7" y1="25.4" x2="12.7" y2="27.94" width="0" layer="19" extent="1-1"/>
+<wire x1="12.7" y1="25.4" x2="12.7" y2="27.94" width="0.6096" layer="16"/>
 </signal>
 <signal name="VCC">
@@
 <contactref element="R5" pad="1"/>
 <wire x1="2.54" y1="25.4" x2="2.54" y2="22.86" width="0.6096" layer="16"/>
-<wire x1="2.54" y1="25.4" x2="2.54" y2="33.02" width="0.6096" layer="16"/>
 <wire x1="2.54" y1="22.86" x2="12.7" y2="22.86" width="0.6096" layer="16"/>
 <wire x1="12.7" y1="22.86" x2="16.51" y2="22.86" width="0.6096" layer="16"/>
+<wire x1="2.54" y1="33.02" x2="2.54" y2="25.4" width="0.6096" layer="16"/>
 </signal>
 <signal name="N$4">
@@
 <contactref element="U$1" pad="8"/>
 <contactref element="IC1" pad="28"/>
-<wire x1="30.48" y1="35.56" x2="24.13" y2="35.56" width="0" layer="19" extent="1-1"/>
+<wire x1="24.13" y1="35.56" x2="30.48" y2="35.56" width="0.6096" layer="16"/>
 </signal>
 <signal name="D6">
 <contactref element="U$1" pad="7"/>
 <contactref element="IC1" pad="27"/>
-<wire x1="30.48" y1="33.02" x2="24.13" y2="33.02" width="0" layer="19" extent="1-1"/>
+<wire x1="30.48" y1="33.02" x2="24.13" y2="33.02" width="0.6096" layer="16"/>
 </signal>
 <signal name="D5">
 <contactref element="U$1" pad="6"/>
 <contactref element="IC1" pad="26"/>
-<wire x1="30.48" y1="30.48" x2="24.13" y2="30.48" width="0" layer="19" extent="1-1"/>
+<wire x1="24.13" y1="30.48" x2="30.48" y2="30.48" width="0.6096" layer="16"/>
 </signal>
 <signal name="D4">
 <contactref element="U$1" pad="5"/>
 <contactref element="IC1" pad="25"/>
-<wire x1="30.48" y1="27.94" x2="24.13" y2="27.94" width="0" layer="19" extent="1-1"/>
+<wire x1="30.48" y1="27.94" x2="24.13" y2="27.94" width="0.6096" layer="16"/>
 </signal>
 <signal name="E">
 <contactref element="U$1" pad="4"/>
 <contactref element="IC1" pad="24"/>
-<wire x1="30.48" y1="25.4" x2="24.13" y2="25.4" width="0" layer="19" extent="1-1"/>
+<wire x1="24.13" y1="25.4" x2="30.48" y2="25.4" width="0.6096" layer="16"/>
 </signal>
 <signal name="RS">
 <contactref element="U$1" pad="3"/>
 <contactref element="IC1" pad="23"/>
-<wire x1="30.48" y1="22.86" x2="24.13" y2="22.86" width="0" layer="19" extent="1-1"/>
+<wire x1="30.48" y1="22.86" x2="24.13" y2="22.86" width="0.6096" layer="16"/>
 </signal>
 </signals>

Commit message: ...
Parts:
- R4: device r:0204/15 -> r:0204/10
- moved R4 9.16 mm to (7.62, 7.62), turned to 0 degrees
- renumbered U$1 to J2
Routing:
- net N$2: track 24.1 -> 39.4 mm
Changed lines of the file:
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@@
 <element name="IC1" library="mcu" package="DIL28-3/V" value="PIC16F876A-X/SP-COMPDIL28-3/V" x="20.32" y="19.05"/>
 <element name="R3" library="r" package="0204/10" value="10k" x="7.62" y="33.02" rot="R180"/>
-<element name="R4" library="r" package="0204/15" value="1.5k" x="12.7" y="15.24" rot="R270"/>
+<element name="R4" library="r" package="0204/10" value="1.5k" x="7.62" y="7.62"/>
 <element name="R5" library="r" package="0204/10" value="1.5k" x="7.62" y="25.4"/>
 <element name="C1" library="c" package="C050-020X036" value="270pF" x="7.62" y="30.48" rot="R90"/>
@@
 <element name="J1" library="pinconn" package="CONN-2P" value="CONN-2P2P/H" x="29.21" y="5.08"/>
 <element name="C2" library="c" package="C025-020X036" value="100nF" x="27.94" y="13.97" rot="R270"/>
-<element name="U$1" library="lcd" package="1X8" value="LCD-8PIN" x="30.48" y="26.67" rot="R90"/>
+<element name="J2" library="lcd" package="1X8" value="LCD-8PIN" x="30.48" y="26.67" rot="R90"/>
 </elements>
 <signals>
@@
 <contactref element="TEST-" pad="1"/>
 <wire x1="2.54" y1="15.24" x2="2.54" y2="22.86" width="0.6096" layer="16"/>
-<wire x1="2.54" y1="22.86" x2="12.7" y2="22.86" width="0.6096" layer="16"/>
-<wire x1="12.7" y1="22.86" x2="12.7" y2="17.78" width="0.6096" layer="16"/>
-<wire x1="12.7" y1="17.78" x2="16.51" y2="17.78" width="0.6096" layer="16"/>
+<wire x1="2.54" y1="22.86" x2="2.54" y2="27.94" width="0.6096" layer="16"/>
 <wire x1="19.05" y1="17.78" x2="19.05" y2="12.7" width="0.6096" layer="16"/>
 <contactref element="J1" pad="1"/>
@@
 <wire x1="5.08" y1="38.1" x2="5.08" y2="33.02" width="0.6096" layer="16"/>
 <wire x1="27.94" y1="12.7" x2="24.13" y2="12.7" width="0.6096" layer="16"/>
-<wire x1="2.54" y1="27.94" x2="2.54" y2="22.86" width="0.6096" layer="16"/>
 <wire x1="5.08" y1="30.48" x2="5.08" y2="33.02" width="0.6096" layer="16"/>
 <wire x1="5.08" y1="33.02" x2="2.54" y2="33.02" width="0.6096" layer="16"/>
 <wire x1="2.54" y1="33.02" x2="2.54" y2="27.94" width="0.6096" layer="16"/>
+<wire x1="16.51" y1="17.78" x2="12.7" y2="17.78" width="0.6096" layer="16"/>
+<wire x1="12.7" y1="17.78" x2="12.7" y2="22.86" width="0.6096" layer="16"/>
+<wire x1="12.7" y1="22.86" x2="2.54" y2="22.86" width="0.6096" layer="16"/>
 </signal>
 <signal name="N$3">
@@
 <contactref element="R4" pad="1"/>
 <contactref element="R5" pad="1"/>
+<wire x1="2.54" y1="33.02" x2="2.54" y2="25.4" width="0.6096" layer="16"/>
+<wire x1="16.51" y1="22.86" x2="2.54" y2="22.86" width="0.6096" layer="16"/>
 <wire x1="2.54" y1="25.4" x2="2.54" y2="22.86" width="0.6096" layer="16"/>
-<wire x1="2.54" y1="22.86" x2="12.7" y2="22.86" width="0.6096" layer="16"/>
-<wire x1="12.7" y1="22.86" x2="16.51" y2="22.86" width="0.6096" layer="16"/>
-<wire x1="2.54" y1="33.02" x2="2.54" y2="25.4" width="0.6096" layer="16"/>
+<wire x1="2.54" y1="7.62" x2="2.54" y2="22.86" width="0.6096" layer="16"/>
 </signal>
 <signal name="N$4">
@@
 </signal>
 <signal name="D7">
-<contactref element="U$1" pad="8"/>
+<contactref element="J2" pad="8"/>
 <contactref element="IC1" pad="28"/>
 <wire x1="24.13" y1="35.56" x2="30.48" y2="35.56" width="0.6096" layer="16"/>
 </signal>
 <signal name="D6">
-<contactref element="U$1" pad="7"/>
+<contactref element="J2" pad="7"/>
 <contactref element="IC1" pad="27"/>
 <wire x1="30.48" y1="33.02" x2="24.13" y2="33.02" width="0.6096" layer="16"/>
 </signal>
 <signal name="D5">
-<contactref element="U$1" pad="6"/>
+<contactref element="J2" pad="6"/>
 <contactref element="IC1" pad="26"/>
 <wire x1="24.13" y1="30.48" x2="30.48" y2="30.48" width="0.6096" layer="16"/>
 </signal>
 <signal name="D4">
-<contactref element="U$1" pad="5"/>
+<contactref element="J2" pad="5"/>
 <contactref element="IC1" pad="25"/>
 <wire x1="30.48" y1="27.94" x2="24.13" y2="27.94" width="0.6096" layer="16"/>
 </signal>
 <signal name="E">
-<contactref element="U$1" pad="4"/>
+<contactref element="J2" pad="4"/>
 <contactref element="IC1" pad="24"/>
 <wire x1="24.13" y1="25.4" x2="30.48" y2="25.4" width="0.6096" layer="16"/>
 </signal>
 <signal name="RS">
-<contactref element="U$1" pad="3"/>
+<contactref element="J2" pad="3"/>
 <contactref element="IC1" pad="23"/>
 <wire x1="30.48" y1="22.86" x2="24.13" y2="22.86" width="0.6096" layer="16"/>
