File: eagle/LCmeter0-LCD-8pinlcd-PIC18F2550-COMP.brd (EAGLE design)
At the start: 61 x 53.3 mm, 35 parts, among them IC1 PIC18F2550-I/SP-COMP-B-V, J1 HD44780-4BITLCD44780-8P, J2 PIC-UART, J3 PIC-ICSP, J4 J4, J5 CONN-2P2P/V, J7 CONN-2P2P/V, K2 DS2Y, Q1 20MHz, SW1 PB-1P-1T, T1 BC547

Commit message: ...
Parts:
- moved LED1 2.54 mm to (26.7, 12.7)
- moved R11 2.54 mm to (33.0, 12.7)
Routing:
- net A0: track 10.2 -> 30.5 mm
- net GND: track 218.4 -> 233.7 mm
- net VCC: track 144.8 -> 152.4 mm
- net RS: track 0.00 -> 7.62 mm
- net N$9: track 0.00 -> 7.62 mm
- net N$10: track 0.00 -> 7.62 mm
- net E: track 0.00 -> 7.62 mm
- net D7: track 2.54 -> 10.2 mm
- net D5: track 0.00 -> 7.62 mm
- net D4: track 0.00 -> 7.62 mm
- net FREQ: track 40.6 -> 47.5 mm
- net OSC2: track 7.62 -> 12.7 mm
- net OSC1: track 5.08 -> 10.2 mm
- net A3: track 38.1 -> 43.2 mm
- net /MCLR: track 22.9 -> 27.9 mm
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
Commit message: ...
Parts:
- moved R11 49.4 mm to (77.5, 34.3), turned to 180 degrees
- moved LED1 47.1 mm to (72.4, 24.1), turned to 270 degrees
- moved C2 7.62 mm to (20.3, 35.6)
- moved J7 3.59 mm to (2.54, 15.2)
- moved J5 3.59 mm to (2.54, 5.08)
- moved C3 3.59 mm to (24.1, 40.6)
- moved C4 3.59 mm to (24.1, 35.6)
- moved K2 2.54 mm to (21.6, 14.0)
- moved L1 2.54 mm to (10.2, 35.6)
- moved R4 2.54 mm to (31.8, 35.6)
- moved SW1 2.54 mm to (20.3, 45.7)
Connections:
- net N$10 renamed /TX
- net N$9 renamed /RX
- net /LC: now also IC1.13; no longer IC1.15
- net /RELAY: now also IC1.12, R6.1; no longer D1.A, K2.1, T1.C
- net N$3: now also IC1.4; no longer IC1.12
- net N$8: now also D1.A, K2.1, T1.C; no longer IC1.16, R6.1
Routing:
- net /LC: track 68.4 -> 43.8 mm
- net A3: track 43.2 -> 54.6 mm, vias 2 -> 7
- net A0: track 30.5 -> 21.4 mm
- net FREQ: track 47.5 -> 38.7 mm
- net C2_CON: track 30.5 -> 22.4 mm
- net IN+: track 20.3 -> 12.3 mm, vias 2 -> 0
- net /RELAY: track 5.08 -> 11.2 mm
- net N$7: track 22.9 -> 18.8 mm
- net N$3: track 2.54 -> 0.00 mm
- net N$1: track 2.54 -> 0.00 mm
- net /MCLR: track 27.9 -> 30.5 mm
- net VCC: track 152.4 -> 154.8 mm
- net PGC: track 7.62 -> 6.13 mm
- net A1: track 17.8 -> 16.3 mm
- net N$8: track 2.54 -> 3.59 mm
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Other:
- board size 61 x 53.3 mm -> 58.4 x 50.8 mm

Commit message: ...
Parts:
- moved R6 12.0 mm to (36.8, 2.54), turned to 90 degrees
- moved T1 2.54 mm to (27.9, 2.54)
- moved D1 2.54 mm to (21.6, 2.54)
Routing:
- net N$6: track 20.3 -> 2.54 mm
- net N$8: track 3.59 -> 5.08 mm
- net VCC: track 154.8 -> 153.8 mm
Changed lines of the file:
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@@
 </element>
 <element name="C9" library="c" package="C025-020X036/V" value="100nF" x="50.8" y="19.05"/>
-<element name="D1" library="d" package="DO34-7" value="1N4148" x="19.05" y="2.54"/>
+<element name="D1" library="d" package="DO34-7" value="1N4148" x="21.59" y="2.54"/>
 <element name="L1" library="r" package="0207/10" value="82μH" x="10.16" y="35.56" rot="R90"/>
 <element name="Q1" library="q" package="HC49" value="20MHz" x="33.02" y="17.78"/>
@@
 <attribute name="VALUE" x="19.05" y="5.08" size="1.27" layer="27"/>
 </element>
-<element name="T1" library="t" package="TO92-CBE-A" value="BC547" x="25.4" y="2.54"/>
+<element name="T1" library="t" package="TO92-CBE-A" value="BC547" x="27.94" y="2.54"/>
 <element name="S1" library="sw" package="SLSW-2P2T" value="SL-SW-2P-2T" x="3.81" y="27.94"/>
 <element name="R7" library="r" package="0202/10-V" value="10k" x="10.16" y="10.16"/>
@@
 <element name="J2" library="pinconn" package="PIC-UART" value="PIC-UART" x="53.34" y="12.7"/>
 <element name="SW1" library="sw" package="PB-1P1T" value="PB-1P-1T" x="20.32" y="45.72" rot="R180"/>
-<element name="R6" library="r" package="0202/7-V" value="10k" x="48.26" y="6.35" rot="R180"/>
+<element name="R6" library="r" package="0202/7-V" value="10k" x="36.83" y="2.54" rot="R90"/>
 <element name="R11" library="r" package="0202/5-V" value="1k" x="77.47" y="34.29" rot="R180"/>
 <element name="J7" library="pinconn" package="CONN-2P-V" value="CONN-2P2P/V" x="2.54" y="15.24"/>
@@
 <wire x1="25.4" y1="20.32" x2="25.4" y2="22.86" width="0.6096" layer="16"/>
 <wire x1="25.4" y1="22.86" x2="35.56" y2="22.86" width="0.6096" layer="16"/>
-<wire x1="25.4" y1="0" x2="50.8" y2="0" width="0.6096" layer="16"/>
-<wire x1="25.4" y1="0" x2="7.62" y2="0" width="0.6096" layer="16"/>
+<wire x1="27.94" y1="0" x2="50.8" y2="0" width="0.6096" layer="16"/>
+<wire x1="27.94" y1="0" x2="7.62" y2="0" width="0.6096" layer="16"/>
 <wire x1="7.62" y1="0" x2="5.08" y2="2.54" width="0.6096" layer="16"/>
 <contactref element="J1" pad="GND"/>
@@
 <via x="38.1" y="43.18" extent="1-16" drill="0.6" shape="square"/>
 <contactref element="D1" pad="C"/>
-<wire x1="15.24" y1="2.54" x2="17.78" y2="5.08" width="0.6096" layer="16"/>
+<wire x1="17.78" y1="2.54" x2="17.78" y2="5.08" width="0.6096" layer="16"/>
 <contactref element="R10" pad="1"/>
 <contactref element="J1" pad="VCC"/>
@@
 <contactref element="T1" pad="C"/>
 <contactref element="D1" pad="A"/>
-<wire x1="25.4" y1="5.08" x2="22.86" y2="2.54" width="0.6096" layer="16"/>
+<wire x1="27.94" y1="5.08" x2="25.4" y2="5.08" width="0.6096" layer="16"/>
+<wire x1="25.4" y1="5.08" x2="25.4" y2="2.54" width="0.6096" layer="16"/>
 </signal>
 <signal name="/MCLR">
@@
 <contactref element="T1" pad="B"/>
 <contactref element="R6" pad="2"/>
-<wire x1="27.94" y1="2.54" x2="48.26" y2="2.54" width="0.6096" layer="16"/>
+<wire x1="30.48" y1="2.54" x2="33.02" y2="2.54" width="0.6096" layer="16"/>
 </signal>
 <signal name="/RELAY">
 <contactref element="R6" pad="1"/>
 <contactref element="IC1" pad="12"/>
-<wire x1="38.1" y1="12.7" x2="39.37" y2="12.7" width="0.6096" layer="16"/>
-<wire x1="39.37" y1="12.7" x2="40.64" y2="11.43" width="0.6096" layer="16"/>
-<wire x1="40.64" y1="11.43" x2="46.99" y2="11.43" width="0.6096" layer="16"/>
-<wire x1="46.99" y1="11.43" x2="48.26" y2="10.16" width="0.6096" layer="16"/>
+<wire x1="38.1" y1="12.7" x2="40.64" y2="10.16" width="0.6096" layer="16"/>
+<wire x1="40.64" y1="10.16" x2="40.64" y2="2.54" width="0.6096" layer="16"/>
 </signal>
 <signal name="/RX">

Commit message: ...
Connections:
- net /MCLR: now also IC1.1
Changed lines of the file:
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@@
 <?xml version="1.0" encoding="utf-8"?>
 <!DOCTYPE eagle SYSTEM "eagle.dtd">
-<eagle version="7.7.0">
+<eagle version="7.6.0">
 <drawing>
 <settings>
@@
 <wire x1="33.02" y1="45.72" x2="22.86" y2="45.72" width="0.6096" layer="16"/>
 <wire x1="35.56" y1="40.64" x2="40.64" y2="40.64" width="0.6096" layer="16"/>
+<contactref element="IC1" pad="1"/>
+<wire x1="35.56" y1="40.64" x2="38.1" y2="40.64" width="0" layer="19" extent="1-1"/>
 </signal>
 <signal name="D5">

Commit message: ...
Other:
- board outline removed
