File: eagle/LCmeter0-LCD-8pinlcd-PIC_COMP.brd (EAGLE design)
At the start: 34 parts, among them IC1 PIC16F876A-X/SP-COMP-B-A, J1 HD44780-4BIT-8PIN, J2 PIC-UART, J3 PIC-ICSP, K2 DS2Y, Q1 20MHz, T1 BC547CBE-A, X1 FREQ, X2 L/C

Commit message: ...
Parts:
- J3: value PIC-ICSP -> PIC-ICSPICSP; device pinconn:CONN-5P -> pinconn:PIC-ICSP
- moved J3 5.08 mm to (40.6, 48.3)
Changed lines of the file:
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@@
 <?xml version="1.0" encoding="utf-8"?>
 <!DOCTYPE eagle SYSTEM "eagle.dtd">
-<eagle version="7.7.0">
+<eagle version="7.2.0">
 <drawing>
 <settings>
@@
 <setting verticaltext="up"/>
 </settings>
-<grid distance="0.05" unitdist="inch" unit="inch" style="lines" multiple="2" display="yes" altdistance="0.0125" altunitdist="inch" altunit="inch"/>
+<grid distance="50" unitdist="mil" unit="mil" style="dots" multiple="2" display="yes" altdistance="0.0125" altunitdist="inch" altunit="inch"/>
 <layers>
 <layer number="1" name="Top" color="4" fill="1" visible="yes" active="yes"/>
@@
 <layer number="21" name="tPlace" color="7" fill="1" visible="yes" active="yes"/>
 <layer number="22" name="bPlace" color="7" fill="1" visible="yes" active="yes"/>
-<layer number="23" name="tOrigins" color="15" fill="1" visible="no" active="yes"/>
-<layer number="24" name="bOrigins" color="15" fill="1" visible="no" active="yes"/>
+<layer number="23" name="tOrigins" color="15" fill="1" visible="yes" active="yes"/>
+<layer number="24" name="bOrigins" color="15" fill="1" visible="yes" active="yes"/>
 <layer number="25" name="tNames" color="7" fill="1" visible="yes" active="yes"/>
 <layer number="26" name="bNames" color="7" fill="1" visible="yes" active="yes"/>
@@
 </element>
 <element name="R7" library="r" package="0202/10" value="10kΩ" x="10.16" y="10.16" rot="R270"/>
-<element name="J3" library="pinconn" package="CONN-5P" value="PIC-ICSP" x="35.56" y="48.26"/>
+<element name="J3" library="pinconn" package="PIC-ICSP" value="PIC-ICSPICSP" x="40.64" y="48.26"/>
 <element name="R8" library="r" package="0202/5" value="100" x="48.26" y="45.72" rot="R180"/>
 <element name="R9" library="r" package="0202/5" value="100" x="48.26" y="40.64" rot="R90"/>

Commit message: ...
Parts:
- IC1: value PIC16F876A-X/SP-COMP-B-A -> PIC16F876A-X/SP-COMP-B-A/V; device mcu:DIL28-3 -> mcu:DIL28-3/V
- moved IC1 54.3 mm to (-11.4, 14.0), turned to 0 degrees
Connections:
- net FREQ: now also IC1.11, R11.2
Routing:
- net A0: track 30.5 -> 10.2 mm
- net GND: track 190.5 -> 172.7 mm
- net RS: track 7.62 -> 0.00 mm
- net E: track 7.62 -> 0.00 mm
- net D5: track 7.62 -> 0.00 mm
- net D4: track 7.62 -> 0.00 mm
- net OSC2: track 12.7 -> 7.62 mm
- net OSC1: track 10.2 -> 5.08 mm
- net D7: track 12.7 -> 7.62 mm
- net A3: track 43.2 -> 38.1 mm
- net /MCLR: track 27.9 -> 22.9 mm
- net D6: track 7.62 -> 5.08 mm
- net A4: track 2.54 -> 0.00 mm
- net A1: track 17.8 -> 15.2 mm
Changed lines of the file:
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@@
 <element name="J2" library="pinconn" package="PIC-UART" value="PIC-UART" x="54.61" y="11.43" rot="R90"/>
 <element name="U$1" library="sw" package="PB-1P1T" value="PB-1P-1T" x="22.86" y="45.72" rot="R180"/>
-<element name="IC1" library="mcu" package="DIL28-3" value="PIC16F876A-X/SP-COMP-B-A" x="41.91" y="24.13" smashed="yes" rot="R270">
-<attribute name="NAME" x="39.37" y="42.037" size="1.27" layer="25"/>
-<attribute name="VALUE" x="41.2877" y="33.8455" size="1.016" layer="27" rot="R270"/>
-</element>
+<element name="IC1" library="mcu" package="DIL28-3/V" value="PIC16F876A-X/SP-COMP-B-A/V" x="-11.43" y="13.97"/>
 </elements>
 <signals>
@@
 <wire x1="25.4" y1="38.1" x2="22.86" y2="38.1" width="1.27" layer="16"/>
 <contactref element="IC1" pad="5"/>
-<wire x1="38.1" y1="30.48" x2="33.02" y2="30.48" width="1.27" layer="16"/>
+<wire x1="-15.24" y1="20.32" x2="25.4" y2="25.4" width="0" layer="19" extent="16-16"/>
 </signal>
 <signal name="N$2">
@@
 <contactref element="IC1" pad="2"/>
 <contactref element="IC1" pad="7"/>
-<wire x1="38.1" y1="38.1" x2="35.56" y2="38.1" width="1.27" layer="16"/>
-<wire x1="38.1" y1="25.4" x2="40.64" y2="25.4" width="1.27" layer="16"/>
-<wire x1="40.64" y1="25.4" x2="40.64" y2="38.1" width="1.27" layer="16"/>
-<wire x1="40.64" y1="38.1" x2="38.1" y2="38.1" width="1.27" layer="16"/>
+<wire x1="-15.24" y1="27.94" x2="33.02" y2="33.02" width="0" layer="19" extent="16-16"/>
+<wire x1="-15.24" y1="15.24" x2="-15.24" y2="27.94" width="0" layer="19" extent="1-1"/>
 </signal>
 <signal name="A1">
@@
 <wire x1="27.94" y1="35.56" x2="27.94" y2="33.02" width="1.27" layer="16"/>
 <contactref element="IC1" pad="3"/>
-<wire x1="35.56" y1="35.56" x2="38.1" y2="35.56" width="1.27" layer="16"/>
+<wire x1="-15.24" y1="25.4" x2="22.86" y2="33.02" width="0" layer="19" extent="1-1"/>
 </signal>
 <signal name="GND">
@@
 <via x="17.78" y="45.72" extent="1-16" drill="0.6" shape="square"/>
 <wire x1="17.78" y1="45.72" x2="17.78" y2="33.02" width="1.27" layer="1"/>
-<contactref element="IC1" pad="19"/>
-<contactref element="IC1" pad="8"/>
-<wire x1="35.56" y1="22.86" x2="38.1" y2="22.86" width="1.27" layer="16"/>
-<wire x1="38.1" y1="22.86" x2="40.64" y2="22.86" width="1.27" layer="16"/>
-<wire x1="40.64" y1="22.86" x2="40.64" y2="17.78" width="1.27" layer="16"/>
-<wire x1="40.64" y1="17.78" x2="45.72" y2="17.78" width="1.27" layer="16"/>
-<wire x1="48.26" y1="17.78" x2="45.72" y2="17.78" width="1.27" layer="16"/>
 <polygon width="0.254" layer="16" isolate="1.27">
 <vertex x="-2.54" y="50.8"/>
@@
 <vertex x="58.42" y="50.8"/>
 </polygon>
+<contactref element="IC1" pad="19"/>
+<contactref element="IC1" pad="8"/>
+<wire x1="-7.62" y1="7.62" x2="-15.24" y2="12.7" width="0" layer="19" extent="1-1"/>
+<wire x1="2.54" y1="5.08" x2="-7.62" y2="7.62" width="0" layer="19" extent="16-16"/>
 </signal>
 <signal name="N$7">
@@
 <wire x1="27.94" y1="20.32" x2="33.02" y2="20.32" width="1.27" layer="16"/>
 <contactref element="IC1" pad="9"/>
-<wire x1="33.02" y1="20.32" x2="38.1" y2="20.32" width="1.27" layer="16"/>
+<wire x1="-15.24" y1="10.16" x2="27.94" y2="20.32" width="0" layer="19" extent="1-1"/>
 </signal>
 <signal name="OSC2">
@@
 <wire x1="33.02" y1="17.78" x2="27.94" y2="17.78" width="1.27" layer="16"/>
 <contactref element="IC1" pad="10"/>
-<wire x1="38.1" y1="17.78" x2="33.02" y2="17.78" width="1.27" layer="16"/>
+<wire x1="-15.24" y1="7.62" x2="27.94" y2="17.78" width="0" layer="19" extent="1-1"/>
 </signal>
 <signal name="VCC">
@@
 <contactref element="J1" pad="5"/>
 <contactref element="IC1" pad="25"/>
-<wire x1="45.72" y1="33.02" x2="53.34" y2="33.02" width="1.27" layer="16"/>
+<wire x1="-7.62" y1="22.86" x2="53.34" y2="33.02" width="0" layer="19" extent="1-1"/>
 </signal>
 <signal name="E">
 <contactref element="J1" pad="4"/>
 <contactref element="IC1" pad="24"/>
-<wire x1="53.34" y1="30.48" x2="45.72" y2="30.48" width="1.27" layer="16"/>
+<wire x1="-7.62" y1="20.32" x2="53.34" y2="30.48" width="0" layer="19" extent="1-1"/>
 </signal>
 <signal name="RS">
 <contactref element="J1" pad="3"/>
 <contactref element="IC1" pad="23"/>
-<wire x1="45.72" y1="27.94" x2="53.34" y2="27.94" width="1.27" layer="16"/>
+<wire x1="-7.62" y1="17.78" x2="53.34" y2="27.94" width="0" layer="19" extent="1-1"/>
 </signal>
 <signal name="A4">
 <contactref element="R5" pad="2"/>
 <contactref element="IC1" pad="6"/>
-<wire x1="35.56" y1="27.94" x2="38.1" y2="27.94" width="1.27" layer="16"/>
+<wire x1="-15.24" y1="17.78" x2="35.56" y2="27.94" width="0" layer="19" extent="1-1"/>
 </signal>
 <signal name="/LC">
@@
 <wire x1="35.56" y1="45.72" x2="25.4" y2="45.72" width="1.27" layer="16"/>
 <contactref element="IC1" pad="1"/>
-<wire x1="38.1" y1="40.64" x2="40.64" y2="40.64" width="1.27" layer="16"/>
-<wire x1="38.1" y1="40.64" x2="35.56" y2="40.64" width="1.27" layer="16"/>
+<wire x1="40.64" y1="40.64" x2="35.56" y2="40.64" width="0" layer="19" extent="16-16"/>
+<wire x1="-15.24" y1="30.48" x2="25.4" y2="45.72" width="0" layer="19" extent="1-1"/>
 </signal>
 <signal name="RC5">
@@
 <contactref element="J1" pad="6"/>
 <contactref element="IC1" pad="26"/>
-<wire x1="53.34" y1="35.56" x2="45.72" y2="35.56" width="1.27" layer="16"/>
+<wire x1="-7.62" y1="25.4" x2="53.34" y2="35.56" width="0" layer="19" extent="1-1"/>
 </signal>
 <signal name="D6">
@@
 <wire x1="48.26" y1="38.1" x2="53.34" y2="38.1" width="1.27" layer="16"/>
 <contactref element="IC1" pad="27"/>
-<wire x1="45.72" y1="38.1" x2="48.26" y2="38.1" width="1.27" layer="16"/>
+<wire x1="-7.62" y1="27.94" x2="48.26" y2="38.1" width="0" layer="19" extent="1-1"/>
 </signal>
 <signal name="D7">
@@
 <wire x1="53.34" y1="40.64" x2="50.8" y2="40.64" width="1.27" layer="16"/>
 <contactref element="IC1" pad="28"/>
-<wire x1="45.72" y1="40.64" x2="50.8" y2="40.64" width="1.27" layer="16"/>
+<wire x1="-7.62" y1="30.48" x2="50.8" y2="40.64" width="0" layer="19" extent="16-16"/>
 </signal>
 <signal name="C2_CON">
@@
 <wire x1="5.08" y1="7.62" x2="33.02" y2="7.62" width="1.27" layer="16"/>
 <wire x1="33.02" y1="7.62" x2="33.02" y2="10.16" width="1.27" layer="16"/>
+<contactref element="IC1" pad="11"/>
+<contactref element="R11" pad="2"/>
+<wire x1="33.02" y1="10.16" x2="38.1" y2="10.16" width="0" layer="19" extent="16-16"/>
+<wire x1="-15.24" y1="5.08" x2="5.08" y2="7.62" width="0" layer="19" extent="1-1"/>
 </signal>
 <signal name="N$1">

Commit message: ...
Parts:
- moved IC1 54.3 mm to (41.9, 24.1)
- moved R11 2.54 mm to (33.0, 10.2)
Connections:
- removed net N$8: J2.17
- new net N$4: IC1.13, R11.2
- new net TX: IC1.17, J2.17
- net /LC: now also IC1.15
- net FREQ: no longer R11.2
- net RC5: now also IC1.16
- net RX: now also IC1.18
- net VCC: now also IC1.20
Routing:
- net A0: track 10.2 -> 30.5 mm
- net GND: track 172.7 -> 190.5 mm
- net FREQ: track 30.5 -> 40.6 mm
- net TX: track 0.00 -> 7.62 mm
- net RX: track 0.00 -> 7.62 mm
- net RS: track 0.00 -> 7.62 mm
- net E: track 0.00 -> 7.62 mm
- net D5: track 0.00 -> 7.62 mm
- net D4: track 0.00 -> 7.62 mm
- net OSC2: track 7.62 -> 12.7 mm
- net OSC1: track 5.08 -> 10.2 mm
- net D7: track 7.62 -> 12.7 mm
- net A3: track 38.1 -> 43.2 mm
- net /MCLR: track 22.9 -> 27.9 mm
- net /LC: track 68.4 -> 73.5 mm
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
Commit message: ...
Parts:
- C7: device c:E2,5-6 -> c:E2,5-5
- R1: device r:0202/7 -> r:0204/10
Routing:
- net VCC: track 144.8 -> 150.5 mm
- net GND: track 190.5 -> 192.2 mm
- net A3: track 43.2 -> 41.9 mm
Changed lines of the file:
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@@
 <element name="C5" library="c" package="C025-020X036" value="33pF" x="25.4" y="17.78"/>
 <element name="C6" library="c" package="C025-020X036" value="33pF" x="25.4" y="20.32"/>
-<element name="C7" library="c" package="E2,5-6" value="100μF" x="52.07" y="7.62" rot="R180"/>
+<element name="C7" library="c" package="E2,5-5" value="100μF" x="52.07" y="7.62" rot="R180"/>
 <element name="C9" library="rcl" package="C025-024X044" value="100nF" x="50.8" y="19.05" smashed="yes" rot="R270">
 <attribute name="NAME" x="49.53" y="16.51" size="1.27" layer="25" ratio="10" rot="R270"/>
@@
 <element name="L1" library="r" package="L-02/5" value="100μH" x="10.16" y="43.18" rot="R90"/>
 <element name="Q1" library="q" package="HC49" value="20MHz" x="33.02" y="17.78" rot="R270"/>
-<element name="R1" library="r" package="0202/7" value="100kΩ" x="31.75" y="38.1" rot="R180"/>
+<element name="R1" library="r" package="0204/10" value="100kΩ" x="31.75" y="38.1" rot="R180"/>
 <element name="R10" library="r" package="0202/7" value="4.7kΩ" x="31.75" y="40.64" rot="R180"/>
 <element name="R2" library="r" package="0202/7" value="100kΩ" x="31.75" y="25.4"/>
@@
 <wire x1="33.02" y1="25.4" x2="33.02" y2="30.48" width="1.27" layer="16"/>
 <wire x1="27.94" y1="43.18" x2="25.4" y2="43.18" width="1.27" layer="16"/>
-<wire x1="25.4" y1="38.1" x2="27.94" y2="38.1" width="1.27" layer="16"/>
+<wire x1="25.4" y1="38.1" x2="26.67" y2="38.1" width="1.27" layer="16"/>
 <wire x1="27.94" y1="25.4" x2="25.4" y2="25.4" width="1.27" layer="16"/>
 <via x="25.4" y="38.1" extent="1-16" drill="0.6" shape="square"/>
@@
 <wire x1="35.56" y1="33.02" x2="33.02" y2="33.02" width="1.27" layer="16"/>
 <wire x1="33.02" y1="33.02" x2="33.02" y2="38.1" width="1.27" layer="16"/>
-<wire x1="33.02" y1="38.1" x2="35.56" y2="38.1" width="1.27" layer="16"/>
+<wire x1="33.02" y1="38.1" x2="36.83" y2="38.1" width="1.27" layer="16"/>
 <contactref element="IC1" pad="2"/>
 <contactref element="IC1" pad="7"/>
-<wire x1="35.56" y1="38.1" x2="38.1" y2="38.1" width="1.27" layer="16"/>
+<wire x1="36.83" y1="38.1" x2="38.1" y2="38.1" width="1.27" layer="16"/>
 <wire x1="38.1" y1="25.4" x2="40.64" y2="25.4" width="1.27" layer="16"/>
 <wire x1="40.64" y1="25.4" x2="40.64" y2="38.1" width="1.27" layer="16"/>
@@
 <wire x1="25.4" y1="0" x2="50.8" y2="0" width="1.27" layer="16"/>
 <wire x1="50.8" y1="0" x2="50.8" y2="2.54" width="1.27" layer="16"/>
-<wire x1="50.8" y1="2.54" x2="50.8" y2="7.62" width="1.27" layer="16"/>
+<wire x1="50.8" y1="2.54" x2="53.34" y2="7.62" width="1.27" layer="16"/>
 <wire x1="25.4" y1="0" x2="2.54" y2="0" width="1.27" layer="16"/>
 <contactref element="J3" pad="1"/>
@@
 <contactref element="J2" pad="19"/>
 <wire x1="53.34" y1="17.78" x2="55.88" y2="17.78" width="1.27" layer="16"/>
-<wire x1="50.8" y1="7.62" x2="50.8" y2="10.16" width="1.27" layer="16"/>
+<wire x1="53.34" y1="7.62" x2="50.8" y2="10.16" width="1.27" layer="16"/>
 <wire x1="50.8" y1="10.16" x2="55.88" y2="10.16" width="1.27" layer="16"/>
 <wire x1="55.88" y1="10.16" x2="55.88" y2="17.78" width="1.27" layer="16"/>
@@
 <contactref element="J1" pad="2"/>
 <contactref element="JP1" pad="1"/>
-<wire x1="53.34" y1="2.54" x2="53.34" y2="7.62" width="1.27" layer="16"/>
-<wire x1="55.88" y1="7.62" x2="53.34" y2="7.62" width="1.27" layer="16"/>
+<wire x1="53.34" y1="2.54" x2="50.8" y2="7.62" width="1.27" layer="16"/>
+<wire x1="55.88" y1="7.62" x2="50.8" y2="7.62" width="1.27" layer="16"/>
 <contactref element="J2" pad="20"/>
 <wire x1="53.34" y1="20.32" x2="55.88" y2="20.32" width="1.27" layer="16"/>
@@
 <wire x1="43.18" y1="20.32" x2="45.72" y2="20.32" width="1.27" layer="16"/>
 <contactref element="R7" pad="2"/>
-<wire x1="10.16" y1="5.08" x2="12.7" y2="5.08" width="0" layer="19" extent="16-16"/>
+<wire x1="10.16" y1="5.08" x2="12.7" y2="5.08" width="1.27" layer="16"/>
 </signal>
 <signal name="D4">

Commit message: ...
Parts:
- R1: device r:0204/10 -> r:0202/7
Routing:
- net A3: track 41.9 -> 43.2 mm
Changed lines of the file:
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@@
 <layer number="23" name="tOrigins" color="15" fill="1" visible="yes" active="yes"/>
 <layer number="24" name="bOrigins" color="15" fill="1" visible="yes" active="yes"/>
-<layer number="25" name="tNames" color="7" fill="1" visible="no" active="yes"/>
+<layer number="25" name="tNames" color="7" fill="1" visible="yes" active="yes"/>
 <layer number="26" name="bNames" color="7" fill="1" visible="no" active="yes"/>
-<layer number="27" name="tValues" color="7" fill="1" visible="no" active="yes"/>
+<layer number="27" name="tValues" color="7" fill="1" visible="yes" active="yes"/>
 <layer number="28" name="bValues" color="7" fill="1" visible="no" active="yes"/>
 <layer number="29" name="tStop" color="7" fill="3" visible="no" active="yes"/>
@@
 <layer number="46" name="Milling" color="3" fill="1" visible="no" active="yes"/>
 <layer number="47" name="Measures" color="7" fill="1" visible="no" active="yes"/>
-<layer number="48" name="Document" color="7" fill="1" visible="no" active="yes"/>
-<layer number="49" name="Reference" color="7" fill="1" visible="no" active="yes"/>
+<layer number="48" name="Document" color="7" fill="1" visible="yes" active="yes"/>
+<layer number="49" name="Reference" color="7" fill="1" visible="yes" active="yes"/>
 <layer number="51" name="tDocu" color="6" fill="1" visible="yes" active="yes"/>
 <layer number="52" name="bDocu" color="7" fill="1" visible="no" active="yes"/>
@@
 <element name="L1" library="r" package="L-02/5" value="100μH" x="10.16" y="43.18" rot="R90"/>
 <element name="Q1" library="q" package="HC49" value="20MHz" x="33.02" y="17.78" rot="R270"/>
-<element name="R1" library="r" package="0204/10" value="100kΩ" x="31.75" y="38.1" rot="R180"/>
+<element name="R1" library="r" package="0202/7" value="100kΩ" x="31.75" y="38.1" rot="R180"/>
 <element name="R10" library="r" package="0202/7" value="4.7kΩ" x="31.75" y="40.64" rot="R180"/>
 <element name="R2" library="r" package="0202/7" value="100kΩ" x="31.75" y="25.4"/>
@@
 <wire x1="33.02" y1="25.4" x2="33.02" y2="30.48" width="1.27" layer="16"/>
 <wire x1="27.94" y1="43.18" x2="25.4" y2="43.18" width="1.27" layer="16"/>
-<wire x1="25.4" y1="38.1" x2="26.67" y2="38.1" width="1.27" layer="16"/>
+<wire x1="25.4" y1="38.1" x2="27.94" y2="38.1" width="1.27" layer="16"/>
 <wire x1="27.94" y1="25.4" x2="25.4" y2="25.4" width="1.27" layer="16"/>
 <via x="25.4" y="38.1" extent="1-16" drill="0.6" shape="square"/>
@@
 <wire x1="35.56" y1="33.02" x2="33.02" y2="33.02" width="1.27" layer="16"/>
 <wire x1="33.02" y1="33.02" x2="33.02" y2="38.1" width="1.27" layer="16"/>
-<wire x1="33.02" y1="38.1" x2="36.83" y2="38.1" width="1.27" layer="16"/>
+<wire x1="33.02" y1="38.1" x2="35.56" y2="38.1" width="1.27" layer="16"/>
 <contactref element="IC1" pad="2"/>
 <contactref element="IC1" pad="7"/>
-<wire x1="36.83" y1="38.1" x2="38.1" y2="38.1" width="1.27" layer="16"/>
+<wire x1="35.56" y1="38.1" x2="38.1" y2="38.1" width="1.27" layer="16"/>
 <wire x1="38.1" y1="25.4" x2="40.64" y2="25.4" width="1.27" layer="16"/>
 <wire x1="40.64" y1="25.4" x2="40.64" y2="38.1" width="1.27" layer="16"/>

Commit message: ...
Parts:
- added R12: 4.7kΩ, r:0202/7
Connections:
- net /MCLR: now also R12.2
- net VCC: now also R12.1
Changed lines of the file:
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@@
 <layer number="23" name="tOrigins" color="15" fill="1" visible="yes" active="yes"/>
 <layer number="24" name="bOrigins" color="15" fill="1" visible="yes" active="yes"/>
-<layer number="25" name="tNames" color="7" fill="1" visible="yes" active="yes"/>
+<layer number="25" name="tNames" color="7" fill="1" visible="no" active="yes"/>
 <layer number="26" name="bNames" color="7" fill="1" visible="no" active="yes"/>
-<layer number="27" name="tValues" color="7" fill="1" visible="yes" active="yes"/>
+<layer number="27" name="tValues" color="7" fill="1" visible="no" active="yes"/>
 <layer number="28" name="bValues" color="7" fill="1" visible="no" active="yes"/>
 <layer number="29" name="tStop" color="7" fill="3" visible="no" active="yes"/>
@@
 <layer number="46" name="Milling" color="3" fill="1" visible="no" active="yes"/>
 <layer number="47" name="Measures" color="7" fill="1" visible="no" active="yes"/>
-<layer number="48" name="Document" color="7" fill="1" visible="yes" active="yes"/>
-<layer number="49" name="Reference" color="7" fill="1" visible="yes" active="yes"/>
+<layer number="48" name="Document" color="7" fill="1" visible="no" active="yes"/>
+<layer number="49" name="Reference" color="7" fill="1" visible="no" active="yes"/>
 <layer number="51" name="tDocu" color="6" fill="1" visible="yes" active="yes"/>
 <layer number="52" name="bDocu" color="7" fill="1" visible="no" active="yes"/>
@@
 <element name="U$1" library="sw" package="PB-1P1T" value="PB-1P-1T" x="22.86" y="45.72" rot="R180"/>
 <element name="IC1" library="mcu" package="DIL28-3/V" value="PIC16F876A-X/SP-COMP-B-A/V" x="41.91" y="24.13"/>
+<element name="R12" library="r" package="0202/7" value="4.7kΩ" x="0" y="-6.35"/>
 </elements>
 <signals>
@@
 <contactref element="R7" pad="2"/>
 <wire x1="10.16" y1="5.08" x2="12.7" y2="5.08" width="1.27" layer="16"/>
+<contactref element="R12" pad="1"/>
+<wire x1="-3.81" y1="-6.35" x2="10.16" y2="5.08" width="0" layer="19" extent="1-1"/>
 </signal>
 <signal name="D4">
@@
 <wire x1="36.83" y1="40.64" x2="38.1" y2="40.64" width="1.27" layer="16"/>
 <wire x1="40.64" y1="40.64" x2="38.1" y2="40.64" width="1.27" layer="16"/>
+<contactref element="R12" pad="2"/>
+<wire x1="3.81" y1="-6.35" x2="25.4" y2="45.72" width="0" layer="19" extent="1-1"/>
 </signal>
 <signal name="RC5">

Commit message: ...
Parts:
- moved R12 51.4 mm to (17.8, 41.9)
Changed lines of the file:
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@@
 <layer number="23" name="tOrigins" color="15" fill="1" visible="yes" active="yes"/>
 <layer number="24" name="bOrigins" color="15" fill="1" visible="yes" active="yes"/>
-<layer number="25" name="tNames" color="7" fill="1" visible="no" active="yes"/>
-<layer number="26" name="bNames" color="7" fill="1" visible="no" active="yes"/>
+<layer number="25" name="tNames" color="7" fill="1" visible="yes" active="yes"/>
+<layer number="26" name="bNames" color="7" fill="1" visible="yes" active="yes"/>
 <layer number="27" name="tValues" color="7" fill="1" visible="no" active="yes"/>
 <layer number="28" name="bValues" color="7" fill="1" visible="no" active="yes"/>
@@
 <element name="U$1" library="sw" package="PB-1P1T" value="PB-1P-1T" x="22.86" y="45.72" rot="R180"/>
 <element name="IC1" library="mcu" package="DIL28-3/V" value="PIC16F876A-X/SP-COMP-B-A/V" x="41.91" y="24.13"/>
-<element name="R12" library="r" package="0202/7" value="4.7kΩ" x="0" y="-6.35"/>
+<element name="R12" library="r" package="0202/7" value="4.7kΩ" x="17.78" y="41.91"/>
 </elements>
 <signals>
@@
 <wire x1="10.16" y1="5.08" x2="12.7" y2="5.08" width="1.27" layer="16"/>
 <contactref element="R12" pad="1"/>
-<wire x1="-3.81" y1="-6.35" x2="10.16" y2="5.08" width="0" layer="19" extent="1-1"/>
+<wire x1="27.94" y1="40.64" x2="13.97" y2="41.91" width="0" layer="19" extent="1-1"/>
 </signal>
 <signal name="D4">
@@
 <wire x1="35.56" y1="45.72" x2="25.4" y2="45.72" width="1.27" layer="16"/>
 <contactref element="IC1" pad="1"/>
-<wire x1="35.56" y1="40.64" x2="36.83" y2="40.64" width="1.27" layer="16"/>
-<wire x1="36.83" y1="40.64" x2="38.1" y2="40.64" width="1.27" layer="16"/>
+<wire x1="35.56" y1="40.64" x2="38.1" y2="40.64" width="1.27" layer="16"/>
 <wire x1="40.64" y1="40.64" x2="38.1" y2="40.64" width="1.27" layer="16"/>
 <contactref element="R12" pad="2"/>
-<wire x1="3.81" y1="-6.35" x2="25.4" y2="45.72" width="0" layer="19" extent="1-1"/>
+<wire x1="21.59" y1="41.91" x2="25.4" y2="45.72" width="0" layer="19" extent="1-1"/>
 </signal>
 <signal name="RC5">
