File: eagle/LCmeter0-LCD-8pinlcd-PIC_COMP.brd (EAGLE design)
At the start: 35 parts, among them IC1 PIC16F876A-X/SP-COMP-B-A/V, J1 HD44780-4BIT-8PIN, J2 PIC-UART, J3 PIC-ICSPICSP, K2 DS2Y, Q1 20MHz, T1 BC547CBE-A, X1 FREQ, X2 L/C

Commit message: ...
Parts:
- removed R12: 4.7kΩ, r:0202/7
Connections:
- net /MCLR: no longer R12.2
- net VCC: no longer R12.1
Changed lines of the file:
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@@
 <layer number="25" name="tNames" color="7" fill="1" visible="yes" active="yes"/>
 <layer number="26" name="bNames" color="7" fill="1" visible="yes" active="yes"/>
-<layer number="27" name="tValues" color="7" fill="1" visible="no" active="yes"/>
-<layer number="28" name="bValues" color="7" fill="1" visible="no" active="yes"/>
+<layer number="27" name="tValues" color="7" fill="1" visible="yes" active="yes"/>
+<layer number="28" name="bValues" color="7" fill="1" visible="yes" active="yes"/>
 <layer number="29" name="tStop" color="7" fill="3" visible="no" active="yes"/>
 <layer number="30" name="bStop" color="7" fill="6" visible="no" active="yes"/>
@@
 <layer number="46" name="Milling" color="3" fill="1" visible="no" active="yes"/>
 <layer number="47" name="Measures" color="7" fill="1" visible="no" active="yes"/>
-<layer number="48" name="Document" color="7" fill="1" visible="no" active="yes"/>
+<layer number="48" name="Document" color="7" fill="1" visible="yes" active="yes"/>
 <layer number="49" name="Reference" color="7" fill="1" visible="no" active="yes"/>
 <layer number="51" name="tDocu" color="6" fill="1" visible="yes" active="yes"/>
@@
 <element name="U$1" library="sw" package="PB-1P1T" value="PB-1P-1T" x="22.86" y="45.72" rot="R180"/>
 <element name="IC1" library="mcu" package="DIL28-3/V" value="PIC16F876A-X/SP-COMP-B-A/V" x="41.91" y="24.13"/>
-<element name="R12" library="r" package="0202/7" value="4.7kΩ" x="17.78" y="41.91"/>
 </elements>
 <signals>
@@
 <contactref element="R7" pad="2"/>
 <wire x1="10.16" y1="5.08" x2="12.7" y2="5.08" width="1.27" layer="16"/>
-<contactref element="R12" pad="1"/>
-<wire x1="27.94" y1="40.64" x2="13.97" y2="41.91" width="0" layer="19" extent="1-1"/>
 </signal>
 <signal name="D4">
@@
 <wire x1="35.56" y1="40.64" x2="38.1" y2="40.64" width="1.27" layer="16"/>
 <wire x1="40.64" y1="40.64" x2="38.1" y2="40.64" width="1.27" layer="16"/>
-<contactref element="R12" pad="2"/>
-<wire x1="21.59" y1="41.91" x2="25.4" y2="45.72" width="0" layer="19" extent="1-1"/>
 </signal>
 <signal name="RC5">
