File: eagle/CapMeter-LCD-16F628A.brd (EAGLE design)
At the start: 35.6 x 35.6 mm, 10 parts, among them IC1 PIC16F628A-COMP, Q1 20MHz

Commit message: ...
Routing:
- net GND: track 72.4 -> 87.6 mm
- net N$2: track 0.00 -> 5.08 mm
Changed lines of the file:
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@@
 <contactref element="R4" pad="2"/>
 <contactref element="R5" pad="2"/>
-<wire x1="12.7" y1="22.86" x2="15.24" y2="22.86" width="0.4064" layer="16"/>
-<wire x1="15.24" y1="22.86" x2="15.24" y2="27.94" width="0.4064" layer="16"/>
-<wire x1="15.24" y1="27.94" x2="12.7" y2="27.94" width="0.4064" layer="16"/>
-<wire x1="7.62" y1="15.24" x2="5.08" y2="15.24" width="0.4064" layer="16"/>
-<wire x1="12.7" y1="22.86" x2="7.62" y2="22.86" width="0.4064" layer="16"/>
-<wire x1="7.62" y1="22.86" x2="7.62" y2="15.24" width="0.4064" layer="16"/>
+<wire x1="12.7" y1="22.86" x2="15.24" y2="22.86" width="0.6096" layer="16"/>
+<wire x1="15.24" y1="22.86" x2="15.24" y2="27.94" width="0.6096" layer="16"/>
+<wire x1="15.24" y1="27.94" x2="12.7" y2="27.94" width="0.6096" layer="16"/>
+<wire x1="7.62" y1="15.24" x2="5.08" y2="15.24" width="0.6096" layer="16"/>
+<wire x1="12.7" y1="22.86" x2="7.62" y2="22.86" width="0.6096" layer="16"/>
+<wire x1="7.62" y1="22.86" x2="7.62" y2="15.24" width="0.6096" layer="16"/>
 </signal>
 <signal name="N$2">
 <contactref element="R4" pad="1"/>
 <contactref element="IC1" pad="9"/>
-<wire x1="7.62" y1="5.08" x2="12.7" y2="5.08" width="0" layer="19" extent="1-1"/>
+<wire x1="7.62" y1="5.08" x2="12.7" y2="5.08" width="0.6096" layer="16"/>
 </signal>
 <signal name="GND">
@@
 <contactref element="C5" pad="1"/>
 <contactref element="IC1" pad="5"/>
-<wire x1="2.54" y1="30.48" x2="17.78" y2="30.48" width="0.4064" layer="16"/>
-<wire x1="31.75" y1="13.97" x2="31.75" y2="20.32" width="0.4064" layer="16"/>
-<wire x1="12.7" y1="15.24" x2="10.16" y2="15.24" width="0.4064" layer="16"/>
-<wire x1="12.7" y1="15.24" x2="15.24" y2="15.24" width="0.4064" layer="16"/>
-<wire x1="15.24" y1="15.24" x2="15.24" y2="0" width="0.4064" layer="16"/>
-<wire x1="15.24" y1="0" x2="31.75" y2="0" width="0.4064" layer="16"/>
-<wire x1="31.75" y1="0" x2="31.75" y2="13.97" width="0.4064" layer="16"/>
-<wire x1="15.24" y1="15.24" x2="17.78" y2="30.48" width="0" layer="19" extent="16-16"/>
+<wire x1="2.54" y1="30.48" x2="17.78" y2="30.48" width="0.6096" layer="16"/>
+<wire x1="31.75" y1="13.97" x2="31.75" y2="20.32" width="0.6096" layer="16"/>
+<wire x1="12.7" y1="15.24" x2="15.24" y2="15.24" width="0.6096" layer="16"/>
+<wire x1="15.24" y1="15.24" x2="15.24" y2="0" width="0.6096" layer="16"/>
+<wire x1="15.24" y1="0" x2="31.75" y2="0" width="0.6096" layer="16"/>
+<wire x1="31.75" y1="0" x2="31.75" y2="13.97" width="0.6096" layer="16"/>
+<wire x1="15.24" y1="15.24" x2="15.24" y2="20.32" width="0.6096" layer="16"/>
+<wire x1="15.24" y1="20.32" x2="17.78" y2="20.32" width="0.6096" layer="16"/>
+<wire x1="17.78" y1="20.32" x2="17.78" y2="30.48" width="0.6096" layer="16"/>
 </signal>
 <signal name="N$3">
@@
 <contactref element="IC1" pad="1"/>
 <contactref element="R3" pad="2"/>
-<wire x1="12.7" y1="25.4" x2="5.08" y2="25.4" width="0.4064" layer="16"/>
-<wire x1="5.08" y1="25.4" x2="2.54" y2="25.4" width="0.4064" layer="16"/>
-<wire x1="2.54" y1="20.32" x2="2.54" y2="15.24" width="0.4064" layer="16"/>
-<wire x1="2.54" y1="20.32" x2="2.54" y2="25.4" width="0.4064" layer="16"/>
+<wire x1="12.7" y1="25.4" x2="5.08" y2="25.4" width="0.6096" layer="16"/>
+<wire x1="5.08" y1="25.4" x2="2.54" y2="25.4" width="0.6096" layer="16"/>
+<wire x1="2.54" y1="20.32" x2="2.54" y2="15.24" width="0.6096" layer="16"/>
+<wire x1="2.54" y1="20.32" x2="2.54" y2="25.4" width="0.6096" layer="16"/>
 </signal>
 <signal name="VCC">
 <contactref element="R2" pad="1"/>
 <contactref element="IC1" pad="14"/>
-<wire x1="20.32" y1="15.24" x2="17.78" y2="15.24" width="0.4064" layer="16"/>
-<wire x1="17.78" y1="15.24" x2="17.78" y2="2.54" width="0.4064" layer="16"/>
-<wire x1="17.78" y1="2.54" x2="2.54" y2="2.54" width="0.4064" layer="1"/>
-<wire x1="2.54" y1="2.54" x2="2.54" y2="5.08" width="0.4064" layer="16"/>
+<wire x1="20.32" y1="15.24" x2="17.78" y2="15.24" width="0.6096" layer="16"/>
+<wire x1="17.78" y1="15.24" x2="17.78" y2="2.54" width="0.6096" layer="16"/>
+<wire x1="17.78" y1="2.54" x2="2.54" y2="2.54" width="0.6096" layer="1"/>
+<wire x1="2.54" y1="2.54" x2="2.54" y2="5.08" width="0.6096" layer="16"/>
 <via x="17.78" y="2.54" extent="1-16" drill="0.6" shape="square"/>
 <via x="2.54" y="2.54" extent="1-16" drill="0.6" shape="square"/>
@@
 <contactref element="R5" pad="1"/>
 <contactref element="C1" pad="1"/>
-<wire x1="22.86" y1="30.48" x2="22.86" y2="22.86" width="0.4064" layer="16"/>
-<wire x1="22.86" y1="22.86" x2="20.32" y2="22.86" width="0.4064" layer="16"/>
-<wire x1="22.86" y1="27.94" x2="22.86" y2="30.48" width="0.4064" layer="16"/>
+<wire x1="22.86" y1="30.48" x2="22.86" y2="22.86" width="0.6096" layer="16"/>
+<wire x1="22.86" y1="22.86" x2="20.32" y2="22.86" width="0.6096" layer="16"/>
+<wire x1="22.86" y1="27.94" x2="22.86" y2="30.48" width="0.6096" layer="16"/>
 </signal>
 <signal name="OSC1">
@@
 <contactref element="Q1" pad="2"/>
 <contactref element="IC1" pad="16"/>
-<wire x1="29.21" y1="20.32" x2="20.32" y2="20.32" width="0.4064" layer="16"/>
+<wire x1="29.21" y1="20.32" x2="20.32" y2="20.32" width="0.6096" layer="16"/>
 <wire x1="29.21" y1="20.32" x2="25.4" y2="20.32" width="0" layer="19" extent="1-1"/>
 </signal>
@@
 <contactref element="Q1" pad="1"/>
 <contactref element="IC1" pad="15"/>
-<wire x1="20.32" y1="17.78" x2="25.4" y2="17.78" width="0.4064" layer="16"/>
-<wire x1="25.4" y1="17.78" x2="25.4" y2="15.24" width="0.4064" layer="16"/>
-<wire x1="25.4" y1="15.24" x2="29.21" y2="15.24" width="0.4064" layer="16"/>
-<wire x1="29.21" y1="15.24" x2="29.21" y2="13.97" width="0.4064" layer="16"/>
+<wire x1="20.32" y1="17.78" x2="25.4" y2="17.78" width="0.6096" layer="16"/>
+<wire x1="25.4" y1="17.78" x2="25.4" y2="15.24" width="0.6096" layer="16"/>
+<wire x1="25.4" y1="15.24" x2="29.21" y2="15.24" width="0.6096" layer="16"/>
+<wire x1="29.21" y1="15.24" x2="29.21" y2="13.97" width="0.6096" layer="16"/>
 </signal>
 </signals>

Commit message: ...
Other:
- board outline removed
Changed lines of the file:
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@@
 <board>
 <plain>
-<wire x1="0" y1="-2.54" x2="35.54" y2="-2.54" width="0" layer="20"/>
-<wire x1="35.54" y1="-2.54" x2="35.56" y2="31.75" width="0" layer="20"/>
-<wire x1="35.56" y1="31.75" x2="35.56" y2="33.02" width="0" layer="20"/>
-<wire x1="35.56" y1="33.02" x2="0" y2="33.02" width="0" layer="20"/>
-<wire x1="0" y1="33.02" x2="0" y2="-2.54" width="0" layer="20"/>
+<wire x1="0" y1="-2.54" x2="35.54" y2="-2.54" width="0" layer="47"/>
+<wire x1="35.54" y1="-2.54" x2="35.56" y2="31.75" width="0" layer="47"/>
+<wire x1="35.56" y1="31.75" x2="35.56" y2="33.02" width="0" layer="47"/>
+<wire x1="35.56" y1="33.02" x2="0" y2="33.02" width="0" layer="47"/>
+<wire x1="0" y1="33.02" x2="0" y2="-2.54" width="0" layer="47"/>
 </plain>
 <attributes>
@@
 <contactref element="R4" pad="2"/>
 <contactref element="R5" pad="2"/>
-<wire x1="12.7" y1="22.86" x2="15.24" y2="22.86" width="0.6096" layer="16"/>
-<wire x1="15.24" y1="22.86" x2="15.24" y2="27.94" width="0.6096" layer="16"/>
-<wire x1="15.24" y1="27.94" x2="12.7" y2="27.94" width="0.6096" layer="16"/>
-<wire x1="7.62" y1="15.24" x2="5.08" y2="15.24" width="0.6096" layer="16"/>
-<wire x1="12.7" y1="22.86" x2="7.62" y2="22.86" width="0.6096" layer="16"/>
-<wire x1="7.62" y1="22.86" x2="7.62" y2="15.24" width="0.6096" layer="16"/>
+<wire x1="12.7" y1="22.86" x2="15.24" y2="22.86" width="1.27" layer="16"/>
+<wire x1="15.24" y1="22.86" x2="15.24" y2="27.94" width="1.27" layer="16"/>
+<wire x1="15.24" y1="27.94" x2="12.7" y2="27.94" width="1.27" layer="16"/>
+<wire x1="7.62" y1="15.24" x2="5.08" y2="15.24" width="1.27" layer="16"/>
+<wire x1="12.7" y1="22.86" x2="7.62" y2="22.86" width="1.27" layer="16"/>
+<wire x1="7.62" y1="22.86" x2="7.62" y2="15.24" width="1.27" layer="16"/>
 </signal>
 <signal name="N$2">
 <contactref element="R4" pad="1"/>
 <contactref element="IC1" pad="9"/>
-<wire x1="7.62" y1="5.08" x2="12.7" y2="5.08" width="0.6096" layer="16"/>
+<wire x1="7.62" y1="5.08" x2="12.7" y2="5.08" width="1.27" layer="16"/>
 </signal>
 <signal name="GND">
@@
 <contactref element="C5" pad="1"/>
 <contactref element="IC1" pad="5"/>
-<wire x1="2.54" y1="30.48" x2="17.78" y2="30.48" width="0.6096" layer="16"/>
-<wire x1="31.75" y1="13.97" x2="31.75" y2="20.32" width="0.6096" layer="16"/>
-<wire x1="12.7" y1="15.24" x2="15.24" y2="15.24" width="0.6096" layer="16"/>
-<wire x1="15.24" y1="15.24" x2="15.24" y2="0" width="0.6096" layer="16"/>
-<wire x1="15.24" y1="0" x2="31.75" y2="0" width="0.6096" layer="16"/>
-<wire x1="31.75" y1="0" x2="31.75" y2="13.97" width="0.6096" layer="16"/>
-<wire x1="15.24" y1="15.24" x2="15.24" y2="20.32" width="0.6096" layer="16"/>
-<wire x1="15.24" y1="20.32" x2="17.78" y2="20.32" width="0.6096" layer="16"/>
-<wire x1="17.78" y1="20.32" x2="17.78" y2="30.48" width="0.6096" layer="16"/>
+<wire x1="2.54" y1="30.48" x2="17.78" y2="30.48" width="1.27" layer="16"/>
+<wire x1="31.75" y1="13.97" x2="31.75" y2="20.32" width="1.27" layer="16"/>
+<wire x1="12.7" y1="15.24" x2="15.24" y2="15.24" width="1.27" layer="16"/>
+<wire x1="15.24" y1="15.24" x2="15.24" y2="0" width="1.27" layer="16"/>
+<wire x1="15.24" y1="0" x2="31.75" y2="0" width="1.27" layer="16"/>
+<wire x1="31.75" y1="0" x2="31.75" y2="13.97" width="1.27" layer="16"/>
+<wire x1="15.24" y1="15.24" x2="15.24" y2="20.32" width="1.27" layer="16"/>
+<wire x1="15.24" y1="20.32" x2="17.78" y2="20.32" width="1.27" layer="16"/>
+<wire x1="17.78" y1="20.32" x2="17.78" y2="30.48" width="1.27" layer="16"/>
 </signal>
 <signal name="N$3">
@@
 <contactref element="IC1" pad="1"/>
 <contactref element="R3" pad="2"/>
-<wire x1="12.7" y1="25.4" x2="5.08" y2="25.4" width="0.6096" layer="16"/>
-<wire x1="5.08" y1="25.4" x2="2.54" y2="25.4" width="0.6096" layer="16"/>
-<wire x1="2.54" y1="20.32" x2="2.54" y2="15.24" width="0.6096" layer="16"/>
-<wire x1="2.54" y1="20.32" x2="2.54" y2="25.4" width="0.6096" layer="16"/>
+<wire x1="12.7" y1="25.4" x2="5.08" y2="25.4" width="1.27" layer="16"/>
+<wire x1="5.08" y1="25.4" x2="2.54" y2="25.4" width="1.27" layer="16"/>
+<wire x1="2.54" y1="20.32" x2="2.54" y2="15.24" width="1.27" layer="16"/>
+<wire x1="2.54" y1="20.32" x2="2.54" y2="25.4" width="1.27" layer="16"/>
 </signal>
 <signal name="VCC">
 <contactref element="R2" pad="1"/>
 <contactref element="IC1" pad="14"/>
-<wire x1="20.32" y1="15.24" x2="17.78" y2="15.24" width="0.6096" layer="16"/>
-<wire x1="17.78" y1="15.24" x2="17.78" y2="2.54" width="0.6096" layer="16"/>
-<wire x1="17.78" y1="2.54" x2="2.54" y2="2.54" width="0.6096" layer="1"/>
-<wire x1="2.54" y1="2.54" x2="2.54" y2="5.08" width="0.6096" layer="16"/>
+<wire x1="20.32" y1="15.24" x2="17.78" y2="15.24" width="1.27" layer="16"/>
+<wire x1="17.78" y1="15.24" x2="17.78" y2="2.54" width="1.27" layer="16"/>
+<wire x1="17.78" y1="2.54" x2="2.54" y2="2.54" width="1.27" layer="1"/>
+<wire x1="2.54" y1="2.54" x2="2.54" y2="5.08" width="1.27" layer="16"/>
 <via x="17.78" y="2.54" extent="1-16" drill="0.6" shape="square"/>
 <via x="2.54" y="2.54" extent="1-16" drill="0.6" shape="square"/>
@@
 <contactref element="R5" pad="1"/>
 <contactref element="C1" pad="1"/>
-<wire x1="22.86" y1="30.48" x2="22.86" y2="22.86" width="0.6096" layer="16"/>
-<wire x1="22.86" y1="22.86" x2="20.32" y2="22.86" width="0.6096" layer="16"/>
-<wire x1="22.86" y1="27.94" x2="22.86" y2="30.48" width="0.6096" layer="16"/>
+<wire x1="22.86" y1="30.48" x2="22.86" y2="22.86" width="1.27" layer="16"/>
+<wire x1="22.86" y1="22.86" x2="20.32" y2="22.86" width="1.27" layer="16"/>
+<wire x1="22.86" y1="27.94" x2="22.86" y2="30.48" width="1.27" layer="16"/>
 </signal>
 <signal name="OSC1">
@@
 <contactref element="Q1" pad="2"/>
 <contactref element="IC1" pad="16"/>
-<wire x1="29.21" y1="20.32" x2="20.32" y2="20.32" width="0.6096" layer="16"/>
+<wire x1="29.21" y1="20.32" x2="20.32" y2="20.32" width="1.27" layer="16"/>
 <wire x1="29.21" y1="20.32" x2="25.4" y2="20.32" width="0" layer="19" extent="1-1"/>
 </signal>
@@
 <contactref element="Q1" pad="1"/>
 <contactref element="IC1" pad="15"/>
-<wire x1="20.32" y1="17.78" x2="25.4" y2="17.78" width="0.6096" layer="16"/>
-<wire x1="25.4" y1="17.78" x2="25.4" y2="15.24" width="0.6096" layer="16"/>
-<wire x1="25.4" y1="15.24" x2="29.21" y2="15.24" width="0.6096" layer="16"/>
-<wire x1="29.21" y1="15.24" x2="29.21" y2="13.97" width="0.6096" layer="16"/>
+<wire x1="20.32" y1="17.78" x2="25.4" y2="17.78" width="1.27" layer="16"/>
+<wire x1="25.4" y1="17.78" x2="25.4" y2="15.24" width="1.27" layer="16"/>
+<wire x1="25.4" y1="15.24" x2="29.21" y2="15.24" width="1.27" layer="16"/>
+<wire x1="29.21" y1="15.24" x2="29.21" y2="13.97" width="1.27" layer="16"/>
 </signal>
 </signals>

Commit message: ...
Parts:
- R1, R2, R3, R4: value 1.5k -> 1.5kΩ
- R5: value 10k -> 10kΩ
Changed lines of the file:
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@@
 <element name="C1" library="c" package="C050-020X036" value="270pF" x="20.32" y="30.48" rot="R90"/>
 <element name="IC1" library="mcu" package="DIL18-3/V" value="PIC16F628A-COMP" x="16.51" y="15.24"/>
-<element name="R1" library="r" package="0204/10" value="1.5k" x="2.54" y="25.4" rot="R270"/>
-<element name="R2" library="r" package="0204/10" value="1.5k" x="2.54" y="10.16" rot="R90"/>
-<element name="R3" library="r" package="0204/10" value="1.5k" x="5.08" y="20.32" rot="R90"/>
-<element name="R4" library="r" package="0204/10" value="1.5k" x="7.62" y="10.16" rot="R90"/>
-<element name="R5" library="r" package="0204/10" value="10k" x="17.78" y="27.94" rot="R180"/>
+<element name="R1" library="r" package="0204/10" value="1.5kΩ" x="2.54" y="25.4" rot="R270"/>
+<element name="R2" library="r" package="0204/10" value="1.5kΩ" x="2.54" y="10.16" rot="R90"/>
+<element name="R3" library="r" package="0204/10" value="1.5kΩ" x="5.08" y="20.32" rot="R90"/>
+<element name="R4" library="r" package="0204/10" value="1.5kΩ" x="7.62" y="10.16" rot="R90"/>
+<element name="R5" library="r" package="0204/10" value="10kΩ" x="17.78" y="27.94" rot="R180"/>
 <element name="C5" library="c" package="C025-020X036" value="33pF" x="31.75" y="13.97" rot="R180"/>
 <element name="C6" library="c" package="C025-020X036" value="33pF" x="31.75" y="20.32" rot="R180"/>
