File: eagle/LCmeter0-LCD-mounted-PIC-COMP.brd (EAGLE design)
At the start: 32 parts, among them IC1 PIC16F876A, J1 HD44780LM016L, J2 PIC-UART, J3 PIC-ICSP, J4 J4, J5 CONN-2P2P/V, J7 CONN-2P2P/V, K2 DS2Y, Q1 20MHz, SW1 PB-1P-1T, T1 BC547

Commit message: ...
Parts:
- R1, R2, R3: value 100k -> 100kΩ
- R10, R5: value 4.7k -> 4.7kΩ
- R11: value 1k -> 1kΩ
- R4: value 47k -> 47kΩ
- R6, R7: value 10k -> 10kΩ
Changed lines of the file:
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@@
 </element>
 <element name="Q1" library="q" package="HC49" value="20MHz" x="55.88" y="20.32" rot="R90"/>
-<element name="R1" library="r" package="0202/7" value="100k" x="35.56" y="24.13" rot="R90"/>
-<element name="R10" library="r" package="0202/7" value="4.7k" x="33.02" y="24.13" rot="R90"/>
-<element name="R11" library="r" package="0202/10-V" value="1k" x="71.12" y="22.86"/>
-<element name="R2" library="r" package="0202/7" value="100k" x="48.26" y="24.13" rot="R270"/>
-<element name="R3" library="r" package="0202/7" value="100k" x="30.48" y="24.13" rot="R90"/>
-<element name="R4" library="r" package="0202/7" value="47k" x="40.64" y="24.13" rot="R90"/>
-<element name="R5" library="r" package="0202/7" value="4.7k" x="45.72" y="24.13" rot="R270"/>
-<element name="R6" library="r" package="0202/10" value="10k" x="78.74" y="48.26"/>
-<element name="R7" library="r" package="0202/7" value="10k" x="72.39" y="38.1" rot="R180"/>
+<element name="R1" library="r" package="0202/7" value="100kΩ" x="35.56" y="24.13" rot="R90"/>
+<element name="R10" library="r" package="0202/7" value="4.7kΩ" x="33.02" y="24.13" rot="R90"/>
+<element name="R11" library="r" package="0202/10-V" value="1kΩ" x="71.12" y="22.86"/>
+<element name="R2" library="r" package="0202/7" value="100kΩ" x="48.26" y="24.13" rot="R270"/>
+<element name="R3" library="r" package="0202/7" value="100kΩ" x="30.48" y="24.13" rot="R90"/>
+<element name="R4" library="r" package="0202/7" value="47kΩ" x="40.64" y="24.13" rot="R90"/>
+<element name="R5" library="r" package="0202/7" value="4.7kΩ" x="45.72" y="24.13" rot="R270"/>
+<element name="R6" library="r" package="0202/10" value="10kΩ" x="78.74" y="48.26"/>
+<element name="R7" library="r" package="0202/7" value="10kΩ" x="72.39" y="38.1" rot="R180"/>
 <element name="S1" library="sw" package="SLSW-2P2T" value="SL-SW-2P-2T" x="13.97" y="17.78"/>
 <element name="SW1" library="sw" package="PB-1P1T" value="PB-1P-1T" x="7.62" y="45.72" rot="R90"/>

Commit message: ...
Other:
- board outline added: 96.5 x 55.9 mm
Changed lines of the file:
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@@
 <board>
 <plain>
-<wire x1="0" y1="0" x2="0" y2="55.88" width="0.0254" layer="47"/>
-<wire x1="0" y1="55.88" x2="96.52" y2="55.88" width="0.0254" layer="47"/>
-<wire x1="96.52" y1="55.88" x2="96.52" y2="0" width="0.0254" layer="47"/>
-<wire x1="96.52" y1="0" x2="0" y2="0" width="0.0254" layer="47"/>
+<wire x1="0" y1="0" x2="0" y2="55.88" width="0.0254" layer="20"/>
+<wire x1="0" y1="55.88" x2="96.52" y2="55.88" width="0.0254" layer="20"/>
+<wire x1="96.52" y1="55.88" x2="96.52" y2="0" width="0.0254" layer="20"/>
+<wire x1="96.52" y1="0" x2="0" y2="0" width="0.0254" layer="20"/>
 </plain>
 <attributes>
