File: eagle/PIC18F2550-USB-HID-LC-Meter.brd (EAGLE design)
At the start: 71.1 x 63.5 mm, 26 parts, among them J1 USB-PRINT, Q1 2N7000, X1 20MHz

Commit message: ...
Other:
- board outline removed

Commit message: ...
Parts:
- L1: device r:L-04/7-M -> r:L-04/10-M
Changed lines of the file:
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@@
 <element name="IN-" library="pad" package="SPAD" value="SPAD" x="33.02" y="17.78"/>
 <element name="J1" library="usb" package="USB-B-PRINT" value="USB-PRINT" x="53.34" y="5.08" rot="R90"/>
-<element name="L1" library="r" package="L-04/7-M" value="100uH" x="19.05" y="26.67" rot="R270"/>
+<element name="L1" library="r" package="L-04/10-M" value="100uH" x="19.05" y="26.67" rot="R270"/>
 <element name="Q1" library="t" package="TO92" value="2N7000" x="33.02" y="30.48" rot="R180"/>
 <element name="R#" library="r" package="0202/7" value="" x="36.83" y="33.02" rot="R180"/>

Commit message: ...
Parts:
- L1: value 100uH -> 100μH
- R1, R2, R3: value 100k -> 100kΩ
- R4: value 47k -> 47kΩ
- R5, R6: value 100 -> 100Ω
- R7: value 4.7k -> 4.7kΩ
Changed lines of the file:
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@@
 <element name="IN-" library="pad" package="SPAD" value="SPAD" x="33.02" y="17.78"/>
 <element name="J1" library="usb" package="USB-B-PRINT" value="USB-PRINT" x="53.34" y="5.08" rot="R90"/>
-<element name="L1" library="r" package="L-04/10-M" value="100uH" x="19.05" y="26.67" rot="R270"/>
+<element name="L1" library="r" package="L-04/10-M" value="100μH" x="19.05" y="26.67" rot="R270"/>
 <element name="Q1" library="t" package="TO92" value="2N7000" x="33.02" y="30.48" rot="R180"/>
 <element name="R#" library="r" package="0202/7" value="" x="36.83" y="33.02" rot="R180"/>
-<element name="R1" library="r" package="0202/7" value="100k" x="24.13" y="45.72"/>
-<element name="R2" library="r" package="0202/7" value="100k" x="45.72" y="36.83" rot="R90"/>
-<element name="R3" library="r" package="0202/7" value="100k" x="24.13" y="38.1" rot="R180"/>
-<element name="R4" library="r" package="0202/7" value="47k" x="29.21" y="48.26"/>
-<element name="R5" library="r" package="0202/7" value="100" x="60.96" y="39.37" rot="R270"/>
-<element name="R6" library="r" package="0202/7" value="100" x="63.5" y="36.83" rot="R270"/>
-<element name="R7" library="r" package="0202/7" value="4.7k" x="44.45" y="50.8" rot="R180"/>
+<element name="R1" library="r" package="0202/7" value="100kΩ" x="24.13" y="45.72"/>
+<element name="R2" library="r" package="0202/7" value="100kΩ" x="45.72" y="36.83" rot="R90"/>
+<element name="R3" library="r" package="0202/7" value="100kΩ" x="24.13" y="38.1" rot="R180"/>
+<element name="R4" library="r" package="0202/7" value="47kΩ" x="29.21" y="48.26"/>
+<element name="R5" library="r" package="0202/7" value="100Ω" x="60.96" y="39.37" rot="R270"/>
+<element name="R6" library="r" package="0202/7" value="100Ω" x="63.5" y="36.83" rot="R270"/>
+<element name="R7" library="r" package="0202/7" value="4.7kΩ" x="44.45" y="50.8" rot="R180"/>
 <element name="U$1" library="sw" package="SLSW-2P2T" value="SW-2P-2T" x="26.67" y="17.78" rot="R90"/>
 <element name="U$2" library="mcu" package="DIL28-3/V" value="PIC18F2550-I/SP-2-V" x="54.61" y="34.29"/>

Commit message: ...
Other:
- board outline added: 71.1 x 63.5 mm
Changed lines of the file:
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@@
 <board>
 <plain>
-<wire x1="0" y1="0" x2="71.12" y2="0" width="0" layer="47"/>
-<wire x1="71.12" y1="0" x2="71.12" y2="63.5" width="0" layer="47"/>
-<wire x1="71.12" y1="63.5" x2="0" y2="63.5" width="0" layer="47"/>
-<wire x1="0" y1="63.5" x2="0" y2="0" width="0" layer="47"/>
+<wire x1="0" y1="0" x2="71.12" y2="0" width="0" layer="20"/>
+<wire x1="71.12" y1="0" x2="71.12" y2="63.5" width="0" layer="20"/>
+<wire x1="71.12" y1="63.5" x2="0" y2="63.5" width="0" layer="20"/>
+<wire x1="0" y1="63.5" x2="0" y2="0" width="0" layer="20"/>
 </plain>
 <attributes>
