File: eagle/LCmeter0-LCD-8pinlcd-PICCOMP.brd (EAGLE design)
At the start: 63.5 x 53.3 mm, 34 parts, among them IC1 PIC16F876A-X/SP-COMP-B-A/V, J1 HD44780, J2 PIC-UART, J3 PIC-ICSP, K2 DS2Y, Q1 20MHz, T1 BC547, X1 FREQ, X2 L/C

Commit message: ...
Routing:
- net VCC: track 141.4 -> 138.4 mm
- net GND: track 185.7 -> 184.2 mm
Changed lines of the file:
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@@
 <wire x1="50.8" y1="20.32" x2="53.34" y2="20.32" width="0.6096" layer="16"/>
 <wire x1="53.34" y1="20.32" x2="58.42" y2="20.32" width="0.6096" layer="16"/>
-<wire x1="60.96" y1="20.32" x2="60.96" y2="2.54" width="0.6096" layer="16"/>
-<wire x1="58.42" y1="2.54" x2="60.96" y2="2.54" width="0.6096" layer="16"/>
+<wire x1="60.96" y1="20.32" x2="60.96" y2="5.08" width="0.6096" layer="16"/>
+<wire x1="60.96" y1="5.08" x2="58.42" y2="2.54" width="0.6096" layer="16" curve="-90"/>
 <wire x1="55.88" y1="10.16" x2="55.88" y2="2.54" width="0.6096" layer="16"/>
 <wire x1="55.88" y1="2.54" x2="58.42" y2="2.54" width="0.6096" layer="16"/>
@@
 <contactref element="Q1" pad="1"/>
 <contactref element="IC1" pad="9"/>
-<wire x1="43.18" y1="22.86" x2="38.1" y2="22.86" width="0.6096" layer="16"/>
-<wire x1="33.02" y1="22.86" x2="38.1" y2="22.86" width="0.6096" layer="16"/>
-<wire x1="38.1" y1="22.86" x2="38.1" y2="24.13" width="0.6096" layer="16"/>
+<wire x1="43.18" y1="22.86" x2="41.91" y2="22.86" width="0.6096" layer="16"/>
+<wire x1="41.91" y1="22.86" x2="40.64" y2="23.495" width="0.6096" layer="16" curve="-75"/>
+<wire x1="40.64" y1="23.495" x2="39.37" y2="24.13" width="0.6096" layer="16" curve="75"/>
+<wire x1="39.37" y1="24.13" x2="38.1" y2="24.13" width="0.6096" layer="16"/>
+<wire x1="33.02" y1="22.86" x2="34.29" y2="24.13" width="0.6096" layer="16" curve="-90"/>
+<wire x1="34.29" y1="24.13" x2="38.1" y2="24.13" width="0.6096" layer="16"/>
 </signal>
 <signal name="OSC2">
@@
 <contactref element="Q1" pad="2"/>
 <contactref element="IC1" pad="10"/>
-<wire x1="43.18" y1="20.32" x2="38.1" y2="20.32" width="0.6096" layer="16"/>
-<wire x1="33.02" y1="20.32" x2="38.1" y2="20.32" width="0.6096" layer="16"/>
-<wire x1="38.1" y1="20.32" x2="38.1" y2="19.05" width="0.6096" layer="16"/>
+<wire x1="43.18" y1="20.32" x2="41.91" y2="20.32" width="0.6096" layer="16"/>
+<wire x1="41.91" y1="20.32" x2="40.64" y2="19.685" width="0.6096" layer="16" curve="75"/>
+<wire x1="40.64" y1="19.685" x2="39.37" y2="19.05" width="0.6096" layer="16" curve="-75"/>
+<wire x1="39.37" y1="19.05" x2="38.1" y2="19.05" width="0.6096" layer="16"/>
+<wire x1="33.02" y1="20.32" x2="34.29" y2="19.05" width="0.6096" layer="16" curve="90"/>
+<wire x1="34.29" y1="19.05" x2="38.1" y2="19.05" width="0.6096" layer="16"/>
 </signal>
 <signal name="VCC">
@@
 <wire x1="55.88" y1="22.86" x2="58.42" y2="22.86" width="0.6096" layer="16"/>
 <wire x1="58.42" y1="5.08" x2="58.42" y2="10.16" width="0.6096" layer="16"/>
-<wire x1="58.42" y1="10.16" x2="58.42" y2="12.7" width="0.6096" layer="16"/>
-<wire x1="58.42" y1="12.7" x2="55.88" y2="12.7" width="0.6096" layer="16"/>
+<wire x1="58.42" y1="10.16" x2="55.88" y2="12.7" width="0.6096" layer="16" curve="90"/>
 <via x="55.88" y="12.7" extent="1-16" drill="0.762" diameter="1.4224"/>
 <wire x1="55.88" y1="12.7" x2="55.88" y2="22.86" width="0.6096" layer="1"/>
@@
 <wire x1="30.48" y1="30.48" x2="25.4" y2="30.48" width="0.6096" layer="16"/>
 <via x="25.4" y="30.48" extent="1-16" drill="0.762" diameter="1.4224"/>
-<wire x1="25.4" y1="30.48" x2="15.24" y2="30.48" width="0.6096" layer="1"/>
-<via x="15.24" y="30.48" extent="1-16" drill="0.762" diameter="1.4224"/>
-<wire x1="15.24" y1="30.48" x2="15.24" y2="17.78" width="0.6096" layer="16"/>
+<wire x1="25.4" y1="30.48" x2="17.78" y2="30.48" width="0.6096" layer="1"/>
+<via x="17.78" y="30.48" extent="1-16" drill="0.762" diameter="1.4224"/>
 <via x="15.24" y="17.78" extent="1-16" drill="0.762" diameter="1.4224"/>
 <wire x1="15.24" y1="17.78" x2="15.24" y2="7.62" width="0.6096" layer="1"/>
@@
 <wire x1="15.24" y1="7.62" x2="12.7" y2="7.62" width="0.6096" layer="16"/>
 <wire x1="35.56" y1="45.72" x2="33.02" y2="43.18" width="0.6096" layer="16" curve="90"/>
+<wire x1="17.78" y1="30.48" x2="15.24" y2="27.94" width="0.6096" layer="16" curve="90"/>
+<wire x1="15.24" y1="27.94" x2="15.24" y2="17.78" width="0.6096" layer="16"/>
 </signal>
 <signal name="D4">

Commit message: ...
Parts:
- R11: device r:0202/7 -> r:0204/10
- moved R11 1.27 mm to (35.6, 12.7)
Routing:
- net GND: track 184.2 -> 177.6 mm
- net /LC: track 77.3 -> 74.3 mm
- net A0: track 24.5 -> 27.3 mm
- net /MCLR: track 30.5 -> 29.0 mm
- net FREQ: track 39.0 -> 39.6 mm
- added copper zone on layer 16, net GND
Other:
- board outline removed
Changed lines of the file:
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@@
 <board>
 <plain>
-<wire x1="0" y1="0" x2="63.5" y2="0" width="0" layer="20"/>
-<wire x1="63.5" y1="0" x2="63.5" y2="53.34" width="0" layer="20"/>
-<wire x1="63.5" y1="53.34" x2="0" y2="53.34" width="0" layer="20"/>
-<wire x1="0" y1="53.34" x2="0" y2="0" width="0" layer="20"/>
+<wire x1="0" y1="0" x2="63.5" y2="0" width="0" layer="48"/>
+<wire x1="63.5" y1="0" x2="63.5" y2="53.34" width="0" layer="48"/>
+<wire x1="63.5" y1="53.34" x2="0" y2="53.34" width="0" layer="48"/>
+<wire x1="0" y1="53.34" x2="0" y2="0" width="0" layer="48"/>
 </plain>
 <attributes>
@@
 <element name="R1" library="r" package="0204/10" value="100kΩ" x="35.56" y="40.64" rot="R180"/>
 <element name="R10" library="r" package="0204/10" value="4.7kΩ" x="35.56" y="43.18"/>
-<element name="R11" library="r" package="0202/7" value="1kΩ" x="36.83" y="12.7"/>
+<element name="R11" library="r" package="0204/10" value="1kΩ" x="35.56" y="12.7"/>
 <element name="R2" library="r" package="0204/10" value="100kΩ" x="35.56" y="27.94" rot="R180"/>
 <element name="R3" library="r" package="0204/10" value="100kΩ" x="35.56" y="45.72"/>
@@
 <contactref element="C3" pad="+"/>
 <contactref element="IC1" pad="5"/>
-<wire x1="43.18" y1="33.02" x2="38.1" y2="33.02" width="0.6096" layer="16"/>
-<wire x1="38.1" y1="33.02" x2="35.56" y2="30.48" width="0.6096" layer="16" curve="90"/>
-<wire x1="35.56" y1="30.48" x2="33.02" y2="27.94" width="0.6096" layer="16" curve="-90"/>
-<wire x1="33.02" y1="27.94" x2="30.48" y2="27.94" width="0.6096" layer="16"/>
+<wire x1="43.18" y1="33.02" x2="40.005" y2="33.02" width="0.6096" layer="16"/>
+<wire x1="40.005" y1="33.02" x2="36.83" y2="30.48" width="0.6096" layer="16" curve="90"/>
+<wire x1="36.83" y1="30.48" x2="34.29" y2="27.94" width="0.6096" layer="16" curve="-90"/>
+<wire x1="34.29" y1="27.94" x2="30.48" y2="27.94" width="0.6096" layer="16"/>
 <wire x1="30.48" y1="45.72" x2="27.94" y2="43.18" width="0.6096" layer="16" curve="90"/>
 <wire x1="27.94" y1="43.18" x2="27.94" y2="40.64" width="0.6096" layer="16"/>
@@
 <contactref element="IC1" pad="2"/>
 <contactref element="IC1" pad="7"/>
-<wire x1="40.64" y1="40.64" x2="38.1" y2="38.1" width="0.6096" layer="16" curve="90"/>
-<wire x1="38.1" y1="38.1" x2="40.64" y2="35.56" width="0.6096" layer="16" curve="90"/>
+<wire x1="40.64" y1="40.64" x2="39.37" y2="40.64" width="0.6096" layer="16"/>
+<wire x1="39.37" y1="40.64" x2="36.83" y2="38.1" width="0.6096" layer="16" curve="90"/>
+<wire x1="36.83" y1="38.1" x2="38.735" y2="35.56" width="0.6096" layer="16" curve="90"/>
+<wire x1="38.735" y1="35.56" x2="40.64" y2="35.56" width="0.6096" layer="16"/>
 <wire x1="43.18" y1="40.64" x2="45.72" y2="38.1" width="0.6096" layer="16" curve="-90"/>
 <wire x1="45.72" y1="38.1" x2="45.72" y2="30.48" width="0.6096" layer="16"/>
@@
 <wire x1="48.26" y1="20.32" x2="45.72" y2="22.86" width="0.6096" layer="16" curve="-90"/>
 <wire x1="45.72" y1="22.86" x2="43.18" y2="25.4" width="0.6096" layer="16" curve="90"/>
-<wire x1="40.64" y1="25.4" x2="43.18" y2="25.4" width="0.6096" layer="16"/>
-<wire x1="58.42" y1="25.4" x2="60.96" y2="22.86" width="0.6096" layer="16" curve="-90"/>
-<wire x1="60.96" y1="22.86" x2="60.96" y2="20.32" width="0.6096" layer="16"/>
+<wire x1="40.64" y1="26.035" x2="43.18" y2="25.4" width="0.6096" layer="16"/>
 <wire x1="60.96" y1="20.32" x2="58.42" y2="20.32" width="0.6096" layer="16"/>
 <wire x1="50.8" y1="20.32" x2="53.34" y2="20.32" width="0.6096" layer="16"/>
@@
 <wire x1="31.75" y1="17.78" x2="30.48" y2="19.05" width="0.6096" layer="16" curve="-90"/>
 <wire x1="30.48" y1="19.05" x2="30.48" y2="20.32" width="0.6096" layer="16"/>
-<wire x1="40.64" y1="25.4" x2="30.48" y2="25.4" width="0.6096" layer="16"/>
-<wire x1="30.48" y1="25.4" x2="30.48" y2="22.86" width="0.6096" layer="16"/>
+<wire x1="40.64" y1="26.035" x2="33.655" y2="26.035" width="0.6096" layer="16"/>
+<wire x1="33.655" y1="26.035" x2="30.48" y2="23.495" width="0.6096" layer="16" curve="77.319617"/>
+<wire x1="30.48" y1="23.495" x2="30.48" y2="22.86" width="0.6096" layer="16" curve="25.360688"/>
 <wire x1="30.48" y1="22.86" x2="30.48" y2="20.32" width="0.6096" layer="16"/>
 <wire x1="27.94" y1="2.54" x2="55.88" y2="2.54" width="0.6096" layer="16"/>
 <wire x1="27.94" y1="2.54" x2="12.7" y2="2.54" width="0.6096" layer="16"/>
 <wire x1="12.7" y1="2.54" x2="7.62" y2="7.62" width="0.6096" layer="16" curve="-90"/>
-<wire x1="40.64" y1="25.4" x2="40.64" y2="27.94" width="0.6096" layer="16"/>
+<wire x1="40.64" y1="26.035" x2="40.64" y2="27.94" width="0.6096" layer="16"/>
 <wire x1="40.64" y1="50.8" x2="25.4" y2="50.8" width="0.6096" layer="16"/>
 <wire x1="25.4" y1="50.8" x2="22.86" y2="48.26" width="0.6096" layer="16" curve="90"/>
@@
 <via x="20.32" y="35.56" extent="1-16" drill="0.762" diameter="1.4224"/>
 <wire x1="17.78" y1="35.56" x2="20.32" y2="35.56" width="0.6096" layer="16"/>
+<wire x1="22.86" y1="27.94" x2="22.86" y2="35.56" width="0.6096" layer="16"/>
+<wire x1="20.32" y1="35.56" x2="22.86" y2="35.56" width="0.6096" layer="16"/>
+<polygon width="0" layer="16">
+<vertex x="0" y="53.34"/>
+<vertex x="63.5" y="53.34"/>
+<vertex x="63.5" y="0"/>
+<vertex x="0" y="0"/>
+</polygon>
+<wire x1="25.4" y1="25.4" x2="27.94" y2="25.4" width="0.6096" layer="16"/>
+<wire x1="27.94" y1="25.4" x2="30.48" y2="22.86" width="0.6096" layer="16" curve="-90"/>
 <wire x1="25.4" y1="25.4" x2="22.86" y2="27.94" width="0.6096" layer="16" curve="-90"/>
-<wire x1="22.86" y1="27.94" x2="22.86" y2="35.56" width="0.6096" layer="16"/>
-<wire x1="25.4" y1="25.4" x2="30.48" y2="25.4" width="0.6096" layer="16"/>
-<wire x1="20.32" y1="35.56" x2="22.86" y2="35.56" width="0.6096" layer="16"/>
 </signal>
 <signal name="N$7">
@@
 <contactref element="S1" pad="6"/>
 <wire x1="50.8" y1="10.16" x2="48.26" y2="7.62" width="0.6096" layer="16" curve="-90"/>
-<wire x1="48.26" y1="7.62" x2="30.48" y2="7.62" width="0.6096" layer="16"/>
-<wire x1="30.48" y1="7.62" x2="30.48" y2="12.7" width="0.6096" layer="1"/>
-<wire x1="30.48" y1="12.7" x2="12.7" y2="12.7" width="0.6096" layer="16"/>
+<wire x1="48.26" y1="7.62" x2="33.02" y2="7.62" width="0.6096" layer="16"/>
+<wire x1="33.02" y1="7.62" x2="27.94" y2="12.7" width="0.6096" layer="1" curve="-90"/>
+<wire x1="27.94" y1="12.7" x2="12.7" y2="12.7" width="0.6096" layer="16"/>
 <wire x1="12.7" y1="12.7" x2="12.7" y2="17.78" width="0.6096" layer="16"/>
-<via x="30.48" y="7.62" extent="1-16" drill="0.762" diameter="1.4224"/>
-<via x="30.48" y="12.7" extent="1-16" drill="0.762" diameter="1.4224"/>
+<via x="33.02" y="7.62" extent="1-16" drill="0.762" diameter="1.4224"/>
+<via x="27.94" y="12.7" extent="1-16" drill="0.762" diameter="1.4224"/>
 <wire x1="12.7" y1="17.78" x2="12.7" y2="33.02" width="0.6096" layer="16"/>
 <via x="12.7" y="33.02" extent="1-16" drill="0.762" diameter="1.4224"/>
@@
 <contactref element="R10" pad="2"/>
 <wire x1="45.72" y1="50.8" x2="45.72" y2="48.26" width="0.6096" layer="16"/>
-<wire x1="45.72" y1="43.18" x2="43.18" y2="43.18" width="0.6096" layer="16"/>
+<wire x1="45.72" y1="45.72" x2="43.18" y2="43.18" width="0.6096" layer="16" curve="-90"/>
 <wire x1="40.64" y1="43.18" x2="43.18" y2="43.18" width="0.6096" layer="16"/>
-<wire x1="45.72" y1="43.18" x2="45.72" y2="48.26" width="0.6096" layer="16"/>
+<wire x1="45.72" y1="45.72" x2="45.72" y2="48.26" width="0.6096" layer="16"/>
 <via x="45.72" y="48.26" extent="1-16" drill="0.762" diameter="1.4224"/>
 <wire x1="45.72" y1="48.26" x2="40.64" y2="48.26" width="0.6096" layer="1"/>
@@
 <contactref element="X1" pad="2"/>
 <contactref element="IC1" pad="11"/>
-<wire x1="43.18" y1="17.78" x2="42.545" y2="17.78" width="0.6096" layer="16"/>
-<wire x1="42.545" y1="17.78" x2="38.1" y2="13.97" width="0.6096" layer="16" curve="90"/>
-<wire x1="38.1" y1="13.97" x2="33.655" y2="10.16" width="0.6096" layer="16" curve="-79.611142"/>
-<wire x1="33.655" y1="10.16" x2="7.62" y2="10.16" width="0.6096" layer="16"/>
+<wire x1="43.18" y1="17.78" x2="40.005" y2="17.78" width="0.6096" layer="16"/>
+<wire x1="40.005" y1="17.78" x2="35.56" y2="12.7" width="0.6096" layer="16" curve="90"/>
+<wire x1="35.56" y1="12.7" x2="33.02" y2="10.16" width="0.6096" layer="16" curve="-79.611142"/>
+<wire x1="33.02" y1="10.16" x2="7.62" y2="10.16" width="0.6096" layer="16"/>
 <wire x1="6.985" y1="10.16" x2="7.62" y2="10.16" width="0.6096" layer="16"/>
 </signal>
@@
 <contactref element="R11" pad="1"/>
 <contactref element="LED" pad="A"/>
-<wire x1="33.02" y1="12.7" x2="33.02" y2="13.97" width="0.6096" layer="16"/>
-<wire x1="33.02" y1="13.97" x2="31.75" y2="15.24" width="0.6096" layer="16" curve="90"/>
+<wire x1="30.48" y1="12.7" x2="30.48" y2="13.97" width="0.6096" layer="16"/>
+<wire x1="30.48" y1="13.97" x2="31.75" y2="15.24" width="0.6096" layer="16" curve="-90"/>
 </signal>
 <signal name="RX">

Commit message: ...
Routing:
- net N$4: track 2.54 -> 0.00 mm
- net GND: track 177.6 -> 176.1 mm
Changed lines of the file:
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@@
 <board>
 <plain>
-<wire x1="0" y1="0" x2="63.5" y2="0" width="0" layer="48"/>
-<wire x1="63.5" y1="0" x2="63.5" y2="53.34" width="0" layer="48"/>
-<wire x1="63.5" y1="53.34" x2="0" y2="53.34" width="0" layer="48"/>
-<wire x1="0" y1="53.34" x2="0" y2="0" width="0" layer="48"/>
 </plain>
 <attributes>
@@
 <classes>
 <class number="0" name="default" width="0" drill="0">
+<clearance class="0" value="0.381"/>
 </class>
 </classes>
@@
 <wire x1="45.72" y1="22.86" x2="43.18" y2="25.4" width="0.6096" layer="16" curve="90"/>
 <wire x1="40.64" y1="26.035" x2="43.18" y2="25.4" width="0.6096" layer="16"/>
-<wire x1="60.96" y1="20.32" x2="58.42" y2="20.32" width="0.6096" layer="16"/>
 <wire x1="50.8" y1="20.32" x2="53.34" y2="20.32" width="0.6096" layer="16"/>
 <wire x1="53.34" y1="20.32" x2="58.42" y2="20.32" width="0.6096" layer="16"/>
-<wire x1="60.96" y1="20.32" x2="60.96" y2="5.08" width="0.6096" layer="16"/>
+<wire x1="58.42" y1="20.32" x2="60.96" y2="17.78" width="0.6096" layer="16" curve="-90"/>
+<wire x1="60.96" y1="17.78" x2="60.96" y2="5.08" width="0.6096" layer="16"/>
 <wire x1="60.96" y1="5.08" x2="58.42" y2="2.54" width="0.6096" layer="16" curve="-90"/>
 <wire x1="55.88" y1="10.16" x2="55.88" y2="2.54" width="0.6096" layer="16"/>
@@
 <contactref element="X1" pad="2"/>
 <contactref element="IC1" pad="11"/>
-<wire x1="43.18" y1="17.78" x2="40.005" y2="17.78" width="0.6096" layer="16"/>
-<wire x1="40.005" y1="17.78" x2="35.56" y2="12.7" width="0.6096" layer="16" curve="90"/>
-<wire x1="35.56" y1="12.7" x2="33.02" y2="10.16" width="0.6096" layer="16" curve="-79.611142"/>
-<wire x1="33.02" y1="10.16" x2="7.62" y2="10.16" width="0.6096" layer="16"/>
+<wire x1="43.18" y1="17.78" x2="42.545" y2="17.78" width="0.6096" layer="16"/>
+<wire x1="42.545" y1="17.78" x2="38.1" y2="12.7" width="0.6096" layer="16" curve="90"/>
+<wire x1="38.1" y1="12.7" x2="35.56" y2="10.16" width="0.6096" layer="16" curve="-79.611142"/>
+<wire x1="35.56" y1="10.16" x2="7.62" y2="10.16" width="0.6096" layer="16"/>
 <wire x1="6.985" y1="10.16" x2="7.62" y2="10.16" width="0.6096" layer="16"/>
 </signal>
@@
 <contactref element="IC1" pad="13"/>
 <contactref element="R11" pad="2"/>
-<wire x1="40.64" y1="12.7" x2="43.18" y2="12.7" width="0.6096" layer="16"/>
+<wire x1="40.64" y1="12.7" x2="43.18" y2="12.7" width="0" layer="19" extent="1-1"/>
 </signal>
 </signals>

Commit message: ...
Routing:
- net GND: track 176.1 -> 175.4 mm
Changed lines of the file:
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@@
 <setting verticaltext="up"/>
 </settings>
-<grid distance="0.025" unitdist="inch" unit="inch" style="lines" multiple="4" display="yes" altdistance="0.005" altunitdist="inch" altunit="inch"/>
+<grid distance="0.01" unitdist="inch" unit="inch" style="lines" multiple="10" display="yes" altdistance="0.005" altunitdist="inch" altunit="inch"/>
 <layers>
 <layer number="1" name="Top" color="4" fill="1" visible="yes" active="yes"/>
@@
 <layer number="48" name="Document" color="7" fill="1" visible="yes" active="yes"/>
 <layer number="49" name="Reference" color="7" fill="1" visible="yes" active="yes"/>
-<layer number="50" name="dxf" color="7" fill="1" visible="yes" active="yes"/>
+<layer number="50" name="dxf" color="7" fill="1" visible="no" active="yes"/>
 <layer number="51" name="tDocu" color="6" fill="1" visible="yes" active="yes"/>
 <layer number="52" name="bDocu" color="7" fill="1" visible="no" active="yes"/>
@@
 <contactref element="JP1" pad="1"/>
 <contactref element="J2" pad="19"/>
-<wire x1="50.8" y1="20.32" x2="48.26" y2="20.32" width="0.6096" layer="16"/>
-<wire x1="48.26" y1="20.32" x2="45.72" y2="22.86" width="0.6096" layer="16" curve="-90"/>
-<wire x1="45.72" y1="22.86" x2="43.18" y2="25.4" width="0.6096" layer="16" curve="90"/>
-<wire x1="40.64" y1="26.035" x2="43.18" y2="25.4" width="0.6096" layer="16"/>
+<wire x1="50.8" y1="20.32" x2="50.546" y2="20.32" width="0.6096" layer="16"/>
+<wire x1="50.546" y1="20.32" x2="46.736" y2="22.606" width="0.6096" layer="16" curve="-60"/>
 <wire x1="50.8" y1="20.32" x2="53.34" y2="20.32" width="0.6096" layer="16"/>
 <wire x1="53.34" y1="20.32" x2="58.42" y2="20.32" width="0.6096" layer="16"/>
@@
 <wire x1="27.94" y1="25.4" x2="30.48" y2="22.86" width="0.6096" layer="16" curve="-90"/>
 <wire x1="25.4" y1="25.4" x2="22.86" y2="27.94" width="0.6096" layer="16" curve="-90"/>
+<wire x1="46.736" y1="22.606" x2="40.64" y2="26.035" width="0.6096" layer="16" curve="60"/>
 </signal>
 <signal name="N$7">
@@
 <contactref element="Q1" pad="1"/>
 <contactref element="IC1" pad="9"/>
-<wire x1="43.18" y1="22.86" x2="41.91" y2="22.86" width="0.6096" layer="16"/>
-<wire x1="41.91" y1="22.86" x2="40.64" y2="23.495" width="0.6096" layer="16" curve="-75"/>
-<wire x1="40.64" y1="23.495" x2="39.37" y2="24.13" width="0.6096" layer="16" curve="75"/>
-<wire x1="39.37" y1="24.13" x2="38.1" y2="24.13" width="0.6096" layer="16"/>
+<wire x1="43.18" y1="22.86" x2="40.64" y2="23.495" width="0.6096" layer="16" curve="-30"/>
+<wire x1="40.64" y1="23.495" x2="38.1" y2="24.13" width="0.6096" layer="16" curve="30"/>
 <wire x1="33.02" y1="22.86" x2="34.29" y2="24.13" width="0.6096" layer="16" curve="-90"/>
 <wire x1="34.29" y1="24.13" x2="38.1" y2="24.13" width="0.6096" layer="16"/>
@@
 <contactref element="Q1" pad="2"/>
 <contactref element="IC1" pad="10"/>
-<wire x1="43.18" y1="20.32" x2="41.91" y2="20.32" width="0.6096" layer="16"/>
-<wire x1="41.91" y1="20.32" x2="40.64" y2="19.685" width="0.6096" layer="16" curve="75"/>
-<wire x1="40.64" y1="19.685" x2="39.37" y2="19.05" width="0.6096" layer="16" curve="-75"/>
-<wire x1="39.37" y1="19.05" x2="38.1" y2="19.05" width="0.6096" layer="16"/>
+<wire x1="43.18" y1="20.32" x2="40.64" y2="19.685" width="0.6096" layer="16" curve="30"/>
+<wire x1="40.64" y1="19.685" x2="38.1" y2="19.05" width="0.6096" layer="16" curve="-30"/>
 <wire x1="33.02" y1="20.32" x2="34.29" y2="19.05" width="0.6096" layer="16" curve="90"/>
 <wire x1="34.29" y1="19.05" x2="38.1" y2="19.05" width="0.6096" layer="16"/>
@@
 <contactref element="C2" pad="2"/>
 <contactref element="K2" pad="4"/>
-<wire x1="15.24" y1="35.56" x2="17.78" y2="33.02" width="0.6096" layer="16" curve="90"/>
-<wire x1="17.78" y1="33.02" x2="20.32" y2="30.48" width="0.6096" layer="16" curve="-90"/>
+<wire x1="15.24" y1="35.56" x2="17.78" y2="33.02" width="0.6096" layer="16" curve="75"/>
+<wire x1="17.78" y1="33.02" x2="20.32" y2="30.48" width="0.6096" layer="16" curve="-75"/>
 <wire x1="20.32" y1="30.48" x2="20.32" y2="20.32" width="0.6096" layer="16"/>
 <wire x1="20.32" y1="20.32" x2="25.4" y2="15.24" width="0.6096" layer="16" curve="90"/>

Commit message: ...
Parts:
- L1: device l:L-02/5V -> l:L-02/7V
- moved L1 1.27 mm to (14.0, 45.7)
Routing:
- net GND: track 175.4 -> 185.3 mm
- net N$4: track 0.00 -> 2.54 mm
- net N$2: track 27.5 -> 30.0 mm
- net /LC: track 74.3 -> 72.0 mm
- removed copper zone on layer 16, net GND
Other:
- board outline added: 63.5 x 53.3 mm
