File: eagle/attic/unrouted/LCmeter0-perfboard-norelay.brd (EAGLE design)
At the start: 161.3 x 100 mm, 25 parts, among them IC1 PIC16F876A-X/SP, Q1 20MHz, Q2 BC548, SW1 SPST, SW2 DPDT

Commit message: ...
Changed lines of the file:
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@@
 <contactref element="R2" pad="2"/>
 <contactref element="C3" pad="+"/>
-<wire x1="30.48" y1="27.94" x2="25.4" y2="27.94" width="0.4064" layer="16"/>
-<wire x1="25.4" y1="27.94" x2="12.7" y2="27.94" width="0.4064" layer="16"/>
-<wire x1="10.16" y1="27.94" x2="12.7" y2="27.94" width="0.4064" layer="16"/>
-<wire x1="12.7" y1="30.48" x2="12.7" y2="27.94" width="0.6096" layer="16"/>
+<wire x1="30.48" y1="27.94" x2="25.4" y2="27.94" width="1.27" layer="16"/>
+<wire x1="25.4" y1="27.94" x2="12.7" y2="27.94" width="1.27" layer="16"/>
+<wire x1="10.16" y1="27.94" x2="12.7" y2="27.94" width="1.27" layer="16"/>
+<wire x1="12.7" y1="30.48" x2="12.7" y2="27.94" width="1.27" layer="16"/>
 </signal>
 <signal name="N$2">
@@
 <contactref element="C3" pad="-"/>
 <contactref element="SW2" pad="1-2"/>
-<wire x1="5.08" y1="20.32" x2="5.08" y2="27.94" width="0.4064" layer="16"/>
-<wire x1="5.08" y1="15.24" x2="5.08" y2="27.94" width="0.4064" layer="16"/>
+<wire x1="5.08" y1="20.32" x2="5.08" y2="27.94" width="1.27" layer="16"/>
+<wire x1="5.08" y1="15.24" x2="5.08" y2="27.94" width="1.27" layer="16"/>
 <wire x1="5.08" y1="33.02" x2="5.08" y2="38.1" width="0" layer="19" extent="1-1"/>
 <wire x1="5.08" y1="27.94" x2="5.08" y2="33.02" width="0" layer="19" extent="1-1"/>
@@
 <contactref element="IC1" pad="2"/>
 <contactref element="IC1" pad="7"/>
-<wire x1="30.48" y1="22.86" x2="33.02" y2="25.4" width="0.4064" layer="16"/>
-<wire x1="33.02" y1="25.4" x2="33.02" y2="33.02" width="0.4064" layer="16"/>
-<wire x1="33.02" y1="33.02" x2="30.48" y2="35.56" width="0.4064" layer="16"/>
-<wire x1="30.48" y1="35.56" x2="27.94" y2="35.56" width="0.4064" layer="16"/>
-<wire x1="27.94" y1="35.56" x2="25.4" y2="35.56" width="0.4064" layer="16"/>
+<wire x1="30.48" y1="22.86" x2="33.02" y2="25.4" width="1.27" layer="16"/>
+<wire x1="33.02" y1="25.4" x2="33.02" y2="33.02" width="1.27" layer="16"/>
+<wire x1="33.02" y1="33.02" x2="30.48" y2="35.56" width="1.27" layer="16"/>
+<wire x1="30.48" y1="35.56" x2="27.94" y2="35.56" width="1.27" layer="16"/>
+<wire x1="27.94" y1="35.56" x2="25.4" y2="35.56" width="1.27" layer="16"/>
 </signal>
 <signal name="A1">
@@
 <contactref element="C4" pad="+"/>
 <contactref element="IC1" pad="3"/>
-<wire x1="30.48" y1="33.02" x2="27.94" y2="33.02" width="0.4064" layer="16"/>
-<wire x1="27.94" y1="33.02" x2="22.86" y2="33.02" width="0.4064" layer="16"/>
+<wire x1="30.48" y1="33.02" x2="27.94" y2="33.02" width="1.27" layer="16"/>
+<wire x1="27.94" y1="33.02" x2="22.86" y2="33.02" width="1.27" layer="16"/>
 </signal>
 <signal name="GND">
@@
 <contactref element="JP1" pad="1"/>
 <contactref element="CLK" pad="1"/>
-<wire x1="22.86" y1="43.18" x2="17.78" y2="43.18" width="0.8128" layer="16"/>
-<wire x1="17.78" y1="43.18" x2="17.78" y2="33.02" width="0.8128" layer="16"/>
+<wire x1="22.86" y1="43.18" x2="17.78" y2="43.18" width="1.27" layer="16"/>
+<wire x1="17.78" y1="43.18" x2="17.78" y2="33.02" width="1.27" layer="16"/>
 <wire x1="17.78" y1="33.02" x2="17.78" y2="20.32" width="0.8128" layer="1"/>
-<wire x1="17.78" y1="20.32" x2="17.78" y2="17.78" width="0.8128" layer="16"/>
-<wire x1="17.78" y1="17.78" x2="17.78" y2="15.24" width="0.8128" layer="16"/>
-<wire x1="30.48" y1="20.32" x2="27.94" y2="20.32" width="0.8128" layer="16"/>
-<wire x1="27.94" y1="20.32" x2="27.94" y2="22.86" width="0.8128" layer="16"/>
-<wire x1="27.94" y1="22.86" x2="22.86" y2="22.86" width="0.8128" layer="16"/>
-<wire x1="22.86" y1="22.86" x2="22.86" y2="20.32" width="0.8128" layer="16"/>
-<wire x1="22.86" y1="20.32" x2="17.78" y2="20.32" width="0.8128" layer="16"/>
-<wire x1="22.86" y1="43.18" x2="27.94" y2="43.18" width="0.8128" layer="16"/>
+<wire x1="17.78" y1="20.32" x2="17.78" y2="17.78" width="1.27" layer="16"/>
+<wire x1="17.78" y1="17.78" x2="17.78" y2="15.24" width="1.27" layer="16"/>
+<wire x1="30.48" y1="20.32" x2="27.94" y2="20.32" width="1.27" layer="16"/>
+<wire x1="27.94" y1="20.32" x2="27.94" y2="22.86" width="1.27" layer="16"/>
+<wire x1="27.94" y1="22.86" x2="22.86" y2="22.86" width="1.27" layer="16"/>
+<wire x1="22.86" y1="22.86" x2="22.86" y2="20.32" width="1.27" layer="16"/>
+<wire x1="22.86" y1="20.32" x2="17.78" y2="20.32" width="1.27" layer="16"/>
+<wire x1="22.86" y1="43.18" x2="27.94" y2="43.18" width="1.27" layer="16"/>
 <via x="17.78" y="20.32" extent="1-16" drill="0.6" shape="square"/>
-<wire x1="17.78" y1="5.08" x2="22.86" y2="5.08" width="0.6096" layer="16"/>
-<wire x1="10.16" y1="7.62" x2="12.7" y2="5.08" width="0.6096" layer="16"/>
-<wire x1="12.7" y1="5.08" x2="17.78" y2="5.08" width="0.6096" layer="16"/>
-<wire x1="17.78" y1="5.08" x2="17.78" y2="15.24" width="0.6096" layer="16"/>
-<wire x1="17.78" y1="15.24" x2="17.78" y2="20.32" width="0.6096" layer="16"/>
-<wire x1="10.16" y1="20.32" x2="17.78" y2="20.32" width="0.6096" layer="16"/>
-<wire x1="12.7" y1="20.32" x2="17.78" y2="20.32" width="0.8128" layer="16"/>
-<wire x1="12.7" y1="20.32" x2="10.16" y2="20.32" width="0.8128" layer="16"/>
+<wire x1="17.78" y1="5.08" x2="22.86" y2="5.08" width="1.27" layer="16"/>
+<wire x1="10.16" y1="7.62" x2="12.7" y2="5.08" width="1.27" layer="16"/>
+<wire x1="12.7" y1="5.08" x2="17.78" y2="5.08" width="1.27" layer="16"/>
+<wire x1="17.78" y1="5.08" x2="17.78" y2="15.24" width="1.27" layer="16"/>
+<wire x1="17.78" y1="15.24" x2="17.78" y2="20.32" width="1.27" layer="16"/>
+<wire x1="10.16" y1="20.32" x2="17.78" y2="20.32" width="1.27" layer="16"/>
+<wire x1="12.7" y1="20.32" x2="17.78" y2="20.32" width="1.27" layer="16"/>
+<wire x1="12.7" y1="20.32" x2="10.16" y2="20.32" width="1.27" layer="16"/>
 <wire x1="46.99" y1="15.24" x2="46.99" y2="20.32" width="0" layer="19" extent="1-1"/>
 <wire x1="40.64" y1="15.24" x2="46.99" y2="15.24" width="0" layer="19" extent="1-1"/>
@@
 <contactref element="IC1" pad="1"/>
 <contactref element="JP1" pad="3"/>
-<wire x1="33.02" y1="43.18" x2="33.02" y2="40.64" width="0.4064" layer="16"/>
-<wire x1="33.02" y1="40.64" x2="30.48" y2="38.1" width="0.4064" layer="16"/>
-<wire x1="30.48" y1="38.1" x2="27.94" y2="38.1" width="0.4064" layer="16"/>
-<wire x1="27.94" y1="38.1" x2="22.86" y2="38.1" width="0.4064" layer="16"/>
+<wire x1="33.02" y1="43.18" x2="33.02" y2="40.64" width="1.27" layer="16"/>
+<wire x1="33.02" y1="40.64" x2="30.48" y2="38.1" width="1.27" layer="16"/>
+<wire x1="30.48" y1="38.1" x2="27.94" y2="38.1" width="1.27" layer="16"/>
+<wire x1="27.94" y1="38.1" x2="22.86" y2="38.1" width="1.27" layer="16"/>
 </signal>
 <signal name="N$5">
@@
 <contactref element="C2" pad="2"/>
 <contactref element="Q2" pad="C"/>
-<wire x1="10.16" y1="15.24" x2="10.16" y2="12.7" width="0.4064" layer="16"/>
+<wire x1="10.16" y1="15.24" x2="10.16" y2="12.7" width="1.27" layer="16"/>
 </signal>
 <signal name="RX">
@@
 <contactref element="IC1" pad="11"/>
 <contactref element="CLK" pad="2"/>
-<wire x1="30.48" y1="12.7" x2="27.94" y2="12.7" width="0.4064" layer="16"/>
-<wire x1="27.94" y1="12.7" x2="25.4" y2="10.16" width="0.4064" layer="16"/>
-<wire x1="25.4" y1="10.16" x2="25.4" y2="5.08" width="0.4064" layer="16"/>
+<wire x1="30.48" y1="12.7" x2="27.94" y2="12.7" width="1.27" layer="16"/>
+<wire x1="27.94" y1="12.7" x2="25.4" y2="10.16" width="1.27" layer="16"/>
+<wire x1="25.4" y1="10.16" x2="25.4" y2="5.08" width="1.27" layer="16"/>
 </signal>
 <signal name="N$3">
